Commit message: fixed changing solution and better parameterization

File: body.urdf (robot description, URDF)
Before this commit: robot robot, 12 links, 13 joints
Links:
- removed link 10
- removed link 11
- removed link 5
- removed link 6
- removed link 7
- removed link 8
- removed link 9
- link 0: geometry collision box size=0.10551505731319763 0.19860711547421198 0.138903373409246; visual box size=0.10551505731319763 0.19860711547421198 0.138903373409246
- link 1: geometry collision box size=0.5579103328953636 0.5449220783795011 0.4445897305473676; visual box size=0.5579103328953636 0.5449220783795011 0.4445897305473676
- link 2: geometry collision box size=0.2758777087190195 0.49059777034090857 0.5007131122632975; visual box size=0.2758777087190195 0.49059777034090857 0.5007131122632975
- link 3: geometry collision box size=0.513862130921519 0.49243706010279553 0.2320159086020013; visual box size=0.513862130921519 0.49243706010279553 0.2320159086020013
- link 4: geometry collision box size=0.4681287448782476 0.25439141455654735 0.4707768439487897; visual box size=0.4681287448782476 0.25439141455654735 0.4707768439487897
Joints:
- removed joint 0_11
- removed joint 0_12
- removed joint 10_11
- removed joint 4_5
- removed joint 5_6
- removed joint 6_7
- removed joint 7_8
- removed joint 8_9
- removed joint 9_101
- removed joint 9_102
- added joint 0_1: type revolute, parent 0, child 1, origin xyz=0 0.09930355773710599 0.3 rpy=0 0 0, axis 1 0 0, limit lower=-3.14159 upper=3.14159 effort=0.0 velocity=0.0
- joint 1_2: axis 1 0 0 -> 0 1 0; origin xyz=0 0.414836840193484 0 rpy=0 0 0 -> xyz=0 0.5449220783795011 0 rpy=0 0 0
- joint 2_3: origin xyz=0 0.4971516350634293 0 rpy=0 0 0 -> xyz=0 0.49059777034090857 0 rpy=0 0 0
- joint 3_4: axis 0 1 0 -> 1 0 0; origin xyz=0 0.15328055195769766 0 rpy=0 0 0 -> xyz=0 0.49243706010279553 0 rpy=0 0 0

Commit message: at elast one sensor

File: body.urdf (robot description, URDF)
Before this commit: robot robot, 5 links, 4 joints
Links:
- link 0: geometry collision box size=0.2293426114734203 0.49100900649655665 0.5718780548394973; visual box size=0.2293426114734203 0.49100900649655665 0.5718780548394973
- link 1: geometry collision box size=0.5936285252410223 0.2433474789494374 0.23353084162222468; visual box size=0.5936285252410223 0.2433474789494374 0.23353084162222468
- link 2: geometry collision box size=0.10092052837123497 0.4300472896762859 0.49448674386183933; visual box size=0.10092052837123497 0.4300472896762859 0.49448674386183933
- link 3: geometry collision box size=0.27725529216483835 0.5291958037766247 0.5532673825298615; visual box size=0.27725529216483835 0.5291958037766247 0.5532673825298615
- link 4: geometry collision box size=0.5356509896937689 0.27437562206901656 0.15858107442595423; visual box size=0.5356509896937689 0.27437562206901656 0.15858107442595423
Joints:
- joint 0_1: origin xyz=0 0.09930355773710599 0.3 rpy=0 0 0 -> xyz=0 0.24550450324827833 0.3 rpy=0 0 0
- joint 1_2: origin xyz=0 0.5449220783795011 0 rpy=0 0 0 -> xyz=0 0.2433474789494374 0 rpy=0 0 0
- joint 2_3: axis 0 1 0 -> 1 0 0; origin xyz=0 0.49059777034090857 0 rpy=0 0 0 -> xyz=0 0.4300472896762859 0 rpy=0 0 0
- joint 3_4: axis 1 0 0 -> 0 1 0; origin xyz=0 0.49243706010279553 0 rpy=0 0 0 -> xyz=0 0.5291958037766247 0 rpy=0 0 0

Commit message: added spheres

File: body.urdf (robot description, URDF)
Before this commit: robot robot, 5 links, 4 joints
Links:
- added link 10, mass 1; collision box size=0.12219642038251102 0.17301749739081332 0.19132775926258708; visual box size=0.12219642038251102 0.17301749739081332 0.19132775926258708
- added link 11, mass 1; collision box size=0.2419966811298007 0.48612393250902275 0.1633041117106769; visual box size=0.2419966811298007 0.48612393250902275 0.1633041117106769
- added link 5, mass 1; collision box size=0.23826855532002408 0.29548824320187483 0.5425828905588547; visual box size=0.23826855532002408 0.29548824320187483 0.5425828905588547
- added link 6, mass 1; collision box size=0.26009728279057853 0.5796416385076466 0.38632629673301255; visual box size=0.26009728279057853 0.5796416385076466 0.38632629673301255
- added link 7, mass 1; collision box size=0.21346941707716413 0.1825520333982282 0.36673354908614697; visual box size=0.21346941707716413 0.1825520333982282 0.36673354908614697
- added link 8, mass 1; collision box size=0.523961460354506 0.4373879472852611 0.11406112732375215; visual box size=0.523961460354506 0.4373879472852611 0.11406112732375215
- added link 9, mass 1; collision box size=0.3141760780199896 0.1279798757842164 0.4562507401448431; visual box size=0.3141760780199896 0.1279798757842164 0.4562507401448431
- link 0: geometry collision box size=0.3257541240465047 0.5921909964655744 0.4560762770283111; visual box size=0.3257541240465047 0.5921909964655744 0.4560762770283111
- link 1: geometry collision box size=0.3361791174776946 0.405365072921401 0.24790054633320188; visual box size=0.3361791174776946 0.405365072921401 0.24790054633320188
- link 2: geometry collision box size=0.11211155595168318 0.4916059296906763 0.13687935912137464; visual box size=0.11211155595168318 0.4916059296906763 0.13687935912137464
- link 3: geometry collision box size=0.30083859808069957 0.4020128103573074 0.3360457874985493; visual box size=0.30083859808069957 0.4020128103573074 0.3360457874985493
- link 4: geometry collision box size=0.2825106691595204 0.2261146708022169 0.35462707640706004; visual box size=0.2825106691595204 0.2261146708022169 0.35462707640706004
Joints:
- added joint 10_11: type revolute, parent 10, child 11, origin xyz=0 0.17301749739081332 0 rpy=0 0 0, axis 1 0 0, limit lower=-3.14159 upper=3.14159 effort=0.0 velocity=0.0
- added joint 4_5: type revolute, parent 4, child 5, origin xyz=0 0.2261146708022169 0 rpy=0 0 0, axis 1 0 0, limit lower=-3.14159 upper=3.14159 effort=0.0 velocity=0.0
- added joint 5_6: type revolute, parent 5, child 6, origin xyz=0 0.29548824320187483 0 rpy=0 0 0, axis 1 0 0, limit lower=-3.14159 upper=3.14159 effort=0.0 velocity=0.0
- added joint 6_7: type revolute, parent 6, child 7, origin xyz=0 0.5796416385076466 0 rpy=0 0 0, axis 1 0 0, limit lower=-3.14159 upper=3.14159 effort=0.0 velocity=0.0
- added joint 7_8: type revolute, parent 7, child 8, origin xyz=0 0.1825520333982282 0 rpy=0 0 0, axis 0 0 1, limit lower=-3.14159 upper=3.14159 effort=0.0 velocity=0.0
- added joint 8_9: type revolute, parent 8, child 9, origin xyz=0 0.4373879472852611 0 rpy=0 0 0, axis 1 0 0, limit lower=-3.14159 upper=3.14159 effort=0.0 velocity=0.0
- added joint 9_10: type revolute, parent 9, child 10, origin xyz=0 0.1279798757842164 0 rpy=0 0 0, axis 1 0 0, limit lower=-3.14159 upper=3.14159 effort=0.0 velocity=0.0
- joint 0_1: axis 1 0 0 -> 0 0 1; origin xyz=0 0.24550450324827833 0.3 rpy=0 0 0 -> xyz=0 0.2960954982327872 0.3 rpy=0 0 0
- joint 1_2: axis 0 1 0 -> 1 0 0; origin xyz=0 0.2433474789494374 0 rpy=0 0 0 -> xyz=0 0.405365072921401 0 rpy=0 0 0
- joint 2_3: axis 1 0 0 -> 0 0 1; origin xyz=0 0.4300472896762859 0 rpy=0 0 0 -> xyz=0 0.4916059296906763 0 rpy=0 0 0
- joint 3_4: axis 0 1 0 -> 1 0 0; origin xyz=0 0.5291958037766247 0 rpy=0 0 0 -> xyz=0 0.4020128103573074 0 rpy=0 0 0

Commit message: functioning code

File: body.urdf (robot description, URDF)
Before this commit: robot robot, 12 links, 11 joints
Links:
- removed link 10
- removed link 2
- removed link 3
- removed link 4
- removed link 5
- removed link 6
- removed link 7
- removed link 8
- removed link 9
- link 0: geometry collision box size=0.5634525266034095 0.10296698036087645 0.44546217019873136; visual box size=0.5634525266034095 0.10296698036087645 0.44546217019873136
- link 1: geometry collision box size=0.33594493409532955 0.32240294929156266 0.3862811828476507; visual box size=0.33594493409532955 0.32240294929156266 0.3862811828476507
- link 11: geometry collision box size=0.2763985970631684 0.16530436005342983 0.576889268752698; visual box size=0.2763985970631684 0.16530436005342983 0.576889268752698
Joints:
- removed joint 10_11
- removed joint 1_2
- removed joint 2_3
- removed joint 3_4
- removed joint 4_5
- removed joint 5_6
- removed joint 6_7
- removed joint 7_8
- removed joint 8_9
- removed joint 9_10
- added joint 1_11: type revolute, parent 1, child 11, origin xyz=0.33594493409532955 0 -0.19314059142382534 rpy=0 0 0, axis 0 1 0, limit lower=-3.14159 upper=3.14159 effort=0.0 velocity=0.0
- joint 0_1: origin xyz=0 0.2960954982327872 0.3 rpy=0 0 0 -> xyz=0.28172626330170475 0 2 rpy=0 0 0

Commit message: Read Me Updated

File: body.urdf (robot description, URDF)
Before this commit: robot robot, 3 links, 2 joints
Links:
- added link 2, mass 1; collision box size=0.15838912915100958 0.17556283838524847 0.5560753664523135; visual box size=0.15838912915100958 0.17556283838524847 0.5560753664523135
- added link 21, mass 1; collision box size=0.5144535908541867 0.2908328949696154 0.11102567607564237; visual box size=0.5144535908541867 0.2908328949696154 0.11102567607564237
- added link 22, mass 1; collision box size=0.13936381034315806 0.417812657375107 0.4419667963613165; visual box size=0.13936381034315806 0.417812657375107 0.4419667963613165
- link 0: geometry collision box size=0.1830161649720735 0.40754701228827395 0.23498988619585595; visual box size=0.1830161649720735 0.40754701228827395 0.23498988619585595
- link 1: geometry collision box size=0.23483698614609913 0.22307614877746082 0.25141732423882357; visual box size=0.23483698614609913 0.22307614877746082 0.25141732423882357
- link 11: geometry collision box size=0.39889317880311514 0.13670274341867464 0.4717774654888164; visual box size=0.39889317880311514 0.13670274341867464 0.4717774654888164
Joints:
- added joint 0_2: type revolute, parent 0, child 2, origin xyz=0 0 1.882505056902072 rpy=0 0 0, axis 0 1 0, limit lower=-3.14159 upper=3.14159 effort=0.0 velocity=0.0
- added joint 2_21: type revolute, parent 2, child 21, origin xyz=0.07919456457550479 0 -0.5560753664523135 rpy=0 0 0, axis 0 1 0, limit lower=-3.14159 upper=3.14159 effort=0.0 velocity=0.0
- added joint 2_22: type revolute, parent 2, child 22, origin xyz=0 -0.08778141919262424 -0.5560753664523135 rpy=0 0 0, axis 1 0 0, limit lower=-3.14159 upper=3.14159 effort=0.0 velocity=0.0
- joint 0_1: axis 0 0 1 -> 1 0 0; origin xyz=0.28172626330170475 0 2 rpy=0 0 0 -> xyz=0 0.20377350614413697 2 rpy=0 0 0
- joint 1_11: axis 0 1 0 -> 1 0 0; origin xyz=0.33594493409532955 0 -0.19314059142382534 rpy=0 0 0 -> xyz=0 0.22307614877746082 0.12570866211941178 rpy=0 0 0

Commit message: body ID

File: body.urdf (robot description, URDF)
Before this commit: robot robot, 6 links, 5 joints
Links:
- added link 111, mass 1; collision box size=0.35399950764610055 0.11125922549572545 0.4448563412059039; visual box size=0.35399950764610055 0.11125922549572545 0.4448563412059039
- added link 112, mass 1; collision box size=0.42567054823825945 0.17645485592087498 0.5844182463708708; visual box size=0.42567054823825945 0.17645485592087498 0.5844182463708708
- added link 211, mass 1; collision box size=0.48180635565651353 0.16061456141093547 0.328399289625551; visual box size=0.48180635565651353 0.16061456141093547 0.328399289625551
- added link 212, mass 1; collision box size=0.30980537187454826 0.2922575772193098 0.5680380890608191; visual box size=0.30980537187454826 0.2922575772193098 0.5680380890608191
- added link 221, mass 1; collision box size=0.24093195747808863 0.1598217290761403 0.2841589619840962; visual box size=0.24093195747808863 0.1598217290761403 0.2841589619840962
- link 0: geometry collision box size=0.5906178884501417 0.4394827752588889 0.2099552660585677; visual box size=0.5906178884501417 0.4394827752588889 0.2099552660585677
- link 1: geometry collision box size=0.1292582771443733 0.45384294291927085 0.1260355352800179; visual box size=0.1292582771443733 0.45384294291927085 0.1260355352800179
- link 11: geometry collision box size=0.1665769977991309 0.5739983846479252 0.2285286189897104; visual box size=0.1665769977991309 0.5739983846479252 0.2285286189897104
- link 2: geometry collision box size=0.5353630535978452 0.5431646785360508 0.4149317583415638; visual box size=0.5353630535978452 0.5431646785360508 0.4149317583415638
- link 21: geometry collision box size=0.10807893790577563 0.3981031282460137 0.35629019814582796; visual box size=0.10807893790577563 0.3981031282460137 0.35629019814582796
- link 22: geometry collision box size=0.589391813606632 0.18122344946513538 0.16850482660622954; visual box size=0.589391813606632 0.18122344946513538 0.16850482660622954
Joints:
- added joint 11_111: type revolute, parent 11, child 111, origin xyz=0.1665769977991309 0 0 rpy=0 0 0, axis 0 1 0, limit lower=-3.14159 upper=3.14159 effort=0.0 velocity=0.0
- added joint 11_112: type revolute, parent 11, child 112, origin xyz=0.1665769977991309 0 0 rpy=0 0 0, axis 0 1 0, limit lower=-3.14159 upper=3.14159 effort=0.0 velocity=0.0
- added joint 21_211: type revolute, parent 21, child 211, origin xyz=-0.10807893790577563 0 0 rpy=0 0 0, axis 0 0 1, limit lower=-3.14159 upper=3.14159 effort=0.0 velocity=0.0
- added joint 21_212: type revolute, parent 21, child 212, origin xyz=-0.10807893790577563 0 0 rpy=0 0 0, axis 0 1 0, limit lower=-3.14159 upper=3.14159 effort=0.0 velocity=0.0
- added joint 22_221: type revolute, parent 22, child 221, origin xyz=-0.589391813606632 0 0 rpy=0 0 0, axis 0 1 0, limit lower=-3.14159 upper=3.14159 effort=0.0 velocity=0.0
- joint 0_1: axis 1 0 0 -> 0 0 1; origin xyz=0 0.20377350614413697 2 rpy=0 0 0 -> xyz=0 0.21974138762944445 2 rpy=0 0 0
- joint 0_2: origin xyz=0 0 1.882505056902072 rpy=0 0 0 -> xyz=0 0 1.8950223669707162 rpy=0 0 0
- joint 1_11: axis 1 0 0 -> 0 0 1; origin xyz=0 0.22307614877746082 0.12570866211941178 rpy=0 0 0 -> xyz=0.06462913857218665 0.45384294291927085 0 rpy=0 0 0
- joint 2_21: origin xyz=0.07919456457550479 0 -0.5560753664523135 rpy=0 0 0 -> xyz=-0.2676815267989226 0 -0.4149317583415638 rpy=0 0 0
- joint 2_22: axis 1 0 0 -> 0 1 0; origin xyz=0 -0.08778141919262424 -0.5560753664523135 rpy=0 0 0 -> xyz=-0.2676815267989226 0 -0.4149317583415638 rpy=0 0 0
