Commit message: working random seed

File: body1.urdf (robot description, URDF)
Before this commit: robot robot, 5 links, 4 joints
Links:
- removed link 000
- removed link 011
- removed link 100
- added link 001, mass 1; collision box size=0.5 0.5 0.5; visual box size=0.5 0.5 0.5
- added link 010, mass 1; collision box size=0.5 0.5 0.5; visual box size=0.5 0.5 0.5
Joints:
- removed joint 000_011
- removed joint 000_100
- removed joint 100_101
- added joint 001_010: type revolute, parent 001, child 010, origin xyz=0.0 0.25 0.5 rpy=0 0 0, axis 1 0 0, limit lower=-3.14159 upper=3.14159 effort=0.0 velocity=0.0
- added joint 001_101: type revolute, parent 001, child 101, origin xyz=0.25 0.0 0.75 rpy=0 0 0, axis 0 1 0, limit lower=-3.14159 upper=3.14159 effort=0.0 velocity=0.0
- joint 101_110: origin xyz=0.0 0.25 0.0 rpy=0 0 0 -> xyz=0.25 0.25 -0.25 rpy=0 0 0

File: body4.urdf (robot description, URDF)
Before this commit: robot robot, 5 links, 4 joints
Links:
- removed link 000
- removed link 011
- added link 010, mass 1; collision box size=0.5 0.5 0.5; visual box size=0.5 0.5 0.5
Joints:
- removed joint 000_011
- removed joint 000_100
- added joint 010_100: type revolute, parent 010, child 100, origin xyz=0.25 0.25 0.25 rpy=0 0 0, axis 0 0 1, limit lower=-3.14159 upper=3.14159 effort=0.0 velocity=0.0
- joint 100_101: origin xyz=0.25 0.0 0.25 rpy=0 0 0 -> xyz=0.25 -0.25 0.25 rpy=0 0 0

File: body5.urdf (robot description, URDF)
Before this commit: robot robot, 5 links, 4 joints
Links:
- removed link 110
- added link 010, mass 1; collision box size=0.5 0.5 0.5; visual box size=0.5 0.5 0.5
- added link 111, mass 1; collision box size=0.5 0.5 0.5; visual box size=0.5 0.5 0.5
Joints:
- removed joint 100_101
- removed joint 101_110
- added joint 000_010: type revolute, parent 000, child 010, origin xyz=0.0 0.25 0.25 rpy=0 0 0, axis 0 0 1, limit lower=-3.14159 upper=3.14159 effort=0.0 velocity=0.0
- added joint 011_101: type revolute, parent 011, child 101, origin xyz=0.25 0.0 0.25 rpy=0 0 0, axis 0 0 1, limit lower=-3.14159 upper=3.14159 effort=0.0 velocity=0.0
- added joint 101_111: type revolute, parent 101, child 111, origin xyz=0.25 0.0 0.0 rpy=0 0 0, axis 0 0 1, limit lower=-3.14159 upper=3.14159 effort=0.0 velocity=0.0
- joint 000_100: axis 0 0 1 -> 0 1 0

File: body6.urdf (robot description, URDF)
Before this commit: robot robot, 5 links, 4 joints
Links:
- removed link 000
- added link 010, mass 1; collision box size=0.5 0.5 0.5; visual box size=0.5 0.5 0.5
- added link 111, mass 1; collision box size=0.5 0.5 0.5; visual box size=0.5 0.5 0.5
Joints:
- removed joint 000_011
- removed joint 000_100
- removed joint 100_101
- added joint 010_011: type revolute, parent 010, child 011, origin xyz=0.0 0.5 0.5 rpy=0 0 0, axis 0 1 0, limit lower=-3.14159 upper=3.14159 effort=0.0 velocity=0.0
- added joint 010_100: type revolute, parent 010, child 100, origin xyz=0.25 0.25 0.25 rpy=0 0 0, axis 0 0 1, limit lower=-3.14159 upper=3.14159 effort=0.0 velocity=0.0
- added joint 011_101: type revolute, parent 011, child 101, origin xyz=0.25 -0.25 0.25 rpy=0 0 0, axis 0 0 1, limit lower=-3.14159 upper=3.14159 effort=0.0 velocity=0.0
- added joint 011_111: type revolute, parent 011, child 111, origin xyz=0.25 0.0 0.25 rpy=0 0 0, axis 0 0 1, limit lower=-3.14159 upper=3.14159 effort=0.0 velocity=0.0
- joint 101_110: origin xyz=0.0 0.25 0.0 rpy=0 0 0 -> xyz=0.25 0.0 -0.25 rpy=0 0 0
