Commit message: bug fixes

File: body3.urdf (robot description, URDF)
Before this commit: robot robot, 20 links, 19 joints
Links:
- removed link 001
- removed link 010
- removed link 102
- removed link 120
- removed link 132
- removed link 200
- removed link 212
- removed link 220
- removed link 231
- added link 000, mass 1; collision box size=0.5 0.5 0.5; visual box size=0.5 0.5 0.5
- added link 030, mass 1; collision box size=0.5 0.5 0.5; visual box size=0.5 0.5 0.5
- added link 032, mass 1; collision box size=0.5 0.5 0.5; visual box size=0.5 0.5 0.5
- added link 110, mass 1; collision box size=0.5 0.5 0.5; visual box size=0.5 0.5 0.5
- added link 122, mass 1; collision box size=0.5 0.5 0.5; visual box size=0.5 0.5 0.5
- added link 130, mass 1; collision box size=0.5 0.5 0.5; visual box size=0.5 0.5 0.5
- added link 201, mass 1; collision box size=0.5 0.5 0.5; visual box size=0.5 0.5 0.5
- added link 210, mass 1; collision box size=0.5 0.5 0.5; visual box size=0.5 0.5 0.5
- added link 221, mass 1; collision box size=0.5 0.5 0.5; visual box size=0.5 0.5 0.5
- added link 232, mass 1; collision box size=0.5 0.5 0.5; visual box size=0.5 0.5 0.5
- link 002: geometry collision box size=0.5 0.5 0.5; visual box size=0.5 0.5 0.5
- link 011: geometry collision box size=0.5 0.5 0.5; visual box size=0.5 0.5 0.5
- link 012: geometry collision box size=0.5 0.5 0.5; visual box size=0.5 0.5 0.5
- link 020: geometry collision box size=0.5 0.5 0.5; visual box size=0.5 0.5 0.5
- link 022: geometry collision box size=0.5 0.5 0.5; visual box size=0.5 0.5 0.5
- link 031: geometry collision box size=0.5 0.5 0.5; visual box size=0.5 0.5 0.5
- link 100: geometry collision box size=0.5 0.5 0.5; visual box size=0.5 0.5 0.5
- link 111: geometry collision box size=0.5 0.5 0.5; visual box size=0.5 0.5 0.5
- link 121: geometry collision box size=0.5 0.5 0.5; visual box size=0.5 0.5 0.5
- link 222: geometry collision box size=0.5 0.5 0.5; visual box size=0.5 0.5 0.5
- link 230: geometry collision box size=0.5 0.5 0.5; visual box size=0.5 0.5 0.5
Joints:
- removed joint 001_002
- removed joint 001_010
- removed joint 001_011
- removed joint 002_102
- removed joint 010_020
- removed joint 010_100
- removed joint 010_120
- removed joint 011_022
- removed joint 020_031
- removed joint 031_121
- removed joint 100_200
- removed joint 111_212
- removed joint 120_220
- removed joint 120_230
- removed joint 121_132
- removed joint 212_222
- removed joint 222_231
- added joint 000_011: type revolute, parent 000, child 011, origin xyz=0.0 0.25 0.5 rpy=0 0 0, axis 1 0 0, limit lower=-3.14159 upper=3.14159 effort=0.0 velocity=0.0
- added joint 000_100: type revolute, parent 000, child 100, origin xyz=0.25 -0.25 0.25 rpy=0 0 0, axis 0 0 1, limit lower=-3.14159 upper=3.14159 effort=0.0 velocity=0.0
- added joint 011_020: type continuous, parent 011, child 020, origin xyz=0.0 0.5 0.0 rpy=0 0 0, axis 1 0 0, limit lower=-3.14159 upper=3.14159 effort=0.0 velocity=0.0
- added joint 011_110: type revolute, parent 011, child 110, origin xyz=0.25 0.25 0.0 rpy=0 0 0, axis 0 1 0, limit lower=-3.14159 upper=3.14159 effort=0.0 velocity=0.0
- added joint 011_121: type continuous, parent 011, child 121, origin xyz=0.25 0.5 0.25 rpy=0 0 0, axis 0 0 1, limit lower=-3.14159 upper=3.14159 effort=0.0 velocity=0.0
- added joint 012_002: type revolute, parent 012, child 002, origin xyz=0.0 0.0 0.5 rpy=0 0 0, axis 1 0 0, limit lower=-3.14159 upper=3.14159 effort=0.0 velocity=0.0
- added joint 012_022: type revolute, parent 012, child 022, origin xyz=0.25 0.5 0.25 rpy=0 0 0, axis 0 0 1, limit lower=-3.14159 upper=3.14159 effort=0.0 velocity=0.0
- added joint 020_030: type continuous, parent 020, child 030, origin xyz=0.25 0.5 -0.25 rpy=0 0 0, axis 0 0 1, limit lower=-3.14159 upper=3.14159 effort=0.0 velocity=0.0
- added joint 022_031: type continuous, parent 022, child 031, origin xyz=-0.25 0.5 -0.25 rpy=0 0 0, axis 1 0 0, limit lower=-3.14159 upper=3.14159 effort=0.0 velocity=0.0
- added joint 031_032: type revolute, parent 031, child 032, origin xyz=0.0 0.0 0.0 rpy=0 0 0, axis 1 0 0, limit lower=-3.14159 upper=3.14159 effort=0.0 velocity=0.0
- added joint 031_130: type revolute, parent 031, child 130, origin xyz=0.25 0.25 -0.5 rpy=0 0 0, axis 0 1 0, limit lower=-3.14159 upper=3.14159 effort=0.0 velocity=0.0
- added joint 100_201: type continuous, parent 100, child 201, origin xyz=0.5 0.25 0.25 rpy=0 0 0, axis 0 1 0, limit lower=-3.14159 upper=3.14159 effort=0.0 velocity=0.0
- added joint 110_210: type revolute, parent 110, child 210, origin xyz=0.5 0.25 -0.25 rpy=0 0 0, axis 0 0 1, limit lower=-3.14159 upper=3.14159 effort=0.0 velocity=0.0
- added joint 111_122: type continuous, parent 111, child 122, origin xyz=0.0 0.5 0.5 rpy=0 0 0, axis 1 0 0, limit lower=-3.14159 upper=3.14159 effort=0.0 velocity=0.0
- added joint 121_222: type revolute, parent 121, child 222, origin xyz=0.5 0.25 0.25 rpy=0 0 0, axis 0 1 0, limit lower=-3.14159 upper=3.14159 effort=0.0 velocity=0.0
- added joint 122_221: type continuous, parent 122, child 221, origin xyz=0.25 0.25 0.0 rpy=0 0 0, axis 0 1 0, limit lower=-3.14159 upper=3.14159 effort=0.0 velocity=0.0
- added joint 122_232: type revolute, parent 122, child 232, origin xyz=0.25 0.5 0.25 rpy=0 0 0, axis 0 0 1, limit lower=-3.14159 upper=3.14159 effort=0.0 velocity=0.0
- added joint 130_230: type continuous, parent 130, child 230, origin xyz=0.5 0.0 -0.5 rpy=0 0 0, axis 0 1 0, limit lower=-3.14159 upper=3.14159 effort=0.0 velocity=0.0
- joint 011_012: axis 0 1 0 -> 1 0 0; origin xyz=0.0 0.25 0.30000000000000004 rpy=0 0 0 -> xyz=0.0 0.0 0.5 rpy=0 0 0
- joint 100_111: origin xyz=0.25 0.0 0.30000000000000004 rpy=0 0 0 -> xyz=0.25 0.5 0.25 rpy=0 0 0; type continuous -> revolute
