Commit message: assignment 7 fixed

File: body0.urdf (robot description, URDF)
Before this commit: robot robot, 7 links, 6 joints
Links:
- removed link 000
- removed link 100
- removed link 200
- removed link 201
- added link 010, mass 1; collision box size=0.5 0.5 0.5; visual box size=0.5 0.5 0.5
- added link 011, mass 1; collision box size=0.5 0.5 0.5; visual box size=0.5 0.5 0.5
- added link 101, mass 1; collision box size=0.5 0.5 0.5; visual box size=0.5 0.5 0.5
Joints:
- removed joint 000_001
- removed joint 000_110
- removed joint 001_100
- removed joint 001_111
- removed joint 110_200
- removed joint 200_201
- added joint 001_010: type revolute, parent 001, child 010, origin xyz=0.0 0.25 0.5 rpy=0 0 0, axis 1 0 0, limit lower=-3.14159 upper=3.14159 effort=0.0 velocity=0.0
- added joint 001_011: type revolute, parent 001, child 011, origin xyz=0.0 0.25 0.75 rpy=0 0 0, axis 1 0 0, limit lower=-3.14159 upper=3.14159 effort=0.0 velocity=0.0
- added joint 011_101: type revolute, parent 011, child 101, origin xyz=0.25 0.0 0.0 rpy=0 0 0, axis 0 0 1, limit lower=-3.14159 upper=3.14159 effort=0.0 velocity=0.0
- added joint 011_110: type revolute, parent 011, child 110, origin xyz=0.25 0.25 -0.25 rpy=0 0 0, axis 0 1 0, limit lower=-3.14159 upper=3.14159 effort=0.0 velocity=0.0
- added joint 110_111: type revolute, parent 110, child 111, origin xyz=0.25 0.0 0.0 rpy=0 0 0, axis 1 0 0, limit lower=-3.14159 upper=3.14159 effort=0.0 velocity=0.0

Commit message: mutate weights, add remove links, add remove sensors

File: body0.urdf (robot description, URDF)
Before this commit: robot robot, 6 links, 5 joints
Links:
- removed link 000
- removed link 100
- removed link 111
- removed link 201
- added link 020, mass 1; collision box size=0.5 0.5 0.5; visual box size=0.5 0.5 0.5
- added link 021, mass 1; collision box size=0.5 0.5 0.5; visual box size=0.5 0.5 0.5
- added link 121, mass 1; collision box size=0.5 0.5 0.5; visual box size=0.5 0.5 0.5
- added link 200, mass 1; collision box size=0.5 0.5 0.5; visual box size=0.5 0.5 0.5
- added link 210, mass 1; collision box size=0.5 0.5 0.5; visual box size=0.5 0.5 0.5
Joints:
- removed joint 000_011
- removed joint 000_100
- removed joint 100_110
- removed joint 110_111
- removed joint 111_201
- added joint 011_020: type continuous, parent 011, child 020, origin xyz=0.0 0.75 0.5 rpy=0 0 0, axis 1 0 0, limit lower=-3.14159 upper=3.14159 effort=0.0 velocity=0.0
- added joint 020_021: type continuous, parent 020, child 021, origin xyz=0.25 0.25 0.0 rpy=0 0 0, axis 0 1 0, limit lower=-3.14159 upper=3.14159 effort=0.0 velocity=0.0
- added joint 020_110: type revolute, parent 020, child 110, origin xyz=0.25 0.0 -0.25 rpy=0 0 0, axis 0 0 1, limit lower=-3.14159 upper=3.14159 effort=0.0 velocity=0.0
- added joint 110_121: type continuous, parent 110, child 121, origin xyz=0.25 0.0 0.25 rpy=0 0 0, axis 1 0 0, limit lower=-3.14159 upper=3.14159 effort=0.0 velocity=0.0
- added joint 110_200: type revolute, parent 110, child 200, origin xyz=0.5 -0.5 0.0 rpy=0 0 0, axis 0 0 1, limit lower=-3.14159 upper=3.14159 effort=0.0 velocity=0.0
- added joint 200_210: type continuous, parent 200, child 210, origin xyz=0.25 0.0 0.0 rpy=0 0 0, axis 0 0 1, limit lower=-3.14159 upper=3.14159 effort=0.0 velocity=0.0
