Commit message: debugging

File: body0.urdf (robot description, URDF)
Before this commit: robot robot, 20 links, 19 joints
Links:
- removed link 001
- removed link 002
- removed link 010
- removed link 012
- removed link 102
- removed link 120
- removed link 200
- removed link 222
- removed link 231
- added link 000, mass 1; collision box size=0.5 0.7000000000000001 0.7000000000000001; visual box size=0.5 0.7000000000000001 0.7000000000000001
- added link 021, mass 1; collision box size=0.5 0.7000000000000001 0.7000000000000001; visual box size=0.5 0.7000000000000001 0.7000000000000001
- added link 030, mass 1; collision box size=0.5 0.7000000000000001 0.7000000000000001; visual box size=0.5 0.7000000000000001 0.7000000000000001
- added link 032, mass 1; collision box size=0.5 0.7000000000000001 0.7000000000000001; visual box size=0.5 0.7000000000000001 0.7000000000000001
- added link 110, mass 1; collision box size=0.5 0.7000000000000001 0.7000000000000001; visual box size=0.5 0.7000000000000001 0.7000000000000001
- added link 122, mass 1; collision box size=0.5 0.7000000000000001 0.7000000000000001; visual box size=0.5 0.7000000000000001 0.7000000000000001
- added link 130, mass 1; collision box size=0.5 0.7000000000000001 0.7000000000000001; visual box size=0.5 0.7000000000000001 0.7000000000000001
- added link 131, mass 1; collision box size=0.5 0.7000000000000001 0.7000000000000001; visual box size=0.5 0.7000000000000001 0.7000000000000001
- added link 202, mass 1; collision box size=0.5 0.7000000000000001 0.7000000000000001; visual box size=0.5 0.7000000000000001 0.7000000000000001
- added link 221, mass 1; collision box size=0.5 0.7000000000000001 0.7000000000000001; visual box size=0.5 0.7000000000000001 0.7000000000000001
- link 011: geometry collision box size=0.5 0.7000000000000001 0.7000000000000001; visual box size=0.5 0.7000000000000001 0.7000000000000001
- link 020: geometry collision box size=0.5 0.7000000000000001 0.7000000000000001; visual box size=0.5 0.7000000000000001 0.7000000000000001
- link 022: geometry collision box size=0.5 0.7000000000000001 0.7000000000000001; visual box size=0.5 0.7000000000000001 0.7000000000000001
- link 031: geometry collision box size=0.5 0.7000000000000001 0.7000000000000001; visual box size=0.5 0.7000000000000001 0.7000000000000001
- link 100: geometry collision box size=0.5 0.7000000000000001 0.7000000000000001; visual box size=0.5 0.7000000000000001 0.7000000000000001
- link 111: geometry collision box size=0.5 0.7000000000000001 0.7000000000000001; visual box size=0.5 0.7000000000000001 0.7000000000000001
- link 121: geometry collision box size=0.5 0.7000000000000001 0.7000000000000001; visual box size=0.5 0.7000000000000001 0.7000000000000001
- link 132: geometry collision box size=0.5 0.7000000000000001 0.7000000000000001; visual box size=0.5 0.7000000000000001 0.7000000000000001
- link 212: geometry collision box size=0.5 0.7000000000000001 0.7000000000000001; visual box size=0.5 0.7000000000000001 0.7000000000000001
- link 220: geometry collision box size=0.5 0.7000000000000001 0.7000000000000001; visual box size=0.5 0.7000000000000001 0.7000000000000001
- link 230: geometry collision box size=0.5 0.7000000000000001 0.7000000000000001; visual box size=0.5 0.7000000000000001 0.7000000000000001
Joints:
- removed joint 001_002
- removed joint 001_010
- removed joint 001_011
- removed joint 002_102
- removed joint 010_020
- removed joint 010_100
- removed joint 010_120
- removed joint 011_012
- removed joint 011_022
- removed joint 031_121
- removed joint 100_200
- removed joint 120_220
- removed joint 120_230
- removed joint 121_132
- removed joint 212_222
- removed joint 222_231
- added joint 000_011: type revolute, parent 000, child 011, origin xyz=0.0 0.35000000000000003 0.7000000000000001 rpy=0 0 0, axis 1 0 0, limit lower=-3.14159 upper=3.14159 effort=0.0 velocity=0.0
- added joint 000_100: type continuous, parent 000, child 100, origin xyz=0.25 0.0 0.35000000000000003 rpy=0 0 0, axis 0 0 1, limit lower=-3.14159 upper=3.14159 effort=0.0 velocity=0.0
- added joint 000_110: type revolute, parent 000, child 110, origin xyz=0.25 0.35000000000000003 0.35000000000000003 rpy=0 0 0, axis 0 0 1, limit lower=-3.14159 upper=3.14159 effort=0.0 velocity=0.0
- added joint 011_020: type revolute, parent 011, child 020, origin xyz=0.0 0.7 0.0 rpy=0 0 0, axis 1 0 0, limit lower=-3.14159 upper=3.14159 effort=0.0 velocity=0.0
- added joint 011_021: type continuous, parent 011, child 021, origin xyz=0.0 0.7 -1.1102230246251565e-16 rpy=0 0 0, axis 1 0 0, limit lower=-3.14159 upper=3.14159 effort=0.0 velocity=0.0
- added joint 020_030: type continuous, parent 020, child 030, origin xyz=0.0 0.7 -0.7000000000000001 rpy=0 0 0, axis 1 0 0, limit lower=-3.14159 upper=3.14159 effort=0.0 velocity=0.0
- added joint 020_121: type revolute, parent 020, child 121, origin xyz=0.25 0.3500000000000001 -1.1102230246251565e-16 rpy=0 0 0, axis 0 1 0, limit lower=-3.14159 upper=3.14159 effort=0.0 velocity=0.0
- added joint 020_130: type continuous, parent 020, child 130, origin xyz=0.25 0.7 -0.35000000000000003 rpy=0 0 0, axis 0 0 1, limit lower=-3.14159 upper=3.14159 effort=0.0 velocity=0.0
- added joint 021_022: type continuous, parent 021, child 022, origin xyz=-0.25 0.3500000000000001 0.7000000000000002 rpy=0 0 0, axis 0 1 0, limit lower=-3.14159 upper=3.14159 effort=0.0 velocity=0.0
- added joint 021_122: type revolute, parent 021, child 122, origin xyz=0.25 0.3500000000000001 0.7000000000000002 rpy=0 0 0, axis 0 1 0, limit lower=-3.14159 upper=3.14159 effort=0.0 velocity=0.0
- added joint 031_032: type continuous, parent 031, child 032, origin xyz=0.0 0.3500000000000001 0.7000000000000002 rpy=0 0 0, axis 0 1 0, limit lower=-3.14159 upper=3.14159 effort=0.0 velocity=0.0
- added joint 031_132: type revolute, parent 031, child 132, origin xyz=0.25 0.3500000000000001 0.7000000000000002 rpy=0 0 0, axis 0 1 0, limit lower=-3.14159 upper=3.14159 effort=0.0 velocity=0.0
- added joint 111_221: type revolute, parent 111, child 221, origin xyz=0.25 0.7 0.3500000000000001 rpy=0 0 0, axis 0 0 1, limit lower=-3.14159 upper=3.14159 effort=0.0 velocity=0.0
- added joint 130_220: type continuous, parent 130, child 220, origin xyz=0.5 2.220446049250313e-16 0.0 rpy=0 0 0, axis 0 0 1, limit lower=-3.14159 upper=3.14159 effort=0.0 velocity=0.0
- added joint 132_131: type continuous, parent 132, child 131, origin xyz=0.0 0.0 0.0 rpy=0 0 0, axis 0 1 0, limit lower=-3.14159 upper=3.14159 effort=0.0 velocity=0.0
- added joint 212_202: type revolute, parent 212, child 202, origin xyz=0.25 -0.35000000000000003 0.0 rpy=0 0 0, axis 1 0 0, limit lower=-3.14159 upper=3.14159 effort=0.0 velocity=0.0
- added joint 221_230: type revolute, parent 221, child 230, origin xyz=0.25 0.7 -0.35 rpy=0 0 0, axis 1 0 0, limit lower=-3.14159 upper=3.14159 effort=0.0 velocity=0.0
- joint 020_031: origin xyz=0.0 0.5 0.30000000000000004 rpy=0 0 0 -> xyz=0.0 0.7 -1.1102230246251565e-16 rpy=0 0 0; type continuous -> revolute
- joint 100_111: origin xyz=0.25 0.0 0.30000000000000004 rpy=0 0 0 -> xyz=0.25 0.35000000000000003 0.3499999999999999 rpy=0 0 0
- joint 111_212: origin xyz=0.25 0.25 0.6000000000000001 rpy=0 0 0 -> xyz=0.25 0.35000000000000003 0.7000000000000002 rpy=0 0 0; type continuous -> revolute

File: body1.urdf (robot description, URDF)
Before this commit: robot robot, 23 links, 22 joints
Links:
- removed link 002
- removed link 010
- removed link 011
- removed link 030
- removed link 032
- removed link 111
- removed link 112
- removed link 200
- removed link 201
- removed link 211
- removed link 222
- added link 000, mass 1; collision box size=0.30000000000000004 0.5 0.5; visual box size=0.30000000000000004 0.5 0.5
- added link 102, mass 1; collision box size=0.30000000000000004 0.5 0.5; visual box size=0.30000000000000004 0.5 0.5
- added link 122, mass 1; collision box size=0.30000000000000004 0.5 0.5; visual box size=0.30000000000000004 0.5 0.5
- added link 232, mass 1; collision box size=0.30000000000000004 0.5 0.5; visual box size=0.30000000000000004 0.5 0.5
- link 001: geometry collision box size=0.30000000000000004 0.5 0.5; visual box size=0.30000000000000004 0.5 0.5
- link 012: geometry collision box size=0.30000000000000004 0.5 0.5; visual box size=0.30000000000000004 0.5 0.5
- link 020: geometry collision box size=0.30000000000000004 0.5 0.5; visual box size=0.30000000000000004 0.5 0.5
- link 022: geometry collision box size=0.30000000000000004 0.5 0.5; visual box size=0.30000000000000004 0.5 0.5
- link 101: geometry collision box size=0.30000000000000004 0.5 0.5; visual box size=0.30000000000000004 0.5 0.5
- link 121: geometry collision box size=0.30000000000000004 0.5 0.5; visual box size=0.30000000000000004 0.5 0.5
- link 130: geometry collision box size=0.30000000000000004 0.5 0.5; visual box size=0.30000000000000004 0.5 0.5
- link 132: geometry collision box size=0.30000000000000004 0.5 0.5; visual box size=0.30000000000000004 0.5 0.5
- link 202: geometry collision box size=0.30000000000000004 0.5 0.5; visual box size=0.30000000000000004 0.5 0.5
- link 212: geometry collision box size=0.30000000000000004 0.5 0.5; visual box size=0.30000000000000004 0.5 0.5
- link 221: geometry collision box size=0.30000000000000004 0.5 0.5; visual box size=0.30000000000000004 0.5 0.5
- link 231: geometry collision box size=0.30000000000000004 0.5 0.5; visual box size=0.30000000000000004 0.5 0.5
Joints:
- removed joint 002_011
- removed joint 002_012
- removed joint 002_101
- removed joint 011_020
- removed joint 011_022
- removed joint 012_111
- removed joint 020_010
- removed joint 020_030
- removed joint 020_121
- removed joint 020_130
- removed joint 022_032
- removed joint 022_132
- removed joint 101_001
- removed joint 101_112
- removed joint 101_200
- removed joint 101_202
- removed joint 111_201
- removed joint 132_222
- removed joint 201_211
- removed joint 211_212
- removed joint 211_221
- removed joint 222_231
- added joint 000_001: type revolute, parent 000, child 001, origin xyz=0.15000000000000002 0.0 0.5 rpy=0 0 0, axis 0 1 0, limit lower=-3.14159 upper=3.14159 effort=0.0 velocity=0.0
- added joint 001_101: type revolute, parent 001, child 101, origin xyz=0.0 -0.25 0.25 rpy=0 0 0, axis 0 0 1, limit lower=-3.14159 upper=3.14159 effort=0.0 velocity=0.0
- added joint 001_102: type continuous, parent 001, child 102, origin xyz=0.0 0.0 0.5 rpy=0 0 0, axis 0 1 0, limit lower=-3.14159 upper=3.14159 effort=0.0 velocity=0.0
- added joint 102_012: type continuous, parent 102, child 012, origin xyz=0.0 0.25 0.25 rpy=0 0 0, axis 0 0 1, limit lower=-3.14159 upper=3.14159 effort=0.0 velocity=0.0
- added joint 102_202: type revolute, parent 102, child 202, origin xyz=0.30000000000000004 -0.25 0.25 rpy=0 0 0, axis 0 0 1, limit lower=-3.14159 upper=3.14159 effort=0.0 velocity=0.0
- added joint 121_022: type continuous, parent 121, child 022, origin xyz=-0.30000000000000004 -0.25 0.25 rpy=0 0 0, axis 0 1 0, limit lower=-3.14159 upper=3.14159 effort=0.0 velocity=0.0
- added joint 121_122: type revolute, parent 121, child 122, origin xyz=-0.15000000000000002 -0.5 0.25 rpy=0 0 0, axis 1 0 0, limit lower=-3.14159 upper=3.14159 effort=0.0 velocity=0.0
- added joint 121_130: type continuous, parent 121, child 130, origin xyz=-0.15000000000000002 0.0 -0.25 rpy=0 0 0, axis 1 0 0, limit lower=-3.14159 upper=3.14159 effort=0.0 velocity=0.0
- added joint 121_132: type continuous, parent 121, child 132, origin xyz=-0.15000000000000002 0.0 0.25 rpy=0 0 0, axis 1 0 0, limit lower=-3.14159 upper=3.14159 effort=0.0 velocity=0.0
- added joint 121_231: type continuous, parent 121, child 231, origin xyz=0.0 0.0 0.0 rpy=0 0 0, axis 0 0 1, limit lower=-3.14159 upper=3.14159 effort=0.0 velocity=0.0
- added joint 130_020: type revolute, parent 130, child 020, origin xyz=-0.15000000000000002 0.0 -0.25 rpy=0 0 0, axis 0 0 1, limit lower=-3.14159 upper=3.14159 effort=0.0 velocity=0.0
- added joint 132_232: type continuous, parent 132, child 232, origin xyz=0.15000000000000002 0.0 0.25 rpy=0 0 0, axis 0 0 1, limit lower=-3.14159 upper=3.14159 effort=0.0 velocity=0.0
- added joint 202_212: type revolute, parent 202, child 212, origin xyz=0.15000000000000002 0.5 0.25 rpy=0 0 0, axis 1 0 0, limit lower=-3.14159 upper=3.14159 effort=0.0 velocity=0.0
- added joint 212_221: type revolute, parent 212, child 221, origin xyz=0.0 0.5 -0.5 rpy=0 0 0, axis 1 0 0, limit lower=-3.14159 upper=3.14159 effort=0.0 velocity=0.0
- added joint 221_121: type revolute, parent 221, child 121, origin xyz=-0.15000000000000002 0.5 -0.25 rpy=0 0 0, axis 0 0 1, limit lower=-3.14159 upper=3.14159 effort=0.0 velocity=0.0

File: body2.urdf (robot description, URDF)
Before this commit: robot robot, 13 links, 12 joints
Links:
- removed link 000
- removed link 002
- removed link 101
- removed link 201
- removed link 220
- added link 031, mass 1; collision box size=0.2 0.8 0.7000000000000001; visual box size=0.2 0.8 0.7000000000000001
- added link 102, mass 1; collision box size=0.2 0.8 0.7000000000000001; visual box size=0.2 0.8 0.7000000000000001
- added link 110, mass 1; collision box size=0.2 0.8 0.7000000000000001; visual box size=0.2 0.8 0.7000000000000001
- added link 111, mass 1; collision box size=0.2 0.8 0.7000000000000001; visual box size=0.2 0.8 0.7000000000000001
- added link 121, mass 1; collision box size=0.2 0.8 0.7000000000000001; visual box size=0.2 0.8 0.7000000000000001
- added link 130, mass 1; collision box size=0.2 0.8 0.7000000000000001; visual box size=0.2 0.8 0.7000000000000001
- added link 132, mass 1; collision box size=0.2 0.8 0.7000000000000001; visual box size=0.2 0.8 0.7000000000000001
- added link 200, mass 1; collision box size=0.2 0.8 0.7000000000000001; visual box size=0.2 0.8 0.7000000000000001
- added link 212, mass 1; collision box size=0.2 0.8 0.7000000000000001; visual box size=0.2 0.8 0.7000000000000001
- added link 222, mass 1; collision box size=0.2 0.8 0.7000000000000001; visual box size=0.2 0.8 0.7000000000000001
- added link 230, mass 1; collision box size=0.2 0.8 0.7000000000000001; visual box size=0.2 0.8 0.7000000000000001
- added link 231, mass 1; collision box size=0.2 0.8 0.7000000000000001; visual box size=0.2 0.8 0.7000000000000001
- link 010: geometry collision box size=0.2 0.8 0.7000000000000001; visual box size=0.2 0.8 0.7000000000000001
- link 020: geometry collision box size=0.2 0.8 0.7000000000000001; visual box size=0.2 0.8 0.7000000000000001
- link 100: geometry collision box size=0.2 0.8 0.7000000000000001; visual box size=0.2 0.8 0.7000000000000001
- link 112: geometry collision box size=0.2 0.8 0.7000000000000001; visual box size=0.2 0.8 0.7000000000000001
- link 131: geometry collision box size=0.2 0.8 0.7000000000000001; visual box size=0.2 0.8 0.7000000000000001
- link 202: geometry collision box size=0.2 0.8 0.7000000000000001; visual box size=0.2 0.8 0.7000000000000001
- link 210: geometry collision box size=0.2 0.8 0.7000000000000001; visual box size=0.2 0.8 0.7000000000000001
- link 221: geometry collision box size=0.2 0.8 0.7000000000000001; visual box size=0.2 0.8 0.7000000000000001
Joints:
- removed joint 000_010
- removed joint 000_100
- removed joint 100_101
- removed joint 100_201
- removed joint 101_112
- removed joint 112_002
- removed joint 201_210
- removed joint 210_220
- removed joint 210_221
- removed joint 221_131
- added joint 010_100: type continuous, parent 010, child 100, origin xyz=0.1 0.4 0.35000000000000003 rpy=0 0 0, axis 0 0 1, limit lower=-3.14159 upper=3.14159 effort=0.0 velocity=0.0
- added joint 010_111: type continuous, parent 010, child 111, origin xyz=0.1 0.8 0.7000000000000001 rpy=0 0 0, axis 0 1 0, limit lower=-3.14159 upper=3.14159 effort=0.0 velocity=0.0
- added joint 020_031: type revolute, parent 020, child 031, origin xyz=0.0 0.8000000000000003 -1.1102230246251565e-16 rpy=0 0 0, axis 1 0 0, limit lower=-3.14159 upper=3.14159 effort=0.0 velocity=0.0
- added joint 020_110: type continuous, parent 020, child 110, origin xyz=0.1 0.0 -0.35000000000000003 rpy=0 0 0, axis 0 0 1, limit lower=-3.14159 upper=3.14159 effort=0.0 velocity=0.0
- added joint 031_131: type revolute, parent 031, child 131, origin xyz=0.1 0.3999999999999999 0.3500000000000001 rpy=0 0 0, axis 0 1 0, limit lower=-3.14159 upper=3.14159 effort=0.0 velocity=0.0
- added joint 100_200: type continuous, parent 100, child 200, origin xyz=0.20000000000000004 -0.8 0.0 rpy=0 0 0, axis 0 0 1, limit lower=-3.14159 upper=3.14159 effort=0.0 velocity=0.0
- added joint 110_121: type revolute, parent 110, child 121, origin xyz=0.1 0.0 0.3499999999999999 rpy=0 0 0, axis 1 0 0, limit lower=-3.14159 upper=3.14159 effort=0.0 velocity=0.0
- added joint 111_112: type continuous, parent 111, child 112, origin xyz=0.1 -0.4 0.7000000000000001 rpy=0 0 0, axis 1 0 0, limit lower=-3.14159 upper=3.14159 effort=0.0 velocity=0.0
- added joint 112_212: type revolute, parent 112, child 212, origin xyz=0.10000000000000003 0.4 0.7 rpy=0 0 0, axis 0 1 0, limit lower=-3.14159 upper=3.14159 effort=0.0 velocity=0.0
- added joint 121_130: type continuous, parent 121, child 130, origin xyz=0.0 0.8000000000000003 1.1102230246251565e-16 rpy=0 0 0, axis 1 0 0, limit lower=-3.14159 upper=3.14159 effort=0.0 velocity=0.0
- added joint 121_132: type revolute, parent 121, child 132, origin xyz=0.0 0.8000000000000003 0.7000000000000002 rpy=0 0 0, axis 1 0 0, limit lower=-3.14159 upper=3.14159 effort=0.0 velocity=0.0
- added joint 131_230: type continuous, parent 131, child 230, origin xyz=0.20000000000000004 0.0 -0.35 rpy=0 0 0, axis 0 1 0, limit lower=-3.14159 upper=3.14159 effort=0.0 velocity=0.0
- added joint 200_210: type revolute, parent 200, child 210, origin xyz=0.0 0.8 0.0 rpy=0 0 0, axis 0 0 1, limit lower=-3.14159 upper=3.14159 effort=0.0 velocity=0.0
- added joint 202_102: type revolute, parent 202, child 102, origin xyz=0.0 -0.4 0.0 rpy=0 0 0, axis 0 1 0, limit lower=-3.14159 upper=3.14159 effort=0.0 velocity=0.0
- added joint 212_221: type revolute, parent 212, child 221, origin xyz=0.09999999999999998 0.40000000000000013 -0.7 rpy=0 0 0, axis 1 0 0, limit lower=-3.14159 upper=3.14159 effort=0.0 velocity=0.0
- added joint 221_222: type continuous, parent 221, child 222, origin xyz=0.0 0.3999999999999999 0.0 rpy=0 0 0, axis 1 0 0, limit lower=-3.14159 upper=3.14159 effort=0.0 velocity=0.0
- added joint 222_231: type revolute, parent 222, child 231, origin xyz=0.0 0.40000000000000036 0.0 rpy=0 0 0, axis 1 0 0, limit lower=-3.14159 upper=3.14159 effort=0.0 velocity=0.0
- joint 010_020: origin xyz=-0.25 0.5 0.25 rpy=0 0 0 -> xyz=0.0 1.2000000000000002 0.7000000000000001 rpy=0 0 0
- joint 112_202: origin xyz=0.25 0.0 0.25 rpy=0 0 0 -> xyz=0.10000000000000003 0.0 0.3500000000000001 rpy=0 0 0

File: body3.urdf (robot description, URDF)
Before this commit: robot robot, 21 links, 20 joints
Links:
- removed link 000
- removed link 011
- removed link 012
- removed link 020
- removed link 022
- removed link 030
- removed link 032
- removed link 100
- removed link 110
- removed link 121
- removed link 122
- removed link 130
- removed link 210
- removed link 232
- added link 001, mass 1; collision box size=0.5 0.5 0.5; visual box size=0.5 0.5 0.5
- added link 021, mass 1; collision box size=0.5 0.5 0.5; visual box size=0.5 0.5 0.5
- added link 101, mass 1; collision box size=0.5 0.5 0.5; visual box size=0.5 0.5 0.5
- added link 120, mass 1; collision box size=0.5 0.5 0.5; visual box size=0.5 0.5 0.5
- added link 131, mass 1; collision box size=0.5 0.5 0.5; visual box size=0.5 0.5 0.5
- added link 132, mass 1; collision box size=0.5 0.5 0.5; visual box size=0.5 0.5 0.5
- added link 212, mass 1; collision box size=0.5 0.5 0.5; visual box size=0.5 0.5 0.5
- added link 231, mass 1; collision box size=0.5 0.5 0.5; visual box size=0.5 0.5 0.5
Joints:
- removed joint 000_011
- removed joint 000_100
- removed joint 011_012
- removed joint 011_020
- removed joint 011_110
- removed joint 011_121
- removed joint 012_002
- removed joint 012_022
- removed joint 020_030
- removed joint 022_031
- removed joint 031_032
- removed joint 031_130
- removed joint 100_111
- removed joint 100_201
- removed joint 110_210
- removed joint 111_122
- removed joint 121_222
- removed joint 122_221
- removed joint 122_232
- removed joint 130_230
- added joint 001_002: type revolute, parent 001, child 002, origin xyz=0.0 -0.25 1.0 rpy=0 0 0, axis 1 0 0, limit lower=-3.14159 upper=3.14159 effort=0.0 velocity=0.0
- added joint 002_101: type continuous, parent 002, child 101, origin xyz=0.25 0.25 0.0 rpy=0 0 0, axis 0 1 0, limit lower=-3.14159 upper=3.14159 effort=0.0 velocity=0.0
- added joint 021_031: type revolute, parent 021, child 031, origin xyz=0.0 0.25 0.25 rpy=0 0 0, axis 0 0 1, limit lower=-3.14159 upper=3.14159 effort=0.0 velocity=0.0
- added joint 101_201: type revolute, parent 101, child 201, origin xyz=0.5 0.25 -0.25 rpy=0 0 0, axis 0 0 1, limit lower=-3.14159 upper=3.14159 effort=0.0 velocity=0.0
- added joint 120_021: type continuous, parent 120, child 021, origin xyz=-0.5 0.0 0.0 rpy=0 0 0, axis 0 1 0, limit lower=-3.14159 upper=3.14159 effort=0.0 velocity=0.0
- added joint 120_111: type revolute, parent 120, child 111, origin xyz=-0.25 -0.25 0.0 rpy=0 0 0, axis 1 0 0, limit lower=-3.14159 upper=3.14159 effort=0.0 velocity=0.0
- added joint 131_132: type continuous, parent 131, child 132, origin xyz=-0.5 0.0 0.5 rpy=0 0 0, axis 0 1 0, limit lower=-3.14159 upper=3.14159 effort=0.0 velocity=0.0
- added joint 201_212: type revolute, parent 201, child 212, origin xyz=0.25 0.0 0.25 rpy=0 0 0, axis 1 0 0, limit lower=-3.14159 upper=3.14159 effort=0.0 velocity=0.0
- added joint 212_221: type continuous, parent 212, child 221, origin xyz=0.0 0.5 0.0 rpy=0 0 0, axis 1 0 0, limit lower=-3.14159 upper=3.14159 effort=0.0 velocity=0.0
- added joint 221_120: type continuous, parent 221, child 120, origin xyz=-0.25 0.25 -0.5 rpy=0 0 0, axis 0 1 0, limit lower=-3.14159 upper=3.14159 effort=0.0 velocity=0.0
- added joint 221_222: type continuous, parent 221, child 222, origin xyz=0.0 0.0 0.0 rpy=0 0 0, axis 1 0 0, limit lower=-3.14159 upper=3.14159 effort=0.0 velocity=0.0
- added joint 221_230: type revolute, parent 221, child 230, origin xyz=0.0 0.5 -0.5 rpy=0 0 0, axis 1 0 0, limit lower=-3.14159 upper=3.14159 effort=0.0 velocity=0.0
- added joint 222_231: type revolute, parent 222, child 231, origin xyz=0.0 0.5 0.0 rpy=0 0 0, axis 1 0 0, limit lower=-3.14159 upper=3.14159 effort=0.0 velocity=0.0
- added joint 230_131: type continuous, parent 230, child 131, origin xyz=-0.25 0.25 0.0 rpy=0 0 0, axis 0 1 0, limit lower=-3.14159 upper=3.14159 effort=0.0 velocity=0.0
