Commit message: debugging

File: body4.urdf (robot description, URDF)
Before this commit: robot robot, 14 links, 13 joints
Links:
- removed link 010
- removed link 110
- removed link 121
- removed link 202
- removed link 221
- added link 001, mass 1; collision box size=0.5 0.4 0.5; visual box size=0.5 0.4 0.5
- added link 012, mass 1; collision box size=0.5 0.4 0.5; visual box size=0.5 0.4 0.5
- added link 022, mass 1; collision box size=0.5 0.4 0.5; visual box size=0.5 0.4 0.5
- added link 031, mass 1; collision box size=0.5 0.4 0.5; visual box size=0.5 0.4 0.5
- added link 100, mass 1; collision box size=0.5 0.4 0.5; visual box size=0.5 0.4 0.5
- added link 102, mass 1; collision box size=0.5 0.4 0.5; visual box size=0.5 0.4 0.5
- added link 111, mass 1; collision box size=0.5 0.4 0.5; visual box size=0.5 0.4 0.5
- added link 112, mass 1; collision box size=0.5 0.4 0.5; visual box size=0.5 0.4 0.5
- added link 200, mass 1; collision box size=0.5 0.4 0.5; visual box size=0.5 0.4 0.5
- added link 211, mass 1; collision box size=0.5 0.4 0.5; visual box size=0.5 0.4 0.5
- added link 220, mass 1; collision box size=0.5 0.4 0.5; visual box size=0.5 0.4 0.5
- added link 230, mass 1; collision box size=0.5 0.4 0.5; visual box size=0.5 0.4 0.5
- added link 232, mass 1; collision box size=0.5 0.4 0.5; visual box size=0.5 0.4 0.5
- link 000: geometry collision box size=0.5 0.4 0.5; visual box size=0.5 0.4 0.5
- link 011: geometry collision box size=0.5 0.4 0.5; visual box size=0.5 0.4 0.5
- link 020: geometry collision box size=0.5 0.4 0.5; visual box size=0.5 0.4 0.5
- link 021: geometry collision box size=0.5 0.4 0.5; visual box size=0.5 0.4 0.5
- link 030: geometry collision box size=0.5 0.4 0.5; visual box size=0.5 0.4 0.5
- link 101: geometry collision box size=0.5 0.4 0.5; visual box size=0.5 0.4 0.5
- link 120: geometry collision box size=0.5 0.4 0.5; visual box size=0.5 0.4 0.5
- link 131: geometry collision box size=0.5 0.4 0.5; visual box size=0.5 0.4 0.5
- link 210: geometry collision box size=0.5 0.4 0.5; visual box size=0.5 0.4 0.5
Joints:
- removed joint 000_010
- removed joint 010_020
- removed joint 011_021
- removed joint 011_121
- removed joint 021_030
- removed joint 101_110
- removed joint 101_202
- removed joint 120_210
- removed joint 121_131
- removed joint 210_221
- added joint 000_001: type revolute, parent 000, child 001, origin xyz=0.0 0.0 0.5 rpy=0 0 0, axis 0 1 0, limit lower=-3.14159 upper=3.14159 effort=0.0 velocity=0.0
- added joint 000_100: type continuous, parent 000, child 100, origin xyz=0.25 -0.2 0.25 rpy=0 0 0, axis 0 0 1, limit lower=-3.14159 upper=3.14159 effort=0.0 velocity=0.0
- added joint 011_012: type continuous, parent 011, child 012, origin xyz=-0.25 0.2 0.5 rpy=0 0 0, axis 0 1 0, limit lower=-3.14159 upper=3.14159 effort=0.0 velocity=0.0
- added joint 011_020: type revolute, parent 011, child 020, origin xyz=0.0 0.4000000000000001 0.0 rpy=0 0 0, axis 1 0 0, limit lower=-3.14159 upper=3.14159 effort=0.0 velocity=0.0
- added joint 012_112: type continuous, parent 012, child 112, origin xyz=0.5 -0.2 0.25 rpy=0 0 0, axis 0 0 1, limit lower=-3.14159 upper=3.14159 effort=0.0 velocity=0.0
- added joint 020_021: type revolute, parent 020, child 021, origin xyz=0.25 0.19999999999999996 0.0 rpy=0 0 0, axis 0 1 0, limit lower=-3.14159 upper=3.14159 effort=0.0 velocity=0.0
- added joint 021_022: type continuous, parent 021, child 022, origin xyz=-0.25 0.0 0.5 rpy=0 0 0, axis 0 1 0, limit lower=-3.14159 upper=3.14159 effort=0.0 velocity=0.0
- added joint 021_031: type continuous, parent 021, child 031, origin xyz=-0.25 0.20000000000000018 0.0 rpy=0 0 0, axis 1 0 0, limit lower=-3.14159 upper=3.14159 effort=0.0 velocity=0.0
- added joint 031_030: type continuous, parent 031, child 030, origin xyz=0.25 0.19999999999999996 0.0 rpy=0 0 0, axis 0 1 0, limit lower=-3.14159 upper=3.14159 effort=0.0 velocity=0.0
- added joint 101_102: type revolute, parent 101, child 102, origin xyz=0.25 -0.4 0.25 rpy=0 0 0, axis 1 0 0, limit lower=-3.14159 upper=3.14159 effort=0.0 velocity=0.0
- added joint 101_200: type revolute, parent 101, child 200, origin xyz=0.5 -0.2 -0.25 rpy=0 0 0, axis 0 1 0, limit lower=-3.14159 upper=3.14159 effort=0.0 velocity=0.0
- added joint 101_211: type continuous, parent 101, child 211, origin xyz=0.5 0.0 0.0 rpy=0 0 0, axis 0 0 1, limit lower=-3.14159 upper=3.14159 effort=0.0 velocity=0.0
- added joint 102_111: type revolute, parent 102, child 111, origin xyz=0.0 0.4 0.0 rpy=0 0 0, axis 1 0 0, limit lower=-3.14159 upper=3.14159 effort=0.0 velocity=0.0
- added joint 120_131: type revolute, parent 120, child 131, origin xyz=0.25 0.20000000000000018 0.0 rpy=0 0 0, axis 1 0 0, limit lower=-3.14159 upper=3.14159 effort=0.0 velocity=0.0
- added joint 120_220: type continuous, parent 120, child 220, origin xyz=0.5 0.19999999999999996 -0.25 rpy=0 0 0, axis 0 0 1, limit lower=-3.14159 upper=3.14159 effort=0.0 velocity=0.0
- added joint 131_230: type revolute, parent 131, child 230, origin xyz=0.25 0.19999999999999996 0.0 rpy=0 0 0, axis 0 1 0, limit lower=-3.14159 upper=3.14159 effort=0.0 velocity=0.0
- added joint 131_232: type continuous, parent 131, child 232, origin xyz=0.25 0.19999999999999996 0.5 rpy=0 0 0, axis 0 1 0, limit lower=-3.14159 upper=3.14159 effort=0.0 velocity=0.0
- added joint 200_210: type revolute, parent 200, child 210, origin xyz=0.5 0.2 -0.25 rpy=0 0 0, axis 0 0 1, limit lower=-3.14159 upper=3.14159 effort=0.0 velocity=0.0
- joint 000_011: origin xyz=0.0 0.25 0.5 rpy=0 0 0 -> xyz=0.0 0.2 0.5 rpy=0 0 0; type continuous -> revolute
- joint 011_101: origin xyz=0.5 0.0 0.25 rpy=0 0 0 -> xyz=0.25 0.0 0.25 rpy=0 0 0; type revolute -> continuous
- joint 021_120: origin xyz=0.5 0.25 0.0 rpy=0 0 0 -> xyz=0.0 0.0 0.0 rpy=0 0 0

Commit message: final adjustments

File: body0.urdf (robot description, URDF)
Before this commit: robot robot, 21 links, 20 joints
Links:
- removed link 122
- removed link 131
- added link 001, mass 1; collision box size=0.5 0.5 0.5; visual box size=0.5 0.5 0.5
- link 000: geometry collision box size=0.5 0.5 0.5; visual box size=0.5 0.5 0.5
- link 011: geometry collision box size=0.5 0.5 0.5; visual box size=0.5 0.5 0.5
- link 020: geometry collision box size=0.5 0.5 0.5; visual box size=0.5 0.5 0.5
- link 021: geometry collision box size=0.5 0.5 0.5; visual box size=0.5 0.5 0.5
- link 022: geometry collision box size=0.5 0.5 0.5; visual box size=0.5 0.5 0.5
- link 030: geometry collision box size=0.5 0.5 0.5; visual box size=0.5 0.5 0.5
- link 031: geometry collision box size=0.5 0.5 0.5; visual box size=0.5 0.5 0.5
- link 032: geometry collision box size=0.5 0.5 0.5; visual box size=0.5 0.5 0.5
- link 100: geometry collision box size=0.5 0.5 0.5; visual box size=0.5 0.5 0.5
- link 110: geometry collision box size=0.5 0.5 0.5; visual box size=0.5 0.5 0.5
- link 111: geometry collision box size=0.5 0.5 0.5; visual box size=0.5 0.5 0.5
- link 121: geometry collision box size=0.5 0.5 0.5; visual box size=0.5 0.5 0.5
- link 130: geometry collision box size=0.5 0.5 0.5; visual box size=0.5 0.5 0.5
- link 132: geometry collision box size=0.5 0.5 0.5; visual box size=0.5 0.5 0.5
- link 202: geometry collision box size=0.5 0.5 0.5; visual box size=0.5 0.5 0.5
- link 212: geometry collision box size=0.5 0.5 0.5; visual box size=0.5 0.5 0.5
- link 220: geometry collision box size=0.5 0.5 0.5; visual box size=0.5 0.5 0.5
- link 221: geometry collision box size=0.5 0.5 0.5; visual box size=0.5 0.5 0.5
- link 230: geometry collision box size=0.5 0.5 0.5; visual box size=0.5 0.5 0.5
Joints:
- removed joint 021_122
- removed joint 132_131
- added joint 000_001: type continuous, parent 000, child 001, origin xyz=0.0 -0.25 0.5 rpy=0 0 0, axis 1 0 0, limit lower=-3.14159 upper=3.14159 effort=0.0 velocity=0.0
- joint 000_011: origin xyz=0.0 0.35000000000000003 0.7000000000000001 rpy=0 0 0 -> xyz=0.0 0.25 0.5 rpy=0 0 0
- joint 000_100: origin xyz=0.25 0.0 0.35000000000000003 rpy=0 0 0 -> xyz=0.25 0.0 0.25 rpy=0 0 0
- joint 000_110: origin xyz=0.25 0.35000000000000003 0.35000000000000003 rpy=0 0 0 -> xyz=0.25 0.25 0.25 rpy=0 0 0
- joint 011_020: origin xyz=0.0 0.7 0.0 rpy=0 0 0 -> xyz=0.0 0.5 0.0 rpy=0 0 0
- joint 011_021: origin xyz=0.0 0.7 -1.1102230246251565e-16 rpy=0 0 0 -> xyz=0.0 0.5 0.0 rpy=0 0 0
- joint 020_030: origin xyz=0.0 0.7 -0.7000000000000001 rpy=0 0 0 -> xyz=0.0 0.5 -0.5 rpy=0 0 0
- joint 020_031: origin xyz=0.0 0.7 -1.1102230246251565e-16 rpy=0 0 0 -> xyz=0.0 0.5 0.0 rpy=0 0 0
- joint 020_121: origin xyz=0.25 0.3500000000000001 -1.1102230246251565e-16 rpy=0 0 0 -> xyz=0.25 0.25 0.0 rpy=0 0 0
- joint 020_130: origin xyz=0.25 0.7 -0.35000000000000003 rpy=0 0 0 -> xyz=0.25 0.5 -0.25 rpy=0 0 0
- joint 021_022: origin xyz=-0.25 0.3500000000000001 0.7000000000000002 rpy=0 0 0 -> xyz=-0.25 0.25 0.5 rpy=0 0 0
- joint 031_032: origin xyz=0.0 0.3500000000000001 0.7000000000000002 rpy=0 0 0 -> xyz=0.0 0.25 0.5 rpy=0 0 0
- joint 031_132: origin xyz=0.25 0.3500000000000001 0.7000000000000002 rpy=0 0 0 -> xyz=0.25 0.25 0.5 rpy=0 0 0
- joint 100_111: origin xyz=0.25 0.35000000000000003 0.3499999999999999 rpy=0 0 0 -> xyz=0.25 0.25 0.25 rpy=0 0 0
- joint 111_212: origin xyz=0.25 0.35000000000000003 0.7000000000000002 rpy=0 0 0 -> xyz=0.25 0.25 0.5 rpy=0 0 0
- joint 111_221: origin xyz=0.25 0.7 0.3500000000000001 rpy=0 0 0 -> xyz=0.25 0.5 0.25 rpy=0 0 0
- joint 130_220: origin xyz=0.5 2.220446049250313e-16 0.0 rpy=0 0 0 -> xyz=0.5 0.0 0.0 rpy=0 0 0
- joint 212_202: origin xyz=0.25 -0.35000000000000003 0.0 rpy=0 0 0 -> xyz=0.25 -0.25 0.0 rpy=0 0 0
- joint 221_230: origin xyz=0.25 0.7 -0.35 rpy=0 0 0 -> xyz=0.25 0.5 -0.25 rpy=0 0 0

File: body1.urdf (robot description, URDF)
Before this commit: robot robot, 16 links, 15 joints
Links:
- removed link 012
- removed link 132
- removed link 231
- removed link 232
- added link 011, mass 1; collision box size=0.5 0.5 0.5; visual box size=0.5 0.5 0.5
- link 000: geometry collision box size=0.5 0.5 0.5; visual box size=0.5 0.5 0.5
- link 001: geometry collision box size=0.5 0.5 0.5; visual box size=0.5 0.5 0.5
- link 020: geometry collision box size=0.5 0.5 0.5; visual box size=0.5 0.5 0.5
- link 022: geometry collision box size=0.5 0.5 0.5; visual box size=0.5 0.5 0.5
- link 101: geometry collision box size=0.5 0.5 0.5; visual box size=0.5 0.5 0.5
- link 102: geometry collision box size=0.5 0.5 0.5; visual box size=0.5 0.5 0.5
- link 121: geometry collision box size=0.5 0.5 0.5; visual box size=0.5 0.5 0.5
- link 122: geometry collision box size=0.5 0.5 0.5; visual box size=0.5 0.5 0.5
- link 130: geometry collision box size=0.5 0.5 0.5; visual box size=0.5 0.5 0.5
- link 202: geometry collision box size=0.5 0.5 0.5; visual box size=0.5 0.5 0.5
- link 212: geometry collision box size=0.5 0.5 0.5; visual box size=0.5 0.5 0.5
- link 221: geometry collision box size=0.5 0.5 0.5; visual box size=0.5 0.5 0.5
Joints:
- removed joint 102_012
- removed joint 121_022
- removed joint 121_130
- removed joint 121_132
- removed joint 121_231
- removed joint 130_020
- removed joint 132_232
- removed joint 202_212
- removed joint 212_221
- removed joint 221_121
- added joint 000_011: type continuous, parent 000, child 011, origin xyz=0.0 0.25 0.5 rpy=0 0 0, axis 1 0 0, limit lower=-3.14159 upper=3.14159 effort=0.0 velocity=0.0
- added joint 011_020: type revolute, parent 011, child 020, origin xyz=0.0 0.5 0.0 rpy=0 0 0, axis 1 0 0, limit lower=-3.14159 upper=3.14159 effort=0.0 velocity=0.0
- added joint 011_022: type continuous, parent 011, child 022, origin xyz=0.0 0.5 0.5 rpy=0 0 0, axis 1 0 0, limit lower=-3.14159 upper=3.14159 effort=0.0 velocity=0.0
- added joint 020_130: type continuous, parent 020, child 130, origin xyz=0.25 0.5 -0.25 rpy=0 0 0, axis 0 0 1, limit lower=-3.14159 upper=3.14159 effort=0.0 velocity=0.0
- added joint 022_121: type revolute, parent 022, child 121, origin xyz=0.25 0.25 0.0 rpy=0 0 0, axis 0 1 0, limit lower=-3.14159 upper=3.14159 effort=0.0 velocity=0.0
- added joint 122_212: type revolute, parent 122, child 212, origin xyz=0.25 0.0 0.25 rpy=0 0 0, axis 0 0 1, limit lower=-3.14159 upper=3.14159 effort=0.0 velocity=0.0
- added joint 122_221: type revolute, parent 122, child 221, origin xyz=0.25 0.25 0.0 rpy=0 0 0, axis 0 1 0, limit lower=-3.14159 upper=3.14159 effort=0.0 velocity=0.0
- joint 000_001: origin xyz=0.15000000000000002 0.0 0.5 rpy=0 0 0 -> xyz=0.25 0.0 0.5 rpy=0 0 0
- joint 102_202: origin xyz=0.30000000000000004 -0.25 0.25 rpy=0 0 0 -> xyz=0.5 -0.25 0.25 rpy=0 0 0
- joint 121_122: origin xyz=-0.15000000000000002 -0.5 0.25 rpy=0 0 0 -> xyz=0.25 -0.25 0.0 rpy=0 0 0

File: body2.urdf (robot description, URDF)
Before this commit: robot robot, 20 links, 19 joints
Links:
- removed link 132
- link 010: geometry collision box size=0.5 0.5 0.5; visual box size=0.5 0.5 0.5
- link 020: geometry collision box size=0.5 0.5 0.5; visual box size=0.5 0.5 0.5
- link 031: geometry collision box size=0.5 0.5 0.5; visual box size=0.5 0.5 0.5
- link 100: geometry collision box size=0.5 0.5 0.5; visual box size=0.5 0.5 0.5
- link 102: geometry collision box size=0.5 0.5 0.5; visual box size=0.5 0.5 0.5
- link 110: geometry collision box size=0.5 0.5 0.5; visual box size=0.5 0.5 0.5
- link 111: geometry collision box size=0.5 0.5 0.5; visual box size=0.5 0.5 0.5
- link 112: geometry collision box size=0.5 0.5 0.5; visual box size=0.5 0.5 0.5
- link 121: geometry collision box size=0.5 0.5 0.5; visual box size=0.5 0.5 0.5
- link 130: geometry collision box size=0.5 0.5 0.5; visual box size=0.5 0.5 0.5
- link 131: geometry collision box size=0.5 0.5 0.5; visual box size=0.5 0.5 0.5
- link 200: geometry collision box size=0.5 0.5 0.5; visual box size=0.5 0.5 0.5
- link 202: geometry collision box size=0.5 0.5 0.5; visual box size=0.5 0.5 0.5
- link 210: geometry collision box size=0.5 0.5 0.5; visual box size=0.5 0.5 0.5
- link 212: geometry collision box size=0.5 0.5 0.5; visual box size=0.5 0.5 0.5
- link 221: geometry collision box size=0.5 0.5 0.5; visual box size=0.5 0.5 0.5
- link 222: geometry collision box size=0.5 0.5 0.5; visual box size=0.5 0.5 0.5
- link 230: geometry collision box size=0.5 0.5 0.5; visual box size=0.5 0.5 0.5
- link 231: geometry collision box size=0.5 0.5 0.5; visual box size=0.5 0.5 0.5
Joints:
- removed joint 121_132
- joint 010_020: origin xyz=0.0 1.2000000000000002 0.7000000000000001 rpy=0 0 0 -> xyz=0.0 0.75 0.5 rpy=0 0 0
- joint 010_100: origin xyz=0.1 0.4 0.35000000000000003 rpy=0 0 0 -> xyz=0.25 0.25 0.25 rpy=0 0 0
- joint 010_111: origin xyz=0.1 0.8 0.7000000000000001 rpy=0 0 0 -> xyz=0.25 0.5 0.5 rpy=0 0 0
- joint 020_031: origin xyz=0.0 0.8000000000000003 -1.1102230246251565e-16 rpy=0 0 0 -> xyz=0.0 0.5 0.0 rpy=0 0 0
- joint 020_110: origin xyz=0.1 0.0 -0.35000000000000003 rpy=0 0 0 -> xyz=0.25 0.0 -0.25 rpy=0 0 0
- joint 031_131: origin xyz=0.1 0.3999999999999999 0.3500000000000001 rpy=0 0 0 -> xyz=0.25 0.25 0.25 rpy=0 0 0
- joint 100_200: origin xyz=0.20000000000000004 -0.8 0.0 rpy=0 0 0 -> xyz=0.5 -0.5 0.0 rpy=0 0 0
- joint 110_121: origin xyz=0.1 0.0 0.3499999999999999 rpy=0 0 0 -> xyz=0.25 0.0 0.25 rpy=0 0 0
- joint 111_112: origin xyz=0.1 -0.4 0.7000000000000001 rpy=0 0 0 -> xyz=0.25 -0.25 0.5 rpy=0 0 0
- joint 112_202: origin xyz=0.10000000000000003 0.0 0.3500000000000001 rpy=0 0 0 -> xyz=0.25 0.0 0.25 rpy=0 0 0
- joint 112_212: origin xyz=0.10000000000000003 0.4 0.7 rpy=0 0 0 -> xyz=0.25 0.25 0.5 rpy=0 0 0
- joint 121_130: origin xyz=0.0 0.8000000000000003 1.1102230246251565e-16 rpy=0 0 0 -> xyz=0.0 0.5 0.0 rpy=0 0 0
- joint 131_230: origin xyz=0.20000000000000004 0.0 -0.35 rpy=0 0 0 -> xyz=0.5 0.0 -0.25 rpy=0 0 0
- joint 200_210: origin xyz=0.0 0.8 0.0 rpy=0 0 0 -> xyz=0.0 0.5 0.0 rpy=0 0 0
- joint 202_102: origin xyz=0.0 -0.4 0.0 rpy=0 0 0 -> xyz=0.0 -0.25 0.0 rpy=0 0 0
- joint 212_221: origin xyz=0.09999999999999998 0.40000000000000013 -0.7 rpy=0 0 0 -> xyz=0.25 0.25 -0.5 rpy=0 0 0
- joint 221_222: origin xyz=0.0 0.3999999999999999 0.0 rpy=0 0 0 -> xyz=0.0 0.25 0.0 rpy=0 0 0
- joint 222_231: origin xyz=0.0 0.40000000000000036 0.0 rpy=0 0 0 -> xyz=0.0 0.25 0.0 rpy=0 0 0

File: body3.urdf (robot description, URDF)
Before this commit: robot robot, 15 links, 14 joints
Links:
- removed link 111
Joints:
- removed joint 120_111

File: body4.urdf (robot description, URDF)
Before this commit: robot robot, 22 links, 21 joints
Links:
- removed link 030
- removed link 210
- added link 212, mass 1; collision box size=0.5 0.5 0.5; visual box size=0.5 0.5 0.5
- link 000: geometry collision box size=0.5 0.5 0.5; visual box size=0.5 0.5 0.5
- link 001: geometry collision box size=0.5 0.5 0.5; visual box size=0.5 0.5 0.5
- link 011: geometry collision box size=0.5 0.5 0.5; visual box size=0.5 0.5 0.5
- link 012: geometry collision box size=0.5 0.5 0.5; visual box size=0.5 0.5 0.5
- link 020: geometry collision box size=0.5 0.5 0.5; visual box size=0.5 0.5 0.5
- link 021: geometry collision box size=0.5 0.5 0.5; visual box size=0.5 0.5 0.5
- link 022: geometry collision box size=0.5 0.5 0.5; visual box size=0.5 0.5 0.5
- link 031: geometry collision box size=0.5 0.5 0.5; visual box size=0.5 0.5 0.5
- link 100: geometry collision box size=0.5 0.5 0.5; visual box size=0.5 0.5 0.5
- link 101: geometry collision box size=0.5 0.5 0.5; visual box size=0.5 0.5 0.5
- link 102: geometry collision box size=0.5 0.5 0.5; visual box size=0.5 0.5 0.5
- link 111: geometry collision box size=0.5 0.5 0.5; visual box size=0.5 0.5 0.5
- link 112: geometry collision box size=0.5 0.5 0.5; visual box size=0.5 0.5 0.5
- link 120: geometry collision box size=0.5 0.5 0.5; visual box size=0.5 0.5 0.5
- link 131: geometry collision box size=0.5 0.5 0.5; visual box size=0.5 0.5 0.5
- link 200: geometry collision box size=0.5 0.5 0.5; visual box size=0.5 0.5 0.5
- link 211: geometry collision box size=0.5 0.5 0.5; visual box size=0.5 0.5 0.5
- link 220: geometry collision box size=0.5 0.5 0.5; visual box size=0.5 0.5 0.5
- link 230: geometry collision box size=0.5 0.5 0.5; visual box size=0.5 0.5 0.5
- link 232: geometry collision box size=0.5 0.5 0.5; visual box size=0.5 0.5 0.5
Joints:
- removed joint 031_030
- removed joint 200_210
- added joint 211_212: type continuous, parent 211, child 212, origin xyz=0.5 0.25 0.25 rpy=0 0 0, axis 0 1 0, limit lower=-3.14159 upper=3.14159 effort=0.0 velocity=0.0
- joint 000_011: origin xyz=0.0 0.2 0.5 rpy=0 0 0 -> xyz=0.0 0.25 0.5 rpy=0 0 0
- joint 000_100: origin xyz=0.25 -0.2 0.25 rpy=0 0 0 -> xyz=0.25 -0.25 0.25 rpy=0 0 0
- joint 011_012: origin xyz=-0.25 0.2 0.5 rpy=0 0 0 -> xyz=-0.25 0.25 0.5 rpy=0 0 0
- joint 011_020: origin xyz=0.0 0.4000000000000001 0.0 rpy=0 0 0 -> xyz=0.0 0.5 0.0 rpy=0 0 0
- joint 012_112: origin xyz=0.5 -0.2 0.25 rpy=0 0 0 -> xyz=0.5 -0.25 0.25 rpy=0 0 0
- joint 020_021: origin xyz=0.25 0.19999999999999996 0.0 rpy=0 0 0 -> xyz=0.25 0.25 0.0 rpy=0 0 0
- joint 021_031: origin xyz=-0.25 0.20000000000000018 0.0 rpy=0 0 0 -> xyz=-0.25 0.25 0.0 rpy=0 0 0
- joint 101_102: origin xyz=0.25 -0.4 0.25 rpy=0 0 0 -> xyz=0.25 -0.5 0.25 rpy=0 0 0
- joint 101_200: origin xyz=0.5 -0.2 -0.25 rpy=0 0 0 -> xyz=0.5 -0.25 -0.25 rpy=0 0 0
- joint 102_111: origin xyz=0.0 0.4 0.0 rpy=0 0 0 -> xyz=0.0 0.5 0.0 rpy=0 0 0
- joint 120_131: origin xyz=0.25 0.20000000000000018 0.0 rpy=0 0 0 -> xyz=0.25 0.25 0.0 rpy=0 0 0
- joint 120_220: origin xyz=0.5 0.19999999999999996 -0.25 rpy=0 0 0 -> xyz=0.5 0.25 -0.25 rpy=0 0 0
- joint 131_230: origin xyz=0.25 0.19999999999999996 0.0 rpy=0 0 0 -> xyz=0.25 0.25 0.0 rpy=0 0 0
- joint 131_232: origin xyz=0.25 0.19999999999999996 0.5 rpy=0 0 0 -> xyz=0.25 0.25 0.5 rpy=0 0 0
