Commit message: updated pickle

File: files/body0.urdf (robot description, URDF)
Before this commit: robot robot, 20 links, 19 joints
Links:
- removed link 000
- removed link 001
- removed link 011
- removed link 020
- removed link 021
- removed link 022
- removed link 110
- removed link 111
- removed link 221
- removed link 230
- added link 002, mass 1; collision box size=0.5 0.5 0.5; visual box size=0.5 0.5 0.5
- added link 010, mass 1; collision box size=0.5 0.5 0.5; visual box size=0.5 0.5 0.5
- added link 101, mass 1; collision box size=0.5 0.5 0.5; visual box size=0.5 0.5 0.5
- added link 112, mass 1; collision box size=0.5 0.5 0.5; visual box size=0.5 0.5 0.5
- added link 122, mass 1; collision box size=0.5 0.5 0.5; visual box size=0.5 0.5 0.5
- added link 131, mass 1; collision box size=0.5 0.5 0.5; visual box size=0.5 0.5 0.5
- added link 201, mass 1; collision box size=0.5 0.5 0.5; visual box size=0.5 0.5 0.5
- added link 231, mass 1; collision box size=0.5 0.5 0.5; visual box size=0.5 0.5 0.5
- added link 232, mass 1; collision box size=0.5 0.5 0.5; visual box size=0.5 0.5 0.5
Joints:
- removed joint 000_001
- removed joint 000_011
- removed joint 000_100
- removed joint 000_110
- removed joint 011_020
- removed joint 011_021
- removed joint 020_030
- removed joint 020_031
- removed joint 020_121
- removed joint 020_130
- removed joint 021_022
- removed joint 031_032
- removed joint 031_132
- removed joint 100_111
- removed joint 111_212
- removed joint 111_221
- removed joint 212_202
- removed joint 221_230
- added joint 002_101: type revolute, parent 002, child 101, origin xyz=0.25 0.0 1.0 rpy=0 0 0, axis 0 1 0, limit lower=-3.14159 upper=3.14159 effort=0.0 velocity=0.0
- added joint 100_010: type continuous, parent 100, child 010, origin xyz=0.0 0.25 -0.25 rpy=0 0 0, axis 0 0 1, limit lower=-3.14159 upper=3.14159 effort=0.0 velocity=0.0
- added joint 101_100: type revolute, parent 101, child 100, origin xyz=0.0 0.0 -0.5 rpy=0 0 0, axis 0 1 0, limit lower=-3.14159 upper=3.14159 effort=0.0 velocity=0.0
- added joint 101_112: type revolute, parent 101, child 112, origin xyz=0.25 0.25 0.0 rpy=0 0 0, axis 1 0 0, limit lower=-3.14159 upper=3.14159 effort=0.0 velocity=0.0
- added joint 101_201: type revolute, parent 101, child 201, origin xyz=0.5 0.25 -0.25 rpy=0 0 0, axis 0 0 1, limit lower=-3.14159 upper=3.14159 effort=0.0 velocity=0.0
- added joint 101_202: type revolute, parent 101, child 202, origin xyz=0.5 0.0 0.0 rpy=0 0 0, axis 0 1 0, limit lower=-3.14159 upper=3.14159 effort=0.0 velocity=0.0
- added joint 112_121: type continuous, parent 112, child 121, origin xyz=0.0 0.5 0.0 rpy=0 0 0, axis 1 0 0, limit lower=-3.14159 upper=3.14159 effort=0.0 velocity=0.0
- added joint 112_122: type continuous, parent 112, child 122, origin xyz=0.25 0.5 0.25 rpy=0 0 0, axis 0 0 1, limit lower=-3.14159 upper=3.14159 effort=0.0 velocity=0.0
- added joint 121_130: type revolute, parent 121, child 130, origin xyz=0.0 0.5 -0.5 rpy=0 0 0, axis 1 0 0, limit lower=-3.14159 upper=3.14159 effort=0.0 velocity=0.0
- added joint 122_032: type revolute, parent 122, child 032, origin xyz=-0.5 0.5 0.0 rpy=0 0 0, axis 0 0 1, limit lower=-3.14159 upper=3.14159 effort=0.0 velocity=0.0
- added joint 122_131: type continuous, parent 122, child 131, origin xyz=-0.25 0.5 -0.25 rpy=0 0 0, axis 1 0 0, limit lower=-3.14159 upper=3.14159 effort=0.0 velocity=0.0
- added joint 122_212: type continuous, parent 122, child 212, origin xyz=0.0 0.0 0.0 rpy=0 0 0, axis 0 0 1, limit lower=-3.14159 upper=3.14159 effort=0.0 velocity=0.0
- added joint 122_232: type continuous, parent 122, child 232, origin xyz=0.0 0.5 0.0 rpy=0 0 0, axis 0 0 1, limit lower=-3.14159 upper=3.14159 effort=0.0 velocity=0.0
- added joint 131_030: type continuous, parent 131, child 030, origin xyz=-0.25 0.25 -0.5 rpy=0 0 0, axis 0 1 0, limit lower=-3.14159 upper=3.14159 effort=0.0 velocity=0.0
- added joint 131_031: type revolute, parent 131, child 031, origin xyz=-0.25 0.5 -0.25 rpy=0 0 0, axis 0 0 1, limit lower=-3.14159 upper=3.14159 effort=0.0 velocity=0.0
- added joint 131_132: type continuous, parent 131, child 132, origin xyz=0.0 0.0 0.0 rpy=0 0 0, axis 1 0 0, limit lower=-3.14159 upper=3.14159 effort=0.0 velocity=0.0
- added joint 131_231: type continuous, parent 131, child 231, origin xyz=0.25 0.25 -0.25 rpy=0 0 0, axis 0 0 1, limit lower=-3.14159 upper=3.14159 effort=0.0 velocity=0.0
- joint 130_220: origin xyz=0.5 0.0 0.0 rpy=0 0 0 -> xyz=0.25 0.0 -0.25 rpy=0 0 0; type continuous -> revolute

File: files/body1.urdf (robot description, URDF)
Before this commit: robot robot, 14 links, 13 joints
Links:
- removed link 001
- removed link 021
- removed link 031
- removed link 131
- removed link 221
- removed link 222
- removed link 230
- removed link 231
- added link 000, mass 1; collision box size=0.5 0.5 0.5; visual box size=0.5 0.5 0.5
- added link 010, mass 1; collision box size=0.5 0.5 0.5; visual box size=0.5 0.5 0.5
- added link 011, mass 1; collision box size=0.5 0.5 0.5; visual box size=0.5 0.5 0.5
- added link 012, mass 1; collision box size=0.5 0.5 0.5; visual box size=0.5 0.5 0.5
- added link 030, mass 1; collision box size=0.5 0.5 0.5; visual box size=0.5 0.5 0.5
- added link 032, mass 1; collision box size=0.5 0.5 0.5; visual box size=0.5 0.5 0.5
- added link 100, mass 1; collision box size=0.5 0.5 0.5; visual box size=0.5 0.5 0.5
- added link 102, mass 1; collision box size=0.5 0.5 0.5; visual box size=0.5 0.5 0.5
- added link 121, mass 1; collision box size=0.5 0.5 0.5; visual box size=0.5 0.5 0.5
- added link 122, mass 1; collision box size=0.5 0.5 0.5; visual box size=0.5 0.5 0.5
- added link 202, mass 1; collision box size=0.5 0.5 0.5; visual box size=0.5 0.5 0.5
- added link 210, mass 1; collision box size=0.5 0.5 0.5; visual box size=0.5 0.5 0.5
- added link 220, mass 1; collision box size=0.5 0.5 0.5; visual box size=0.5 0.5 0.5
Joints:
- removed joint 001_002
- removed joint 002_101
- removed joint 021_031
- removed joint 101_201
- removed joint 120_021
- removed joint 131_132
- removed joint 201_212
- removed joint 212_221
- removed joint 221_120
- removed joint 221_222
- removed joint 221_230
- removed joint 222_231
- removed joint 230_131
- added joint 000_010: type revolute, parent 000, child 010, origin xyz=-0.25 0.25 0.25 rpy=0 0 0, axis 0 0 1, limit lower=-3.14159 upper=3.14159 effort=0.0 velocity=0.0
- added joint 000_011: type revolute, parent 000, child 011, origin xyz=0.0 0.25 0.5 rpy=0 0 0, axis 1 0 0, limit lower=-3.14159 upper=3.14159 effort=0.0 velocity=0.0
- added joint 000_100: type continuous, parent 000, child 100, origin xyz=0.25 -0.25 0.25 rpy=0 0 0, axis 0 0 1, limit lower=-3.14159 upper=3.14159 effort=0.0 velocity=0.0
- added joint 010_120: type continuous, parent 010, child 120, origin xyz=0.5 0.5 0.0 rpy=0 0 0, axis 0 0 1, limit lower=-3.14159 upper=3.14159 effort=0.0 velocity=0.0
- added joint 011_002: type continuous, parent 011, child 002, origin xyz=0.0 0.0 0.5 rpy=0 0 0, axis 1 0 0, limit lower=-3.14159 upper=3.14159 effort=0.0 velocity=0.0
- added joint 011_012: type revolute, parent 011, child 012, origin xyz=0.0 0.5 0.5 rpy=0 0 0, axis 1 0 0, limit lower=-3.14159 upper=3.14159 effort=0.0 velocity=0.0
- added joint 012_102: type continuous, parent 012, child 102, origin xyz=0.25 -0.5 0.25 rpy=0 0 0, axis 0 0 1, limit lower=-3.14159 upper=3.14159 effort=0.0 velocity=0.0
- added joint 100_101: type continuous, parent 100, child 101, origin xyz=0.25 0.0 0.25 rpy=0 0 0, axis 1 0 0, limit lower=-3.14159 upper=3.14159 effort=0.0 velocity=0.0
- added joint 102_201: type revolute, parent 102, child 201, origin xyz=0.5 -0.25 -0.25 rpy=0 0 0, axis 0 1 0, limit lower=-3.14159 upper=3.14159 effort=0.0 velocity=0.0
- added joint 120_030: type revolute, parent 120, child 030, origin xyz=0.0 0.5 0.0 rpy=0 0 0, axis 0 0 1, limit lower=-3.14159 upper=3.14159 effort=0.0 velocity=0.0
- added joint 120_121: type continuous, parent 120, child 121, origin xyz=0.25 0.0 0.25 rpy=0 0 0, axis 1 0 0, limit lower=-3.14159 upper=3.14159 effort=0.0 velocity=0.0
- added joint 120_220: type continuous, parent 120, child 220, origin xyz=0.5 0.5 0.0 rpy=0 0 0, axis 0 0 1, limit lower=-3.14159 upper=3.14159 effort=0.0 velocity=0.0
- added joint 121_122: type continuous, parent 121, child 122, origin xyz=-0.25 0.25 0.5 rpy=0 0 0, axis 0 1 0, limit lower=-3.14159 upper=3.14159 effort=0.0 velocity=0.0
- added joint 122_032: type continuous, parent 122, child 032, origin xyz=0.0 0.25 0.25 rpy=0 0 0, axis 0 0 1, limit lower=-3.14159 upper=3.14159 effort=0.0 velocity=0.0
- added joint 122_132: type continuous, parent 122, child 132, origin xyz=0.5 0.25 0.25 rpy=0 0 0, axis 0 0 1, limit lower=-3.14159 upper=3.14159 effort=0.0 velocity=0.0
- added joint 201_202: type continuous, parent 201, child 202, origin xyz=0.25 -0.25 0.0 rpy=0 0 0, axis 1 0 0, limit lower=-3.14159 upper=3.14159 effort=0.0 velocity=0.0
- added joint 201_210: type revolute, parent 201, child 210, origin xyz=0.25 0.25 -0.5 rpy=0 0 0, axis 1 0 0, limit lower=-3.14159 upper=3.14159 effort=0.0 velocity=0.0
- added joint 202_212: type continuous, parent 202, child 212, origin xyz=0.0 0.5 0.25 rpy=0 0 0, axis 0 0 1, limit lower=-3.14159 upper=3.14159 effort=0.0 velocity=0.0

File: files/body3.urdf (robot description, URDF)
Before this commit: robot robot, 19 links, 18 joints
Links:
- removed link 010
- removed link 100
- removed link 102
- removed link 111
- removed link 222
- removed link 230
- removed link 231
- added link 000, mass 1; collision box size=0.5 0.5 0.5; visual box size=0.5 0.5 0.5
- added link 001, mass 1; collision box size=0.5 0.5 0.5; visual box size=0.5 0.5 0.5
- added link 002, mass 1; collision box size=0.5 0.5 0.5; visual box size=0.5 0.5 0.5
- added link 011, mass 1; collision box size=0.5 0.5 0.5; visual box size=0.5 0.5 0.5
- added link 012, mass 1; collision box size=0.5 0.5 0.5; visual box size=0.5 0.5 0.5
- added link 021, mass 1; collision box size=0.5 0.5 0.5; visual box size=0.5 0.5 0.5
- added link 022, mass 1; collision box size=0.5 0.5 0.5; visual box size=0.5 0.5 0.5
- added link 032, mass 1; collision box size=0.5 0.5 0.5; visual box size=0.5 0.5 0.5
- added link 101, mass 1; collision box size=0.5 0.5 0.5; visual box size=0.5 0.5 0.5
- added link 120, mass 1; collision box size=0.5 0.5 0.5; visual box size=0.5 0.5 0.5
- added link 201, mass 1; collision box size=0.5 0.5 0.5; visual box size=0.5 0.5 0.5
- added link 220, mass 1; collision box size=0.5 0.5 0.5; visual box size=0.5 0.5 0.5
- added link 232, mass 1; collision box size=0.5 0.5 0.5; visual box size=0.5 0.5 0.5
Joints:
- removed joint 010_020
- removed joint 010_100
- removed joint 010_111
- removed joint 020_031
- removed joint 020_110
- removed joint 031_131
- removed joint 100_200
- removed joint 110_121
- removed joint 111_112
- removed joint 112_212
- removed joint 121_130
- removed joint 131_230
- removed joint 200_210
- removed joint 202_102
- removed joint 212_221
- removed joint 221_222
- removed joint 222_231
- added joint 000_001: type revolute, parent 000, child 001, origin xyz=0.0 0.25 0.5 rpy=0 0 0, axis 1 0 0, limit lower=-3.14159 upper=3.14159 effort=0.0 velocity=0.0
- added joint 000_101: type revolute, parent 000, child 101, origin xyz=0.25 0.0 0.5 rpy=0 0 0, axis 0 1 0, limit lower=-3.14159 upper=3.14159 effort=0.0 velocity=0.0
- added joint 000_110: type continuous, parent 000, child 110, origin xyz=0.25 0.25 0.25 rpy=0 0 0, axis 0 0 1, limit lower=-3.14159 upper=3.14159 effort=0.0 velocity=0.0
- added joint 001_002: type continuous, parent 001, child 002, origin xyz=0.25 -0.25 0.5 rpy=0 0 0, axis 0 1 0, limit lower=-3.14159 upper=3.14159 effort=0.0 velocity=0.0
- added joint 001_011: type revolute, parent 001, child 011, origin xyz=0.0 0.0 0.5 rpy=0 0 0, axis 1 0 0, limit lower=-3.14159 upper=3.14159 effort=0.0 velocity=0.0
- added joint 001_012: type continuous, parent 001, child 012, origin xyz=0.0 0.0 0.5 rpy=0 0 0, axis 1 0 0, limit lower=-3.14159 upper=3.14159 effort=0.0 velocity=0.0
- added joint 011_020: type continuous, parent 011, child 020, origin xyz=0.0 0.5 -0.5 rpy=0 0 0, axis 1 0 0, limit lower=-3.14159 upper=3.14159 effort=0.0 velocity=0.0
- added joint 011_121: type continuous, parent 011, child 121, origin xyz=0.25 0.5 -0.25 rpy=0 0 0, axis 0 0 1, limit lower=-3.14159 upper=3.14159 effort=0.0 velocity=0.0
- added joint 012_021: type continuous, parent 012, child 021, origin xyz=0.0 0.5 0.0 rpy=0 0 0, axis 1 0 0, limit lower=-3.14159 upper=3.14159 effort=0.0 velocity=0.0
- added joint 012_112: type continuous, parent 012, child 112, origin xyz=0.25 0.0 0.25 rpy=0 0 0, axis 0 0 1, limit lower=-3.14159 upper=3.14159 effort=0.0 velocity=0.0
- added joint 021_022: type revolute, parent 021, child 022, origin xyz=0.0 0.5 0.0 rpy=0 0 0, axis 1 0 0, limit lower=-3.14159 upper=3.14159 effort=0.0 velocity=0.0
- added joint 021_120: type continuous, parent 021, child 120, origin xyz=0.25 0.25 -0.5 rpy=0 0 0, axis 0 1 0, limit lower=-3.14159 upper=3.14159 effort=0.0 velocity=0.0
- added joint 022_031: type continuous, parent 022, child 031, origin xyz=0.0 0.0 0.0 rpy=0 0 0, axis 1 0 0, limit lower=-3.14159 upper=3.14159 effort=0.0 velocity=0.0
- added joint 031_032: type continuous, parent 031, child 032, origin xyz=0.25 0.25 0.0 rpy=0 0 0, axis 0 1 0, limit lower=-3.14159 upper=3.14159 effort=0.0 velocity=0.0
- added joint 101_201: type revolute, parent 101, child 201, origin xyz=0.5 -0.25 0.25 rpy=0 0 0, axis 0 0 1, limit lower=-3.14159 upper=3.14159 effort=0.0 velocity=0.0
- added joint 110_200: type continuous, parent 110, child 200, origin xyz=0.5 0.0 0.0 rpy=0 0 0, axis 0 0 1, limit lower=-3.14159 upper=3.14159 effort=0.0 velocity=0.0
- added joint 120_130: type continuous, parent 120, child 130, origin xyz=0.25 0.25 -0.25 rpy=0 0 0, axis 0 0 1, limit lower=-3.14159 upper=3.14159 effort=0.0 velocity=0.0
- added joint 121_131: type revolute, parent 121, child 131, origin xyz=0.0 0.5 0.0 rpy=0 0 0, axis 0 0 1, limit lower=-3.14159 upper=3.14159 effort=0.0 velocity=0.0
- added joint 121_221: type revolute, parent 121, child 221, origin xyz=0.5 0.0 0.0 rpy=0 0 0, axis 0 0 1, limit lower=-3.14159 upper=3.14159 effort=0.0 velocity=0.0
- added joint 201_210: type revolute, parent 201, child 210, origin xyz=0.25 0.5 -0.25 rpy=0 0 0, axis 1 0 0, limit lower=-3.14159 upper=3.14159 effort=0.0 velocity=0.0
- added joint 201_212: type continuous, parent 201, child 212, origin xyz=0.25 0.5 0.25 rpy=0 0 0, axis 1 0 0, limit lower=-3.14159 upper=3.14159 effort=0.0 velocity=0.0
- added joint 210_220: type continuous, parent 210, child 220, origin xyz=0.25 0.5 -0.25 rpy=0 0 0, axis 0 0 1, limit lower=-3.14159 upper=3.14159 effort=0.0 velocity=0.0
- added joint 221_232: type revolute, parent 221, child 232, origin xyz=0.25 0.5 0.25 rpy=0 0 0, axis 1 0 0, limit lower=-3.14159 upper=3.14159 effort=0.0 velocity=0.0
- joint 112_202: origin xyz=0.25 0.0 0.25 rpy=0 0 0 -> xyz=0.5 0.0 0.0 rpy=0 0 0

File: files/body4.urdf (robot description, URDF)
Before this commit: robot robot, 21 links, 20 joints
Links:
- removed link 021
- removed link 022
- removed link 031
- removed link 211
- removed link 220
- removed link 230
- added link 010, mass 1; collision box size=0.5 0.5 0.5; visual box size=0.5 0.5 0.5
- added link 030, mass 1; collision box size=0.5 0.5 0.5; visual box size=0.5 0.5 0.5
- added link 032, mass 1; collision box size=0.5 0.5 0.5; visual box size=0.5 0.5 0.5
- added link 132, mass 1; collision box size=0.5 0.5 0.5; visual box size=0.5 0.5 0.5
- added link 202, mass 1; collision box size=0.5 0.5 0.5; visual box size=0.5 0.5 0.5
- added link 231, mass 1; collision box size=0.5 0.5 0.5; visual box size=0.5 0.5 0.5
Joints:
- removed joint 011_012
- removed joint 012_112
- removed joint 020_021
- removed joint 021_022
- removed joint 021_031
- removed joint 021_120
- removed joint 101_200
- removed joint 101_211
- removed joint 102_111
- removed joint 120_220
- removed joint 131_230
- removed joint 131_232
- removed joint 211_212
- added joint 001_010: type continuous, parent 001, child 010, origin xyz=0.0 0.0 0.0 rpy=0 0 0, axis 1 0 0, limit lower=-3.14159 upper=3.14159 effort=0.0 velocity=0.0
- added joint 001_012: type revolute, parent 001, child 012, origin xyz=0.0 0.0 0.5 rpy=0 0 0, axis 1 0 0, limit lower=-3.14159 upper=3.14159 effort=0.0 velocity=0.0
- added joint 011_112: type revolute, parent 011, child 112, origin xyz=0.25 0.25 0.5 rpy=0 0 0, axis 0 1 0, limit lower=-3.14159 upper=3.14159 effort=0.0 velocity=0.0
- added joint 020_030: type revolute, parent 020, child 030, origin xyz=0.25 0.5 -0.25 rpy=0 0 0, axis 0 0 1, limit lower=-3.14159 upper=3.14159 effort=0.0 velocity=0.0
- added joint 100_200: type continuous, parent 100, child 200, origin xyz=0.5 0.25 0.25 rpy=0 0 0, axis 0 1 0, limit lower=-3.14159 upper=3.14159 effort=0.0 velocity=0.0
- added joint 101_111: type revolute, parent 101, child 111, origin xyz=0.5 0.0 0.0 rpy=0 0 0, axis 0 0 1, limit lower=-3.14159 upper=3.14159 effort=0.0 velocity=0.0
- added joint 101_202: type revolute, parent 101, child 202, origin xyz=0.5 -0.25 0.25 rpy=0 0 0, axis 0 1 0, limit lower=-3.14159 upper=3.14159 effort=0.0 velocity=0.0
- added joint 111_120: type revolute, parent 111, child 120, origin xyz=-0.25 0.5 -0.25 rpy=0 0 0, axis 1 0 0, limit lower=-3.14159 upper=3.14159 effort=0.0 velocity=0.0
- added joint 112_212: type continuous, parent 112, child 212, origin xyz=0.5 0.0 0.5 rpy=0 0 0, axis 0 1 0, limit lower=-3.14159 upper=3.14159 effort=0.0 velocity=0.0
- added joint 131_032: type continuous, parent 131, child 032, origin xyz=-0.25 0.25 0.5 rpy=0 0 0, axis 0 1 0, limit lower=-3.14159 upper=3.14159 effort=0.0 velocity=0.0
- added joint 131_132: type continuous, parent 131, child 132, origin xyz=0.25 0.25 0.5 rpy=0 0 0, axis 0 1 0, limit lower=-3.14159 upper=3.14159 effort=0.0 velocity=0.0
- added joint 131_231: type revolute, parent 131, child 231, origin xyz=0.25 0.0 0.25 rpy=0 0 0, axis 0 0 1, limit lower=-3.14159 upper=3.14159 effort=0.0 velocity=0.0
- added joint 231_232: type continuous, parent 231, child 232, origin xyz=0.25 0.25 0.25 rpy=0 0 0, axis 1 0 0, limit lower=-3.14159 upper=3.14159 effort=0.0 velocity=0.0
- joint 000_001: axis 0 1 0 -> 1 0 0; origin xyz=0.0 0.0 0.5 rpy=0 0 0 -> xyz=0.0 0.25 0.5 rpy=0 0 0
- joint 011_101: type continuous -> revolute
- joint 101_102: origin xyz=0.25 -0.5 0.25 rpy=0 0 0 -> xyz=0.25 -0.25 0.25 rpy=0 0 0; type revolute -> continuous
- joint 120_131: origin xyz=0.25 0.25 0.0 rpy=0 0 0 -> xyz=0.0 0.5 0.0 rpy=0 0 0
