Commit message: complete

File: files/body0.urdf (robot description, URDF)
Before this commit: robot robot, 19 links, 18 joints
Links:
- removed link 002
- removed link 010
- removed link 101
- removed link 112
- removed link 122
- removed link 131
- removed link 201
- removed link 231
- removed link 232
- added link 000, mass 1; collision box size=0.5 0.5 0.5; visual box size=0.5 0.5 0.5
- added link 001, mass 1; collision box size=0.5 0.5 0.5; visual box size=0.5 0.5 0.5
- added link 011, mass 1; collision box size=0.5 0.5 0.5; visual box size=0.5 0.5 0.5
- added link 020, mass 1; collision box size=0.5 0.5 0.5; visual box size=0.5 0.5 0.5
- added link 021, mass 1; collision box size=0.5 0.5 0.5; visual box size=0.5 0.5 0.5
- added link 022, mass 1; collision box size=0.5 0.5 0.5; visual box size=0.5 0.5 0.5
- added link 110, mass 1; collision box size=0.5 0.5 0.5; visual box size=0.5 0.5 0.5
- added link 111, mass 1; collision box size=0.5 0.5 0.5; visual box size=0.5 0.5 0.5
- added link 221, mass 1; collision box size=0.5 0.5 0.5; visual box size=0.5 0.5 0.5
- added link 230, mass 1; collision box size=0.5 0.5 0.5; visual box size=0.5 0.5 0.5
Joints:
- removed joint 002_101
- removed joint 100_010
- removed joint 101_100
- removed joint 101_112
- removed joint 101_201
- removed joint 101_202
- removed joint 112_121
- removed joint 112_122
- removed joint 121_130
- removed joint 122_032
- removed joint 122_131
- removed joint 122_212
- removed joint 122_232
- removed joint 131_030
- removed joint 131_031
- removed joint 131_132
- removed joint 131_231
- added joint 000_001: type continuous, parent 000, child 001, origin xyz=0.0 -0.25 0.5 rpy=0 0 0, axis 1 0 0, limit lower=-3.14159 upper=3.14159 effort=0.0 velocity=0.0
- added joint 000_011: type revolute, parent 000, child 011, origin xyz=0.0 0.25 0.5 rpy=0 0 0, axis 1 0 0, limit lower=-3.14159 upper=3.14159 effort=0.0 velocity=0.0
- added joint 000_100: type continuous, parent 000, child 100, origin xyz=0.25 0.0 0.25 rpy=0 0 0, axis 0 0 1, limit lower=-3.14159 upper=3.14159 effort=0.0 velocity=0.0
- added joint 000_110: type revolute, parent 000, child 110, origin xyz=0.25 0.25 0.25 rpy=0 0 0, axis 0 0 1, limit lower=-3.14159 upper=3.14159 effort=0.0 velocity=0.0
- added joint 011_020: type revolute, parent 011, child 020, origin xyz=0.0 0.5 0.0 rpy=0 0 0, axis 1 0 0, limit lower=-3.14159 upper=3.14159 effort=0.0 velocity=0.0
- added joint 011_021: type continuous, parent 011, child 021, origin xyz=0.0 0.5 0.0 rpy=0 0 0, axis 1 0 0, limit lower=-3.14159 upper=3.14159 effort=0.0 velocity=0.0
- added joint 020_030: type continuous, parent 020, child 030, origin xyz=0.0 0.5 -0.5 rpy=0 0 0, axis 1 0 0, limit lower=-3.14159 upper=3.14159 effort=0.0 velocity=0.0
- added joint 020_031: type revolute, parent 020, child 031, origin xyz=0.0 0.5 0.0 rpy=0 0 0, axis 1 0 0, limit lower=-3.14159 upper=3.14159 effort=0.0 velocity=0.0
- added joint 020_121: type revolute, parent 020, child 121, origin xyz=0.25 0.25 0.0 rpy=0 0 0, axis 0 1 0, limit lower=-3.14159 upper=3.14159 effort=0.0 velocity=0.0
- added joint 020_130: type continuous, parent 020, child 130, origin xyz=0.25 0.5 -0.25 rpy=0 0 0, axis 0 0 1, limit lower=-3.14159 upper=3.14159 effort=0.0 velocity=0.0
- added joint 021_022: type continuous, parent 021, child 022, origin xyz=-0.25 0.25 0.5 rpy=0 0 0, axis 0 1 0, limit lower=-3.14159 upper=3.14159 effort=0.0 velocity=0.0
- added joint 031_032: type continuous, parent 031, child 032, origin xyz=0.0 0.25 0.5 rpy=0 0 0, axis 0 1 0, limit lower=-3.14159 upper=3.14159 effort=0.0 velocity=0.0
- added joint 031_132: type revolute, parent 031, child 132, origin xyz=0.25 0.25 0.5 rpy=0 0 0, axis 0 1 0, limit lower=-3.14159 upper=3.14159 effort=0.0 velocity=0.0
- added joint 100_111: type continuous, parent 100, child 111, origin xyz=0.25 0.25 0.25 rpy=0 0 0, axis 1 0 0, limit lower=-3.14159 upper=3.14159 effort=0.0 velocity=0.0
- added joint 111_212: type revolute, parent 111, child 212, origin xyz=0.25 0.25 0.5 rpy=0 0 0, axis 0 1 0, limit lower=-3.14159 upper=3.14159 effort=0.0 velocity=0.0
- added joint 111_221: type revolute, parent 111, child 221, origin xyz=0.25 0.5 0.25 rpy=0 0 0, axis 0 0 1, limit lower=-3.14159 upper=3.14159 effort=0.0 velocity=0.0
- added joint 212_202: type revolute, parent 212, child 202, origin xyz=0.25 -0.25 0.0 rpy=0 0 0, axis 1 0 0, limit lower=-3.14159 upper=3.14159 effort=0.0 velocity=0.0
- added joint 221_230: type revolute, parent 221, child 230, origin xyz=0.25 0.5 -0.25 rpy=0 0 0, axis 1 0 0, limit lower=-3.14159 upper=3.14159 effort=0.0 velocity=0.0
- joint 130_220: origin xyz=0.25 0.0 -0.25 rpy=0 0 0 -> xyz=0.5 0.0 0.0 rpy=0 0 0; type revolute -> continuous

File: files/body1.urdf (robot description, URDF)
Before this commit: robot robot, 19 links, 18 joints
Links:
- removed link 002
- removed link 010
- removed link 012
- removed link 030
- removed link 032
- removed link 100
- removed link 120
- removed link 132
- removed link 201
- removed link 210
- removed link 220
- added link 001, mass 1; collision box size=0.5 0.5 0.5; visual box size=0.5 0.5 0.5
- added link 020, mass 1; collision box size=0.5 0.5 0.5; visual box size=0.5 0.5 0.5
- added link 022, mass 1; collision box size=0.5 0.5 0.5; visual box size=0.5 0.5 0.5
- added link 130, mass 1; collision box size=0.5 0.5 0.5; visual box size=0.5 0.5 0.5
- added link 221, mass 1; collision box size=0.5 0.5 0.5; visual box size=0.5 0.5 0.5
Joints:
- removed joint 000_010
- removed joint 000_100
- removed joint 010_120
- removed joint 011_002
- removed joint 011_012
- removed joint 012_102
- removed joint 100_101
- removed joint 102_201
- removed joint 120_030
- removed joint 120_121
- removed joint 120_220
- removed joint 122_032
- removed joint 122_132
- removed joint 201_202
- removed joint 201_210
- removed joint 202_212
- added joint 000_001: type revolute, parent 000, child 001, origin xyz=0.25 0.0 0.5 rpy=0 0 0, axis 0 1 0, limit lower=-3.14159 upper=3.14159 effort=0.0 velocity=0.0
- added joint 001_101: type revolute, parent 001, child 101, origin xyz=0.0 -0.25 0.25 rpy=0 0 0, axis 0 0 1, limit lower=-3.14159 upper=3.14159 effort=0.0 velocity=0.0
- added joint 001_102: type continuous, parent 001, child 102, origin xyz=0.0 0.0 0.5 rpy=0 0 0, axis 0 1 0, limit lower=-3.14159 upper=3.14159 effort=0.0 velocity=0.0
- added joint 011_020: type revolute, parent 011, child 020, origin xyz=0.0 0.5 0.0 rpy=0 0 0, axis 1 0 0, limit lower=-3.14159 upper=3.14159 effort=0.0 velocity=0.0
- added joint 011_022: type continuous, parent 011, child 022, origin xyz=0.0 0.5 0.5 rpy=0 0 0, axis 1 0 0, limit lower=-3.14159 upper=3.14159 effort=0.0 velocity=0.0
- added joint 020_130: type continuous, parent 020, child 130, origin xyz=0.25 0.5 -0.25 rpy=0 0 0, axis 0 0 1, limit lower=-3.14159 upper=3.14159 effort=0.0 velocity=0.0
- added joint 022_121: type revolute, parent 022, child 121, origin xyz=0.25 0.25 0.0 rpy=0 0 0, axis 0 1 0, limit lower=-3.14159 upper=3.14159 effort=0.0 velocity=0.0
- added joint 102_202: type revolute, parent 102, child 202, origin xyz=0.5 -0.25 0.25 rpy=0 0 0, axis 0 0 1, limit lower=-3.14159 upper=3.14159 effort=0.0 velocity=0.0
- added joint 122_212: type revolute, parent 122, child 212, origin xyz=0.25 0.0 0.25 rpy=0 0 0, axis 0 0 1, limit lower=-3.14159 upper=3.14159 effort=0.0 velocity=0.0
- added joint 122_221: type revolute, parent 122, child 221, origin xyz=0.25 0.25 0.0 rpy=0 0 0, axis 0 1 0, limit lower=-3.14159 upper=3.14159 effort=0.0 velocity=0.0
- joint 000_011: type revolute -> continuous
- joint 121_122: axis 0 1 0 -> 1 0 0; origin xyz=-0.25 0.25 0.5 rpy=0 0 0 -> xyz=0.25 -0.25 0.0 rpy=0 0 0; type continuous -> revolute

File: files/body2.urdf (robot description, URDF)
Before this commit: robot robot, 23 links, 22 joints
Links:
- removed link 000
- removed link 001
- removed link 002
- removed link 021
- removed link 030
- removed link 032
- removed link 120
- removed link 122
- removed link 132
- removed link 211
- removed link 220
- added link 020, mass 1; collision box size=0.5 0.5 0.5; visual box size=0.5 0.5 0.5
- added link 100, mass 1; collision box size=0.5 0.5 0.5; visual box size=0.5 0.5 0.5
- added link 110, mass 1; collision box size=0.5 0.5 0.5; visual box size=0.5 0.5 0.5
- added link 111, mass 1; collision box size=0.5 0.5 0.5; visual box size=0.5 0.5 0.5
- added link 121, mass 1; collision box size=0.5 0.5 0.5; visual box size=0.5 0.5 0.5
- added link 131, mass 1; collision box size=0.5 0.5 0.5; visual box size=0.5 0.5 0.5
- added link 222, mass 1; collision box size=0.5 0.5 0.5; visual box size=0.5 0.5 0.5
Joints:
- removed joint 000_001
- removed joint 001_002
- removed joint 001_010
- removed joint 002_102
- removed joint 010_021
- removed joint 021_030
- removed joint 021_032
- removed joint 030_031
- removed joint 030_120
- removed joint 031_130
- removed joint 032_122
- removed joint 032_132
- removed joint 102_112
- removed joint 112_211
- removed joint 120_210
- removed joint 120_220
- removed joint 211_200
- removed joint 211_212
- removed joint 211_221
- removed joint 220_230
- removed joint 220_231
- added joint 010_020: type continuous, parent 010, child 020, origin xyz=0.0 0.75 0.5 rpy=0 0 0, axis 1 0 0, limit lower=-3.14159 upper=3.14159 effort=0.0 velocity=0.0
- added joint 010_100: type continuous, parent 010, child 100, origin xyz=0.25 0.25 0.25 rpy=0 0 0, axis 0 0 1, limit lower=-3.14159 upper=3.14159 effort=0.0 velocity=0.0
- added joint 010_111: type continuous, parent 010, child 111, origin xyz=0.25 0.5 0.5 rpy=0 0 0, axis 0 1 0, limit lower=-3.14159 upper=3.14159 effort=0.0 velocity=0.0
- added joint 020_031: type revolute, parent 020, child 031, origin xyz=0.0 0.5 0.0 rpy=0 0 0, axis 1 0 0, limit lower=-3.14159 upper=3.14159 effort=0.0 velocity=0.0
- added joint 020_110: type continuous, parent 020, child 110, origin xyz=0.25 0.0 -0.25 rpy=0 0 0, axis 0 0 1, limit lower=-3.14159 upper=3.14159 effort=0.0 velocity=0.0
- added joint 031_131: type revolute, parent 031, child 131, origin xyz=0.25 0.25 0.25 rpy=0 0 0, axis 0 1 0, limit lower=-3.14159 upper=3.14159 effort=0.0 velocity=0.0
- added joint 100_200: type continuous, parent 100, child 200, origin xyz=0.5 -0.5 0.0 rpy=0 0 0, axis 0 0 1, limit lower=-3.14159 upper=3.14159 effort=0.0 velocity=0.0
- added joint 110_121: type revolute, parent 110, child 121, origin xyz=0.25 0.0 0.25 rpy=0 0 0, axis 1 0 0, limit lower=-3.14159 upper=3.14159 effort=0.0 velocity=0.0
- added joint 111_112: type continuous, parent 111, child 112, origin xyz=0.25 -0.25 0.5 rpy=0 0 0, axis 1 0 0, limit lower=-3.14159 upper=3.14159 effort=0.0 velocity=0.0
- added joint 112_212: type revolute, parent 112, child 212, origin xyz=0.25 0.25 0.5 rpy=0 0 0, axis 0 1 0, limit lower=-3.14159 upper=3.14159 effort=0.0 velocity=0.0
- added joint 121_130: type continuous, parent 121, child 130, origin xyz=0.0 0.5 0.0 rpy=0 0 0, axis 1 0 0, limit lower=-3.14159 upper=3.14159 effort=0.0 velocity=0.0
- added joint 131_230: type continuous, parent 131, child 230, origin xyz=0.5 0.0 -0.25 rpy=0 0 0, axis 0 1 0, limit lower=-3.14159 upper=3.14159 effort=0.0 velocity=0.0
- added joint 200_210: type revolute, parent 200, child 210, origin xyz=0.0 0.5 0.0 rpy=0 0 0, axis 0 0 1, limit lower=-3.14159 upper=3.14159 effort=0.0 velocity=0.0
- added joint 202_102: type revolute, parent 202, child 102, origin xyz=0.0 -0.25 0.0 rpy=0 0 0, axis 0 1 0, limit lower=-3.14159 upper=3.14159 effort=0.0 velocity=0.0
- added joint 212_221: type revolute, parent 212, child 221, origin xyz=0.25 0.25 -0.5 rpy=0 0 0, axis 1 0 0, limit lower=-3.14159 upper=3.14159 effort=0.0 velocity=0.0
- added joint 221_222: type continuous, parent 221, child 222, origin xyz=0.0 0.25 0.0 rpy=0 0 0, axis 1 0 0, limit lower=-3.14159 upper=3.14159 effort=0.0 velocity=0.0
- added joint 222_231: type revolute, parent 222, child 231, origin xyz=0.0 0.25 0.0 rpy=0 0 0, axis 1 0 0, limit lower=-3.14159 upper=3.14159 effort=0.0 velocity=0.0
- joint 112_202: type revolute -> continuous

File: files/body3.urdf (robot description, URDF)
Before this commit: robot robot, 25 links, 24 joints
Links:
- removed link 000
- removed link 011
- removed link 012
- removed link 020
- removed link 022
- removed link 032
- removed link 110
- removed link 112
- removed link 121
- removed link 130
- removed link 200
- removed link 202
- removed link 210
- removed link 220
- removed link 232
- added link 132, mass 1; collision box size=0.5 0.5 0.5; visual box size=0.5 0.5 0.5
- added link 222, mass 1; collision box size=0.5 0.5 0.5; visual box size=0.5 0.5 0.5
- added link 230, mass 1; collision box size=0.5 0.5 0.5; visual box size=0.5 0.5 0.5
- added link 231, mass 1; collision box size=0.5 0.5 0.5; visual box size=0.5 0.5 0.5
Joints:
- removed joint 000_001
- removed joint 000_101
- removed joint 000_110
- removed joint 001_011
- removed joint 001_012
- removed joint 011_020
- removed joint 011_121
- removed joint 012_021
- removed joint 012_112
- removed joint 021_022
- removed joint 021_120
- removed joint 022_031
- removed joint 031_032
- removed joint 110_200
- removed joint 112_202
- removed joint 120_130
- removed joint 121_131
- removed joint 121_221
- removed joint 201_210
- removed joint 210_220
- removed joint 221_232
- added joint 002_101: type continuous, parent 002, child 101, origin xyz=0.25 0.25 0.0 rpy=0 0 0, axis 0 1 0, limit lower=-3.14159 upper=3.14159 effort=0.0 velocity=0.0
- added joint 021_031: type revolute, parent 021, child 031, origin xyz=0.0 0.25 0.25 rpy=0 0 0, axis 0 0 1, limit lower=-3.14159 upper=3.14159 effort=0.0 velocity=0.0
- added joint 120_021: type continuous, parent 120, child 021, origin xyz=-0.5 0.0 0.0 rpy=0 0 0, axis 0 1 0, limit lower=-3.14159 upper=3.14159 effort=0.0 velocity=0.0
- added joint 131_132: type continuous, parent 131, child 132, origin xyz=-0.5 0.0 0.5 rpy=0 0 0, axis 0 1 0, limit lower=-3.14159 upper=3.14159 effort=0.0 velocity=0.0
- added joint 212_221: type continuous, parent 212, child 221, origin xyz=0.0 0.5 0.0 rpy=0 0 0, axis 1 0 0, limit lower=-3.14159 upper=3.14159 effort=0.0 velocity=0.0
- added joint 221_120: type continuous, parent 221, child 120, origin xyz=-0.25 0.25 -0.5 rpy=0 0 0, axis 0 1 0, limit lower=-3.14159 upper=3.14159 effort=0.0 velocity=0.0
- added joint 221_222: type continuous, parent 221, child 222, origin xyz=0.0 0.0 0.0 rpy=0 0 0, axis 1 0 0, limit lower=-3.14159 upper=3.14159 effort=0.0 velocity=0.0
- added joint 221_230: type revolute, parent 221, child 230, origin xyz=0.0 0.5 -0.5 rpy=0 0 0, axis 1 0 0, limit lower=-3.14159 upper=3.14159 effort=0.0 velocity=0.0
- added joint 222_231: type revolute, parent 222, child 231, origin xyz=0.0 0.5 0.0 rpy=0 0 0, axis 1 0 0, limit lower=-3.14159 upper=3.14159 effort=0.0 velocity=0.0
- added joint 230_131: type continuous, parent 230, child 131, origin xyz=-0.25 0.25 0.0 rpy=0 0 0, axis 0 1 0, limit lower=-3.14159 upper=3.14159 effort=0.0 velocity=0.0
- joint 001_002: axis 0 1 0 -> 1 0 0; origin xyz=0.25 -0.25 0.5 rpy=0 0 0 -> xyz=0.0 -0.25 1.0 rpy=0 0 0; type continuous -> revolute
- joint 101_201: origin xyz=0.5 -0.25 0.25 rpy=0 0 0 -> xyz=0.5 0.25 -0.25 rpy=0 0 0
- joint 201_212: origin xyz=0.25 0.5 0.25 rpy=0 0 0 -> xyz=0.25 0.0 0.25 rpy=0 0 0; type continuous -> revolute

File: files/body4.urdf (robot description, URDF)
Before this commit: robot robot, 21 links, 20 joints
Links:
- removed link 010
- removed link 030
- removed link 032
- removed link 132
- removed link 202
- removed link 231
- added link 021, mass 1; collision box size=0.5 0.5 0.5; visual box size=0.5 0.5 0.5
- added link 022, mass 1; collision box size=0.5 0.5 0.5; visual box size=0.5 0.5 0.5
- added link 031, mass 1; collision box size=0.5 0.5 0.5; visual box size=0.5 0.5 0.5
- added link 211, mass 1; collision box size=0.5 0.5 0.5; visual box size=0.5 0.5 0.5
- added link 220, mass 1; collision box size=0.5 0.5 0.5; visual box size=0.5 0.5 0.5
- added link 230, mass 1; collision box size=0.5 0.5 0.5; visual box size=0.5 0.5 0.5
Joints:
- removed joint 001_010
- removed joint 001_012
- removed joint 011_112
- removed joint 020_030
- removed joint 100_200
- removed joint 101_111
- removed joint 101_202
- removed joint 111_120
- removed joint 112_212
- removed joint 131_032
- removed joint 131_132
- removed joint 131_231
- removed joint 231_232
- added joint 011_012: type continuous, parent 011, child 012, origin xyz=-0.25 0.25 0.5 rpy=0 0 0, axis 0 1 0, limit lower=-3.14159 upper=3.14159 effort=0.0 velocity=0.0
- added joint 012_112: type continuous, parent 012, child 112, origin xyz=0.5 -0.25 0.25 rpy=0 0 0, axis 0 0 1, limit lower=-3.14159 upper=3.14159 effort=0.0 velocity=0.0
- added joint 020_021: type revolute, parent 020, child 021, origin xyz=0.25 0.25 0.0 rpy=0 0 0, axis 0 1 0, limit lower=-3.14159 upper=3.14159 effort=0.0 velocity=0.0
- added joint 021_022: type continuous, parent 021, child 022, origin xyz=-0.25 0.0 0.5 rpy=0 0 0, axis 0 1 0, limit lower=-3.14159 upper=3.14159 effort=0.0 velocity=0.0
- added joint 021_031: type continuous, parent 021, child 031, origin xyz=-0.25 0.25 0.0 rpy=0 0 0, axis 1 0 0, limit lower=-3.14159 upper=3.14159 effort=0.0 velocity=0.0
- added joint 021_120: type continuous, parent 021, child 120, origin xyz=0.0 0.0 0.0 rpy=0 0 0, axis 0 1 0, limit lower=-3.14159 upper=3.14159 effort=0.0 velocity=0.0
- added joint 101_200: type revolute, parent 101, child 200, origin xyz=0.5 -0.25 -0.25 rpy=0 0 0, axis 0 1 0, limit lower=-3.14159 upper=3.14159 effort=0.0 velocity=0.0
- added joint 101_211: type continuous, parent 101, child 211, origin xyz=0.5 0.0 0.0 rpy=0 0 0, axis 0 0 1, limit lower=-3.14159 upper=3.14159 effort=0.0 velocity=0.0
- added joint 102_111: type revolute, parent 102, child 111, origin xyz=0.0 0.5 0.0 rpy=0 0 0, axis 1 0 0, limit lower=-3.14159 upper=3.14159 effort=0.0 velocity=0.0
- added joint 120_220: type continuous, parent 120, child 220, origin xyz=0.5 0.25 -0.25 rpy=0 0 0, axis 0 0 1, limit lower=-3.14159 upper=3.14159 effort=0.0 velocity=0.0
- added joint 131_230: type revolute, parent 131, child 230, origin xyz=0.25 0.25 0.0 rpy=0 0 0, axis 0 1 0, limit lower=-3.14159 upper=3.14159 effort=0.0 velocity=0.0
- added joint 131_232: type continuous, parent 131, child 232, origin xyz=0.25 0.25 0.5 rpy=0 0 0, axis 0 1 0, limit lower=-3.14159 upper=3.14159 effort=0.0 velocity=0.0
- added joint 211_212: type continuous, parent 211, child 212, origin xyz=0.5 0.25 0.25 rpy=0 0 0, axis 0 1 0, limit lower=-3.14159 upper=3.14159 effort=0.0 velocity=0.0
- joint 000_001: axis 1 0 0 -> 0 1 0; origin xyz=0.0 0.25 0.5 rpy=0 0 0 -> xyz=0.0 0.0 0.5 rpy=0 0 0
- joint 011_101: type revolute -> continuous
- joint 101_102: origin xyz=0.25 -0.25 0.25 rpy=0 0 0 -> xyz=0.25 -0.5 0.25 rpy=0 0 0; type continuous -> revolute
- joint 120_131: origin xyz=0.0 0.5 0.0 rpy=0 0 0 -> xyz=0.25 0.25 0.0 rpy=0 0 0
