Commit message: analysis

File: files/body0.urdf (robot description, URDF)
Before this commit: robot robot, 20 links, 19 joints
Links:
- removed link 000
- removed link 001
- removed link 011
- removed link 020
- removed link 021
- removed link 022
- removed link 110
- removed link 111
- removed link 202
- removed link 212
- removed link 221
- removed link 230
- added link 002, mass 1; collision box size=0.5 0.5 0.5; visual box size=0.5 0.5 0.5
- added link 010, mass 1; collision box size=0.5 0.5 0.5; visual box size=0.5 0.5 0.5
- added link 101, mass 1; collision box size=0.5 0.5 0.5; visual box size=0.5 0.5 0.5
- added link 112, mass 1; collision box size=0.5 0.5 0.5; visual box size=0.5 0.5 0.5
- added link 122, mass 1; collision box size=0.5 0.5 0.5; visual box size=0.5 0.5 0.5
- added link 131, mass 1; collision box size=0.5 0.5 0.5; visual box size=0.5 0.5 0.5
- added link 201, mass 1; collision box size=0.5 0.5 0.5; visual box size=0.5 0.5 0.5
- added link 231, mass 1; collision box size=0.5 0.5 0.5; visual box size=0.5 0.5 0.5
- added link 232, mass 1; collision box size=0.5 0.5 0.5; visual box size=0.5 0.5 0.5
Joints:
- removed joint 000_001
- removed joint 000_011
- removed joint 000_100
- removed joint 000_110
- removed joint 011_020
- removed joint 011_021
- removed joint 020_030
- removed joint 020_031
- removed joint 020_121
- removed joint 020_130
- removed joint 021_022
- removed joint 031_032
- removed joint 031_132
- removed joint 100_111
- removed joint 111_212
- removed joint 111_221
- removed joint 212_202
- removed joint 221_230
- added joint 002_101: type revolute, parent 002, child 101, origin xyz=0.25 0.0 1.0 rpy=0 0 0, axis 0 1 0, limit lower=-3.14159 upper=3.14159 effort=0.0 velocity=0.0
- added joint 100_010: type continuous, parent 100, child 010, origin xyz=0.0 0.25 -0.25 rpy=0 0 0, axis 0 0 1, limit lower=-3.14159 upper=3.14159 effort=0.0 velocity=0.0
- added joint 101_100: type revolute, parent 101, child 100, origin xyz=0.0 0.0 -0.5 rpy=0 0 0, axis 0 1 0, limit lower=-3.14159 upper=3.14159 effort=0.0 velocity=0.0
- added joint 101_112: type revolute, parent 101, child 112, origin xyz=0.25 0.25 0.0 rpy=0 0 0, axis 1 0 0, limit lower=-3.14159 upper=3.14159 effort=0.0 velocity=0.0
- added joint 101_201: type revolute, parent 101, child 201, origin xyz=0.5 0.25 -0.25 rpy=0 0 0, axis 0 0 1, limit lower=-3.14159 upper=3.14159 effort=0.0 velocity=0.0
- added joint 112_121: type continuous, parent 112, child 121, origin xyz=0.0 0.5 0.0 rpy=0 0 0, axis 1 0 0, limit lower=-3.14159 upper=3.14159 effort=0.0 velocity=0.0
- added joint 112_122: type continuous, parent 112, child 122, origin xyz=0.25 0.5 0.25 rpy=0 0 0, axis 0 0 1, limit lower=-3.14159 upper=3.14159 effort=0.0 velocity=0.0
- added joint 121_130: type revolute, parent 121, child 130, origin xyz=0.0 0.5 -0.5 rpy=0 0 0, axis 1 0 0, limit lower=-3.14159 upper=3.14159 effort=0.0 velocity=0.0
- added joint 122_032: type revolute, parent 122, child 032, origin xyz=-0.5 0.5 0.0 rpy=0 0 0, axis 0 0 1, limit lower=-3.14159 upper=3.14159 effort=0.0 velocity=0.0
- added joint 122_131: type continuous, parent 122, child 131, origin xyz=-0.25 0.5 -0.25 rpy=0 0 0, axis 1 0 0, limit lower=-3.14159 upper=3.14159 effort=0.0 velocity=0.0
- added joint 122_232: type continuous, parent 122, child 232, origin xyz=0.0 0.5 0.0 rpy=0 0 0, axis 0 0 1, limit lower=-3.14159 upper=3.14159 effort=0.0 velocity=0.0
- added joint 131_030: type continuous, parent 131, child 030, origin xyz=-0.25 0.25 -0.5 rpy=0 0 0, axis 0 1 0, limit lower=-3.14159 upper=3.14159 effort=0.0 velocity=0.0
- added joint 131_031: type revolute, parent 131, child 031, origin xyz=-0.25 0.5 -0.25 rpy=0 0 0, axis 0 0 1, limit lower=-3.14159 upper=3.14159 effort=0.0 velocity=0.0
- added joint 131_132: type continuous, parent 131, child 132, origin xyz=0.0 0.0 0.0 rpy=0 0 0, axis 1 0 0, limit lower=-3.14159 upper=3.14159 effort=0.0 velocity=0.0
- added joint 131_231: type continuous, parent 131, child 231, origin xyz=0.25 0.25 -0.25 rpy=0 0 0, axis 0 0 1, limit lower=-3.14159 upper=3.14159 effort=0.0 velocity=0.0
- joint 130_220: origin xyz=0.5 0.0 0.0 rpy=0 0 0 -> xyz=0.25 0.0 -0.25 rpy=0 0 0; type continuous -> revolute

File: files/body1.urdf (robot description, URDF)
Before this commit: robot robot, 13 links, 12 joints
Links:
- removed link 001
- removed link 020
- removed link 101
- removed link 122
- removed link 130
- removed link 202
- removed link 212
- removed link 221
- added link 010, mass 1; collision box size=0.5 0.5 0.5; visual box size=0.5 0.5 0.5
- added link 012, mass 1; collision box size=0.5 0.5 0.5; visual box size=0.5 0.5 0.5
- added link 030, mass 1; collision box size=0.5 0.5 0.5; visual box size=0.5 0.5 0.5
- added link 031, mass 1; collision box size=0.5 0.5 0.5; visual box size=0.5 0.5 0.5
- added link 032, mass 1; collision box size=0.5 0.5 0.5; visual box size=0.5 0.5 0.5
- added link 112, mass 1; collision box size=0.5 0.5 0.5; visual box size=0.5 0.5 0.5
- added link 120, mass 1; collision box size=0.5 0.5 0.5; visual box size=0.5 0.5 0.5
- added link 131, mass 1; collision box size=0.5 0.5 0.5; visual box size=0.5 0.5 0.5
- added link 132, mass 1; collision box size=0.5 0.5 0.5; visual box size=0.5 0.5 0.5
- added link 200, mass 1; collision box size=0.5 0.5 0.5; visual box size=0.5 0.5 0.5
- added link 201, mass 1; collision box size=0.5 0.5 0.5; visual box size=0.5 0.5 0.5
- added link 210, mass 1; collision box size=0.5 0.5 0.5; visual box size=0.5 0.5 0.5
- added link 220, mass 1; collision box size=0.5 0.5 0.5; visual box size=0.5 0.5 0.5
- added link 230, mass 1; collision box size=0.5 0.5 0.5; visual box size=0.5 0.5 0.5
- added link 232, mass 1; collision box size=0.5 0.5 0.5; visual box size=0.5 0.5 0.5
Joints:
- removed joint 000_001
- removed joint 001_101
- removed joint 001_102
- removed joint 011_020
- removed joint 020_130
- removed joint 022_121
- removed joint 102_202
- removed joint 121_122
- removed joint 122_212
- removed joint 122_221
- added joint 011_010: type continuous, parent 011, child 010, origin xyz=0.0 0.5 0.0 rpy=0 0 0, axis 1 0 0, limit lower=-3.14159 upper=3.14159 effort=0.0 velocity=0.0
- added joint 011_012: type revolute, parent 011, child 012, origin xyz=0.25 0.25 0.5 rpy=0 0 0, axis 0 1 0, limit lower=-3.14159 upper=3.14159 effort=0.0 velocity=0.0
- added joint 012_102: type revolute, parent 012, child 102, origin xyz=0.0 -0.25 0.25 rpy=0 0 0, axis 0 0 1, limit lower=-3.14159 upper=3.14159 effort=0.0 velocity=0.0
- added joint 012_112: type continuous, parent 012, child 112, origin xyz=0.0 -0.25 0.25 rpy=0 0 0, axis 0 0 1, limit lower=-3.14159 upper=3.14159 effort=0.0 velocity=0.0
- added joint 022_031: type continuous, parent 022, child 031, origin xyz=0.0 0.5 0.0 rpy=0 0 0, axis 1 0 0, limit lower=-3.14159 upper=3.14159 effort=0.0 velocity=0.0
- added joint 022_032: type revolute, parent 022, child 032, origin xyz=0.0 0.5 0.25 rpy=0 0 0, axis 0 0 1, limit lower=-3.14159 upper=3.14159 effort=0.0 velocity=0.0
- added joint 031_030: type continuous, parent 031, child 030, origin xyz=0.0 0.25 -0.5 rpy=0 0 0, axis 0 1 0, limit lower=-3.14159 upper=3.14159 effort=0.0 velocity=0.0
- added joint 031_121: type revolute, parent 031, child 121, origin xyz=0.25 0.0 -0.25 rpy=0 0 0, axis 0 0 1, limit lower=-3.14159 upper=3.14159 effort=0.0 velocity=0.0
- added joint 031_132: type revolute, parent 031, child 132, origin xyz=0.25 0.25 0.0 rpy=0 0 0, axis 0 1 0, limit lower=-3.14159 upper=3.14159 effort=0.0 velocity=0.0
- added joint 032_131: type continuous, parent 032, child 131, origin xyz=0.25 0.25 -0.25 rpy=0 0 0, axis 0 1 0, limit lower=-3.14159 upper=3.14159 effort=0.0 velocity=0.0
- added joint 102_201: type revolute, parent 102, child 201, origin xyz=0.5 -0.25 -0.25 rpy=0 0 0, axis 0 1 0, limit lower=-3.14159 upper=3.14159 effort=0.0 velocity=0.0
- added joint 121_120: type continuous, parent 121, child 120, origin xyz=0.5 -0.25 -0.25 rpy=0 0 0, axis 0 1 0, limit lower=-3.14159 upper=3.14159 effort=0.0 velocity=0.0
- added joint 131_230: type revolute, parent 131, child 230, origin xyz=0.5 0.0 -0.5 rpy=0 0 0, axis 0 1 0, limit lower=-3.14159 upper=3.14159 effort=0.0 velocity=0.0
- added joint 131_232: type revolute, parent 131, child 232, origin xyz=0.5 0.0 0.0 rpy=0 0 0, axis 0 1 0, limit lower=-3.14159 upper=3.14159 effort=0.0 velocity=0.0
- added joint 201_200: type revolute, parent 201, child 200, origin xyz=0.5 0.0 -0.5 rpy=0 0 0, axis 0 1 0, limit lower=-3.14159 upper=3.14159 effort=0.0 velocity=0.0
- added joint 201_210: type revolute, parent 201, child 210, origin xyz=0.25 0.25 -0.5 rpy=0 0 0, axis 1 0 0, limit lower=-3.14159 upper=3.14159 effort=0.0 velocity=0.0
- added joint 210_220: type revolute, parent 210, child 220, origin xyz=0.0 0.5 0.0 rpy=0 0 0, axis 1 0 0, limit lower=-3.14159 upper=3.14159 effort=0.0 velocity=0.0
- joint 011_022: type continuous -> revolute

File: files/body2.urdf (robot description, URDF)
Before this commit: robot robot, 19 links, 18 joints
Links:
- removed link 010
- removed link 020
- removed link 031
- removed link 210
- removed link 212
- removed link 221
- added link 002, mass 1; collision box size=0.5 0.5 0.5; visual box size=0.5 0.5 0.5
- added link 011, mass 1; collision box size=0.5 0.5 0.5; visual box size=0.5 0.5 0.5
- added link 012, mass 1; collision box size=0.5 0.5 0.5; visual box size=0.5 0.5 0.5
- added link 021, mass 1; collision box size=0.5 0.5 0.5; visual box size=0.5 0.5 0.5
- added link 030, mass 1; collision box size=0.5 0.5 0.5; visual box size=0.5 0.5 0.5
- added link 032, mass 1; collision box size=0.5 0.5 0.5; visual box size=0.5 0.5 0.5
- added link 101, mass 1; collision box size=0.5 0.5 0.5; visual box size=0.5 0.5 0.5
- added link 122, mass 1; collision box size=0.5 0.5 0.5; visual box size=0.5 0.5 0.5
- added link 211, mass 1; collision box size=0.5 0.5 0.5; visual box size=0.5 0.5 0.5
- added link 220, mass 1; collision box size=0.5 0.5 0.5; visual box size=0.5 0.5 0.5
- added link 232, mass 1; collision box size=0.5 0.5 0.5; visual box size=0.5 0.5 0.5
Joints:
- removed joint 010_020
- removed joint 010_100
- removed joint 010_111
- removed joint 020_031
- removed joint 020_110
- removed joint 031_131
- removed joint 100_200
- removed joint 110_121
- removed joint 111_112
- removed joint 112_212
- removed joint 121_130
- removed joint 131_230
- removed joint 200_210
- removed joint 202_102
- removed joint 212_221
- removed joint 221_222
- added joint 002_011: type continuous, parent 002, child 011, origin xyz=0.0 0.25 1.0 rpy=0 0 0, axis 1 0 0, limit lower=-3.14159 upper=3.14159 effort=0.0 velocity=0.0
- added joint 002_101: type revolute, parent 002, child 101, origin xyz=0.25 0.0 1.0 rpy=0 0 0, axis 0 1 0, limit lower=-3.14159 upper=3.14159 effort=0.0 velocity=0.0
- added joint 011_012: type revolute, parent 011, child 012, origin xyz=0.0 0.0 0.0 rpy=0 0 0, axis 1 0 0, limit lower=-3.14159 upper=3.14159 effort=0.0 velocity=0.0
- added joint 011_021: type revolute, parent 011, child 021, origin xyz=0.0 0.5 -0.5 rpy=0 0 0, axis 1 0 0, limit lower=-3.14159 upper=3.14159 effort=0.0 velocity=0.0
- added joint 011_110: type continuous, parent 011, child 110, origin xyz=0.25 0.25 -0.5 rpy=0 0 0, axis 0 1 0, limit lower=-3.14159 upper=3.14159 effort=0.0 velocity=0.0
- added joint 011_112: type continuous, parent 011, child 112, origin xyz=0.25 0.25 0.0 rpy=0 0 0, axis 0 1 0, limit lower=-3.14159 upper=3.14159 effort=0.0 velocity=0.0
- added joint 021_030: type revolute, parent 021, child 030, origin xyz=0.0 0.5 0.0 rpy=0 0 0, axis 1 0 0, limit lower=-3.14159 upper=3.14159 effort=0.0 velocity=0.0
- added joint 021_032: type continuous, parent 021, child 032, origin xyz=0.0 0.5 0.5 rpy=0 0 0, axis 1 0 0, limit lower=-3.14159 upper=3.14159 effort=0.0 velocity=0.0
- added joint 021_122: type continuous, parent 021, child 122, origin xyz=0.25 0.25 0.5 rpy=0 0 0, axis 0 1 0, limit lower=-3.14159 upper=3.14159 effort=0.0 velocity=0.0
- added joint 030_130: type revolute, parent 030, child 130, origin xyz=0.25 0.25 0.0 rpy=0 0 0, axis 0 1 0, limit lower=-3.14159 upper=3.14159 effort=0.0 velocity=0.0
- added joint 030_131: type continuous, parent 030, child 131, origin xyz=0.25 0.25 0.0 rpy=0 0 0, axis 0 1 0, limit lower=-3.14159 upper=3.14159 effort=0.0 velocity=0.0
- added joint 101_102: type continuous, parent 101, child 102, origin xyz=0.5 0.0 0.0 rpy=0 0 0, axis 0 1 0, limit lower=-3.14159 upper=3.14159 effort=0.0 velocity=0.0
- added joint 110_111: type revolute, parent 110, child 111, origin xyz=0.25 0.0 0.0 rpy=0 0 0, axis 1 0 0, limit lower=-3.14159 upper=3.14159 effort=0.0 velocity=0.0
- added joint 110_200: type revolute, parent 110, child 200, origin xyz=0.5 -0.25 -0.25 rpy=0 0 0, axis 0 0 1, limit lower=-3.14159 upper=3.14159 effort=0.0 velocity=0.0
- added joint 112_211: type continuous, parent 112, child 211, origin xyz=0.5 0.0 0.0 rpy=0 0 0, axis 0 1 0, limit lower=-3.14159 upper=3.14159 effort=0.0 velocity=0.0
- added joint 112_222: type continuous, parent 112, child 222, origin xyz=0.5 0.25 0.25 rpy=0 0 0, axis 0 0 1, limit lower=-3.14159 upper=3.14159 effort=0.0 velocity=0.0
- added joint 130_230: type continuous, parent 130, child 230, origin xyz=0.5 -0.25 -0.25 rpy=0 0 0, axis 0 0 1, limit lower=-3.14159 upper=3.14159 effort=0.0 velocity=0.0
- added joint 131_121: type continuous, parent 131, child 121, origin xyz=0.5 -0.25 0.25 rpy=0 0 0, axis 0 0 1, limit lower=-3.14159 upper=3.14159 effort=0.0 velocity=0.0
- added joint 200_100: type revolute, parent 200, child 100, origin xyz=0.0 -0.25 -0.25 rpy=0 0 0, axis 0 1 0, limit lower=-3.14159 upper=3.14159 effort=0.0 velocity=0.0
- added joint 211_220: type continuous, parent 211, child 220, origin xyz=0.25 0.25 -0.5 rpy=0 0 0, axis 1 0 0, limit lower=-3.14159 upper=3.14159 effort=0.0 velocity=0.0
- added joint 231_232: type continuous, parent 231, child 232, origin xyz=-0.25 0.25 0.0 rpy=0 0 0, axis 0 1 0, limit lower=-3.14159 upper=3.14159 effort=0.0 velocity=0.0
- joint 112_202: origin xyz=0.25 0.0 0.25 rpy=0 0 0 -> xyz=0.5 -0.25 0.25 rpy=0 0 0; type continuous -> revolute
- joint 222_231: origin xyz=0.0 0.25 0.0 rpy=0 0 0 -> xyz=0.25 0.5 -0.25 rpy=0 0 0; type revolute -> continuous

File: files/body6.urdf (robot description, URDF)
Before this commit: robot robot, 18 links, 17 joints
Links:
- removed link 010
- removed link 120
- removed link 212
- added link 112, mass 1; collision box size=0.5 0.5 0.5; visual box size=0.5 0.5 0.5
- added link 122, mass 1; collision box size=0.5 0.5 0.5; visual box size=0.5 0.5 0.5
- added link 210, mass 1; collision box size=0.5 0.5 0.5; visual box size=0.5 0.5 0.5
Joints:
- removed joint 000_010
- removed joint 010_011
- removed joint 010_120
- removed joint 120_230
- removed joint 211_212
- added joint 000_011: type revolute, parent 000, child 011, origin xyz=0.0 0.25 0.5 rpy=0 0 0, axis 1 0 0, limit lower=-3.14159 upper=3.14159 effort=0.0 velocity=0.0
- added joint 012_112: type continuous, parent 012, child 112, origin xyz=0.25 -0.25 0.25 rpy=0 0 0, axis 0 0 1, limit lower=-3.14159 upper=3.14159 effort=0.0 velocity=0.0
- added joint 022_122: type revolute, parent 022, child 122, origin xyz=0.25 0.25 0.0 rpy=0 0 0, axis 0 1 0, limit lower=-3.14159 upper=3.14159 effort=0.0 velocity=0.0
- added joint 131_230: type continuous, parent 131, child 230, origin xyz=0.5 0.0 -0.5 rpy=0 0 0, axis 0 1 0, limit lower=-3.14159 upper=3.14159 effort=0.0 velocity=0.0
- added joint 201_210: type revolute, parent 201, child 210, origin xyz=0.0 0.0 -0.25 rpy=0 0 0, axis 1 0 0, limit lower=-3.14159 upper=3.14159 effort=0.0 velocity=0.0
- joint 011_012: origin xyz=0.25 0.0 0.5 rpy=0 0 0 -> xyz=0.0 0.25 0.5 rpy=0 0 0
- joint 011_022: origin xyz=0.25 0.25 0.5 rpy=0 0 0 -> xyz=0.0 0.5 0.5 rpy=0 0 0

File: files/body8.urdf (robot description, URDF)
Before this commit: robot robot, 19 links, 18 joints
Links:
- removed link 001
- removed link 010
- removed link 020
- removed link 021
- removed link 032
- removed link 100
- removed link 111
- removed link 132
- removed link 200
- removed link 201
- removed link 210
- removed link 220
- removed link 221
- removed link 222
- added link 011, mass 1; collision box size=0.5 0.5 0.5; visual box size=0.5 0.5 0.5
- added link 022, mass 1; collision box size=0.5 0.5 0.5; visual box size=0.5 0.5 0.5
- added link 121, mass 1; collision box size=0.5 0.5 0.5; visual box size=0.5 0.5 0.5
- added link 122, mass 1; collision box size=0.5 0.5 0.5; visual box size=0.5 0.5 0.5
- added link 130, mass 1; collision box size=0.5 0.5 0.5; visual box size=0.5 0.5 0.5
- added link 131, mass 1; collision box size=0.5 0.5 0.5; visual box size=0.5 0.5 0.5
- added link 211, mass 1; collision box size=0.5 0.5 0.5; visual box size=0.5 0.5 0.5
- added link 212, mass 1; collision box size=0.5 0.5 0.5; visual box size=0.5 0.5 0.5
Joints:
- removed joint 001_010
- removed joint 001_012
- removed joint 010_020
- removed joint 010_021
- removed joint 010_100
- removed joint 012_111
- removed joint 012_112
- removed joint 020_031
- removed joint 031_032
- removed joint 032_132
- removed joint 100_200
- removed joint 112_222
- removed joint 200_201
- removed joint 201_210
- removed joint 210_220
- removed joint 220_221
- removed joint 220_230
- added joint 012_022: type continuous, parent 012, child 022, origin xyz=0.0 0.75 1.0 rpy=0 0 0, axis 1 0 0, limit lower=-3.14159 upper=3.14159 effort=0.0 velocity=0.0
- added joint 022_031: type revolute, parent 022, child 031, origin xyz=0.0 0.5 0.0 rpy=0 0 0, axis 1 0 0, limit lower=-3.14159 upper=3.14159 effort=0.0 velocity=0.0
- added joint 022_112: type continuous, parent 022, child 112, origin xyz=0.25 0.0 0.25 rpy=0 0 0, axis 0 0 1, limit lower=-3.14159 upper=3.14159 effort=0.0 velocity=0.0
- added joint 022_121: type revolute, parent 022, child 121, origin xyz=0.25 0.25 0.0 rpy=0 0 0, axis 0 1 0, limit lower=-3.14159 upper=3.14159 effort=0.0 velocity=0.0
- added joint 112_011: type continuous, parent 112, child 011, origin xyz=0.0 -0.25 -0.25 rpy=0 0 0, axis 0 1 0, limit lower=-3.14159 upper=3.14159 effort=0.0 velocity=0.0
- added joint 112_211: type revolute, parent 112, child 211, origin xyz=0.5 -0.25 -0.25 rpy=0 0 0, axis 0 1 0, limit lower=-3.14159 upper=3.14159 effort=0.0 velocity=0.0
- added joint 121_122: type continuous, parent 121, child 122, origin xyz=0.5 0.0 0.0 rpy=0 0 0, axis 0 1 0, limit lower=-3.14159 upper=3.14159 effort=0.0 velocity=0.0
- added joint 121_130: type continuous, parent 121, child 130, origin xyz=0.25 0.25 -0.5 rpy=0 0 0, axis 1 0 0, limit lower=-3.14159 upper=3.14159 effort=0.0 velocity=0.0
- added joint 130_131: type continuous, parent 130, child 131, origin xyz=-0.25 0.25 0.0 rpy=0 0 0, axis 0 1 0, limit lower=-3.14159 upper=3.14159 effort=0.0 velocity=0.0
- added joint 130_230: type revolute, parent 130, child 230, origin xyz=0.25 0.5 -0.25 rpy=0 0 0, axis 0 0 1, limit lower=-3.14159 upper=3.14159 effort=0.0 velocity=0.0
- added joint 211_212: type continuous, parent 211, child 212, origin xyz=0.25 -0.25 0.0 rpy=0 0 0, axis 1 0 0, limit lower=-3.14159 upper=3.14159 effort=0.0 velocity=0.0
- joint 112_202: origin xyz=0.5 -0.25 0.25 rpy=0 0 0 -> xyz=0.5 -0.5 0.0 rpy=0 0 0; type revolute -> continuous

File: files/body9.urdf (robot description, URDF)
Before this commit: robot robot, 14 links, 13 joints
Links:
- removed link 031
- removed link 112
- removed link 210
- added link 020, mass 1; collision box size=0.5 0.5 0.5; visual box size=0.5 0.5 0.5
- added link 022, mass 1; collision box size=0.5 0.5 0.5; visual box size=0.5 0.5 0.5
- added link 221, mass 1; collision box size=0.5 0.5 0.5; visual box size=0.5 0.5 0.5
Joints:
- removed joint 002_112
- removed joint 021_031
- removed joint 112_121
- removed joint 112_211
- removed joint 201_210
- added joint 021_020: type continuous, parent 021, child 020, origin xyz=0.0 0.5 -0.5 rpy=0 0 0, axis 1 0 0, limit lower=-3.14159 upper=3.14159 effort=0.0 velocity=0.0
- added joint 021_121: type continuous, parent 021, child 121, origin xyz=0.25 0.0 -0.25 rpy=0 0 0, axis 0 0 1, limit lower=-3.14159 upper=3.14159 effort=0.0 velocity=0.0
- added joint 121_022: type continuous, parent 121, child 022, origin xyz=0.0 0.25 0.25 rpy=0 0 0, axis 0 1 0, limit lower=-3.14159 upper=3.14159 effort=0.0 velocity=0.0
- added joint 121_221: type revolute, parent 121, child 221, origin xyz=0.5 0.25 0.0 rpy=0 0 0, axis 0 1 0, limit lower=-3.14159 upper=3.14159 effort=0.0 velocity=0.0
- added joint 201_211: type revolute, parent 201, child 211, origin xyz=0.5 0.25 -0.25 rpy=0 0 0, axis 0 0 1, limit lower=-3.14159 upper=3.14159 effort=0.0 velocity=0.0
- joint 211_220: origin xyz=0.25 0.25 -0.5 rpy=0 0 0 -> xyz=-0.25 0.5 -0.25 rpy=0 0 0
