Commit message: diagrams

File: files/body0.urdf (robot description, URDF)
Before this commit: robot robot, 17 links, 16 joints
Links:
- removed link 002
- removed link 030
- removed link 031
- removed link 032
- removed link 100
- removed link 132
- removed link 201
- removed link 231
- removed link 232
- added link 000, mass 1; collision box size=0.5 0.5 0.5; visual box size=0.5 0.5 0.5
- added link 011, mass 1; collision box size=0.5 0.5 0.5; visual box size=0.5 0.5 0.5
- added link 012, mass 1; collision box size=0.5 0.5 0.5; visual box size=0.5 0.5 0.5
- added link 020, mass 1; collision box size=0.5 0.5 0.5; visual box size=0.5 0.5 0.5
- added link 022, mass 1; collision box size=0.5 0.5 0.5; visual box size=0.5 0.5 0.5
- added link 110, mass 1; collision box size=0.5 0.5 0.5; visual box size=0.5 0.5 0.5
- added link 202, mass 1; collision box size=0.5 0.5 0.5; visual box size=0.5 0.5 0.5
- added link 212, mass 1; collision box size=0.5 0.5 0.5; visual box size=0.5 0.5 0.5
- added link 222, mass 1; collision box size=0.5 0.5 0.5; visual box size=0.5 0.5 0.5
- added link 230, mass 1; collision box size=0.5 0.5 0.5; visual box size=0.5 0.5 0.5
Joints:
- removed joint 002_101
- removed joint 100_010
- removed joint 101_100
- removed joint 101_201
- removed joint 112_121
- removed joint 112_122
- removed joint 121_130
- removed joint 122_032
- removed joint 122_131
- removed joint 122_232
- removed joint 131_030
- removed joint 131_031
- removed joint 131_132
- removed joint 131_231
- added joint 000_010: type continuous, parent 000, child 010, origin xyz=0.25 0.25 0.25 rpy=0 0 0, axis 0 0 1, limit lower=-3.14159 upper=3.14159 effort=0.0 velocity=0.0
- added joint 000_101: type revolute, parent 000, child 101, origin xyz=0.25 0.0 0.5 rpy=0 0 0, axis 0 1 0, limit lower=-3.14159 upper=3.14159 effort=0.0 velocity=0.0
- added joint 010_011: type continuous, parent 010, child 011, origin xyz=-0.25 0.5 0.25 rpy=0 0 0, axis 1 0 0, limit lower=-3.14159 upper=3.14159 effort=0.0 velocity=0.0
- added joint 010_110: type revolute, parent 010, child 110, origin xyz=0.0 0.25 0.0 rpy=0 0 0, axis 0 0 1, limit lower=-3.14159 upper=3.14159 effort=0.0 velocity=0.0
- added joint 011_012: type revolute, parent 011, child 012, origin xyz=0.0 -0.5 0.5 rpy=0 0 0, axis 1 0 0, limit lower=-3.14159 upper=3.14159 effort=0.0 velocity=0.0
- added joint 011_020: type continuous, parent 011, child 020, origin xyz=0.0 0.0 0.0 rpy=0 0 0, axis 1 0 0, limit lower=-3.14159 upper=3.14159 effort=0.0 velocity=0.0
- added joint 011_022: type revolute, parent 011, child 022, origin xyz=0.0 0.0 0.5 rpy=0 0 0, axis 1 0 0, limit lower=-3.14159 upper=3.14159 effort=0.0 velocity=0.0
- added joint 020_130: type revolute, parent 020, child 130, origin xyz=0.25 0.5 -0.25 rpy=0 0 0, axis 0 0 1, limit lower=-3.14159 upper=3.14159 effort=0.0 velocity=0.0
- added joint 022_121: type revolute, parent 022, child 121, origin xyz=0.25 0.25 0.0 rpy=0 0 0, axis 0 1 0, limit lower=-3.14159 upper=3.14159 effort=0.0 velocity=0.0
- added joint 112_202: type continuous, parent 112, child 202, origin xyz=0.25 0.0 0.25 rpy=0 0 0, axis 0 0 1, limit lower=-3.14159 upper=3.14159 effort=0.0 velocity=0.0
- added joint 112_212: type revolute, parent 112, child 212, origin xyz=0.25 0.25 0.0 rpy=0 0 0, axis 0 1 0, limit lower=-3.14159 upper=3.14159 effort=0.0 velocity=0.0
- added joint 121_122: type revolute, parent 121, child 122, origin xyz=0.25 0.0 0.0 rpy=0 0 0, axis 0 1 0, limit lower=-3.14159 upper=3.14159 effort=0.0 velocity=0.0
- added joint 121_131: type continuous, parent 121, child 131, origin xyz=0.5 0.25 -0.25 rpy=0 0 0, axis 0 0 1, limit lower=-3.14159 upper=3.14159 effort=0.0 velocity=0.0
- added joint 121_222: type revolute, parent 121, child 222, origin xyz=0.5 0.0 0.0 rpy=0 0 0, axis 0 1 0, limit lower=-3.14159 upper=3.14159 effort=0.0 velocity=0.0
- added joint 220_230: type continuous, parent 220, child 230, origin xyz=0.25 0.0 0.25 rpy=0 0 0, axis 1 0 0, limit lower=-3.14159 upper=3.14159 effort=0.0 velocity=0.0
- joint 101_112: origin xyz=0.25 0.25 0.0 rpy=0 0 0 -> xyz=0.25 0.25 0.5 rpy=0 0 0; type revolute -> continuous
- joint 130_220: origin xyz=0.25 0.0 -0.25 rpy=0 0 0 -> xyz=0.5 0.0 0.0 rpy=0 0 0

File: files/body1.urdf (robot description, URDF)
Before this commit: robot robot, 20 links, 19 joints
Links:
- removed link 000
- removed link 010
- removed link 011
- removed link 022
- removed link 032
- removed link 120
- removed link 131
- removed link 200
- removed link 201
- removed link 210
- removed link 220
- added link 001, mass 1; collision box size=0.5 0.5 0.5; visual box size=0.5 0.5 0.5
- added link 002, mass 1; collision box size=0.5 0.5 0.5; visual box size=0.5 0.5 0.5
- added link 020, mass 1; collision box size=0.5 0.5 0.5; visual box size=0.5 0.5 0.5
- added link 100, mass 1; collision box size=0.5 0.5 0.5; visual box size=0.5 0.5 0.5
- added link 110, mass 1; collision box size=0.5 0.5 0.5; visual box size=0.5 0.5 0.5
- added link 122, mass 1; collision box size=0.5 0.5 0.5; visual box size=0.5 0.5 0.5
- added link 211, mass 1; collision box size=0.5 0.5 0.5; visual box size=0.5 0.5 0.5
- added link 222, mass 1; collision box size=0.5 0.5 0.5; visual box size=0.5 0.5 0.5
- added link 231, mass 1; collision box size=0.5 0.5 0.5; visual box size=0.5 0.5 0.5
Joints:
- removed joint 000_011
- removed joint 011_010
- removed joint 011_012
- removed joint 011_022
- removed joint 012_102
- removed joint 022_031
- removed joint 022_032
- removed joint 031_030
- removed joint 031_121
- removed joint 031_132
- removed joint 032_131
- removed joint 102_201
- removed joint 121_120
- removed joint 131_230
- removed joint 131_232
- removed joint 201_200
- removed joint 201_210
- removed joint 210_220
- added joint 001_002: type revolute, parent 001, child 002, origin xyz=0.25 0.0 1.0 rpy=0 0 0, axis 0 1 0, limit lower=-3.14159 upper=3.14159 effort=0.0 velocity=0.0
- added joint 001_012: type revolute, parent 001, child 012, origin xyz=0.0 0.25 1.0 rpy=0 0 0, axis 1 0 0, limit lower=-3.14159 upper=3.14159 effort=0.0 velocity=0.0
- added joint 001_100: type revolute, parent 001, child 100, origin xyz=0.25 0.0 0.5 rpy=0 0 0, axis 0 1 0, limit lower=-3.14159 upper=3.14159 effort=0.0 velocity=0.0
- added joint 002_102: type revolute, parent 002, child 102, origin xyz=0.0 0.0 0.5 rpy=0 0 0, axis 0 1 0, limit lower=-3.14159 upper=3.14159 effort=0.0 velocity=0.0
- added joint 012_122: type revolute, parent 012, child 122, origin xyz=0.25 0.5 0.25 rpy=0 0 0, axis 0 0 1, limit lower=-3.14159 upper=3.14159 effort=0.0 velocity=0.0
- added joint 020_030: type continuous, parent 020, child 030, origin xyz=-0.25 0.25 -0.5 rpy=0 0 0, axis 1 0 0, limit lower=-3.14159 upper=3.14159 effort=0.0 velocity=0.0
- added joint 030_031: type revolute, parent 030, child 031, origin xyz=0.0 0.5 0.5 rpy=0 0 0, axis 1 0 0, limit lower=-3.14159 upper=3.14159 effort=0.0 velocity=0.0
- added joint 100_110: type continuous, parent 100, child 110, origin xyz=0.0 0.25 -0.25 rpy=0 0 0, axis 0 0 1, limit lower=-3.14159 upper=3.14159 effort=0.0 velocity=0.0
- added joint 112_121: type continuous, parent 112, child 121, origin xyz=0.25 0.25 -0.5 rpy=0 0 0, axis 1 0 0, limit lower=-3.14159 upper=3.14159 effort=0.0 velocity=0.0
- added joint 112_211: type revolute, parent 112, child 211, origin xyz=0.5 0.0 -0.5 rpy=0 0 0, axis 0 1 0, limit lower=-3.14159 upper=3.14159 effort=0.0 velocity=0.0
- added joint 121_020: type revolute, parent 121, child 020, origin xyz=-0.25 0.25 -0.5 rpy=0 0 0, axis 0 1 0, limit lower=-3.14159 upper=3.14159 effort=0.0 velocity=0.0
- added joint 121_132: type revolute, parent 121, child 132, origin xyz=0.0 0.5 0.0 rpy=0 0 0, axis 1 0 0, limit lower=-3.14159 upper=3.14159 effort=0.0 velocity=0.0
- added joint 121_231: type revolute, parent 121, child 231, origin xyz=0.25 0.5 -0.25 rpy=0 0 0, axis 0 0 1, limit lower=-3.14159 upper=3.14159 effort=0.0 velocity=0.0
- added joint 211_222: type revolute, parent 211, child 222, origin xyz=0.25 0.25 0.0 rpy=0 0 0, axis 1 0 0, limit lower=-3.14159 upper=3.14159 effort=0.0 velocity=0.0
- added joint 231_230: type continuous, parent 231, child 230, origin xyz=0.0 0.25 -0.25 rpy=0 0 0, axis 0 1 0, limit lower=-3.14159 upper=3.14159 effort=0.0 velocity=0.0
- added joint 231_232: type revolute, parent 231, child 232, origin xyz=0.25 0.0 0.25 rpy=0 0 0, axis 1 0 0, limit lower=-3.14159 upper=3.14159 effort=0.0 velocity=0.0
- joint 012_112: axis 0 0 1 -> 0 1 0; origin xyz=0.0 -0.25 0.25 rpy=0 0 0 -> xyz=0.25 0.25 0.5 rpy=0 0 0; type continuous -> revolute

File: files/body2.urdf (robot description, URDF)
Before this commit: robot robot, 24 links, 23 joints
Links:
- removed link 002
- removed link 011
- removed link 012
- removed link 030
- removed link 032
- removed link 100
- removed link 102
- removed link 110
- removed link 121
- removed link 122
- removed link 130
- removed link 202
- removed link 211
- removed link 220
- removed link 222
- removed link 230
- added link 010, mass 1; collision box size=0.5 0.5 0.5; visual box size=0.5 0.5 0.5
- added link 020, mass 1; collision box size=0.5 0.5 0.5; visual box size=0.5 0.5 0.5
- added link 022, mass 1; collision box size=0.5 0.5 0.5; visual box size=0.5 0.5 0.5
- added link 031, mass 1; collision box size=0.5 0.5 0.5; visual box size=0.5 0.5 0.5
- added link 132, mass 1; collision box size=0.5 0.5 0.5; visual box size=0.5 0.5 0.5
- added link 210, mass 1; collision box size=0.5 0.5 0.5; visual box size=0.5 0.5 0.5
Joints:
- removed joint 002_011
- removed joint 002_101
- removed joint 011_012
- removed joint 011_021
- removed joint 011_110
- removed joint 011_112
- removed joint 021_030
- removed joint 021_032
- removed joint 021_122
- removed joint 030_130
- removed joint 030_131
- removed joint 101_102
- removed joint 110_111
- removed joint 110_200
- removed joint 112_202
- removed joint 112_211
- removed joint 112_222
- removed joint 130_230
- removed joint 131_121
- removed joint 200_100
- removed joint 211_220
- removed joint 222_231
- removed joint 231_232
- added joint 010_020: type continuous, parent 010, child 020, origin xyz=0.0 0.75 0.25 rpy=0 0 0, axis 0 0 1, limit lower=-3.14159 upper=3.14159 effort=0.0 velocity=0.0
- added joint 010_021: type continuous, parent 010, child 021, origin xyz=0.0 0.75 0.5 rpy=0 0 0, axis 1 0 0, limit lower=-3.14159 upper=3.14159 effort=0.0 velocity=0.0
- added joint 010_111: type continuous, parent 010, child 111, origin xyz=0.25 0.5 0.5 rpy=0 0 0, axis 0 1 0, limit lower=-3.14159 upper=3.14159 effort=0.0 velocity=0.0
- added joint 021_022: type revolute, parent 021, child 022, origin xyz=0.25 0.25 0.5 rpy=0 0 0, axis 0 1 0, limit lower=-3.14159 upper=3.14159 effort=0.0 velocity=0.0
- added joint 022_031: type revolute, parent 022, child 031, origin xyz=-0.25 0.25 0.0 rpy=0 0 0, axis 1 0 0, limit lower=-3.14159 upper=3.14159 effort=0.0 velocity=0.0
- added joint 022_112: type revolute, parent 022, child 112, origin xyz=0.0 -0.25 0.25 rpy=0 0 0, axis 0 0 1, limit lower=-3.14159 upper=3.14159 effort=0.0 velocity=0.0
- added joint 031_131: type continuous, parent 031, child 131, origin xyz=0.25 0.0 -0.25 rpy=0 0 0, axis 0 0 1, limit lower=-3.14159 upper=3.14159 effort=0.0 velocity=0.0
- added joint 101_200: type continuous, parent 101, child 200, origin xyz=0.25 -0.25 -0.5 rpy=0 0 0, axis 0 1 0, limit lower=-3.14159 upper=3.14159 effort=0.0 velocity=0.0
- added joint 111_210: type revolute, parent 111, child 210, origin xyz=0.5 0.0 0.0 rpy=0 0 0, axis 0 1 0, limit lower=-3.14159 upper=3.14159 effort=0.0 velocity=0.0
- added joint 112_101: type revolute, parent 112, child 101, origin xyz=0.25 -0.5 -0.25 rpy=0 0 0, axis 1 0 0, limit lower=-3.14159 upper=3.14159 effort=0.0 velocity=0.0
- added joint 131_132: type revolute, parent 131, child 132, origin xyz=0.5 0.25 0.25 rpy=0 0 0, axis 0 1 0, limit lower=-3.14159 upper=3.14159 effort=0.0 velocity=0.0
- added joint 131_232: type revolute, parent 131, child 232, origin xyz=0.5 0.25 0.25 rpy=0 0 0, axis 0 1 0, limit lower=-3.14159 upper=3.14159 effort=0.0 velocity=0.0
- added joint 132_231: type continuous, parent 132, child 231, origin xyz=0.0 0.0 0.0 rpy=0 0 0, axis 0 1 0, limit lower=-3.14159 upper=3.14159 effort=0.0 velocity=0.0

File: files/body3.urdf (robot description, URDF)
Before this commit: robot robot, 14 links, 13 joints
Links:
- removed link 001
- removed link 002
- removed link 021
- removed link 131
- removed link 201
- removed link 212
- removed link 221
- removed link 222
- removed link 230
- removed link 231
- added link 000, mass 1; collision box size=0.5 0.5 0.5; visual box size=0.5 0.5 0.5
- added link 010, mass 1; collision box size=0.5 0.5 0.5; visual box size=0.5 0.5 0.5
- added link 011, mass 1; collision box size=0.5 0.5 0.5; visual box size=0.5 0.5 0.5
- added link 022, mass 1; collision box size=0.5 0.5 0.5; visual box size=0.5 0.5 0.5
- added link 030, mass 1; collision box size=0.5 0.5 0.5; visual box size=0.5 0.5 0.5
- added link 102, mass 1; collision box size=0.5 0.5 0.5; visual box size=0.5 0.5 0.5
- added link 112, mass 1; collision box size=0.5 0.5 0.5; visual box size=0.5 0.5 0.5
- added link 121, mass 1; collision box size=0.5 0.5 0.5; visual box size=0.5 0.5 0.5
- added link 122, mass 1; collision box size=0.5 0.5 0.5; visual box size=0.5 0.5 0.5
- added link 200, mass 1; collision box size=0.5 0.5 0.5; visual box size=0.5 0.5 0.5
- added link 202, mass 1; collision box size=0.5 0.5 0.5; visual box size=0.5 0.5 0.5
Joints:
- removed joint 001_002
- removed joint 002_101
- removed joint 021_031
- removed joint 101_201
- removed joint 120_021
- removed joint 131_132
- removed joint 201_212
- removed joint 212_221
- removed joint 221_120
- removed joint 221_222
- removed joint 221_230
- removed joint 222_231
- removed joint 230_131
- added joint 000_010: type continuous, parent 000, child 010, origin xyz=0.0 0.25 0.5 rpy=0 0 0, axis 1 0 0, limit lower=-3.14159 upper=3.14159 effort=0.0 velocity=0.0
- added joint 000_101: type revolute, parent 000, child 101, origin xyz=0.25 0.0 0.5 rpy=0 0 0, axis 0 1 0, limit lower=-3.14159 upper=3.14159 effort=0.0 velocity=0.0
- added joint 010_011: type continuous, parent 010, child 011, origin xyz=0.25 0.25 0.0 rpy=0 0 0, axis 0 1 0, limit lower=-3.14159 upper=3.14159 effort=0.0 velocity=0.0
- added joint 010_120: type revolute, parent 010, child 120, origin xyz=0.25 0.5 -0.25 rpy=0 0 0, axis 0 0 1, limit lower=-3.14159 upper=3.14159 effort=0.0 velocity=0.0
- added joint 011_022: type revolute, parent 011, child 022, origin xyz=-0.25 0.25 0.5 rpy=0 0 0, axis 1 0 0, limit lower=-3.14159 upper=3.14159 effort=0.0 velocity=0.0
- added joint 011_112: type revolute, parent 011, child 112, origin xyz=0.0 0.0 0.5 rpy=0 0 0, axis 0 1 0, limit lower=-3.14159 upper=3.14159 effort=0.0 velocity=0.0
- added joint 022_031: type revolute, parent 022, child 031, origin xyz=0.0 0.5 0.0 rpy=0 0 0, axis 1 0 0, limit lower=-3.14159 upper=3.14159 effort=0.0 velocity=0.0
- added joint 031_030: type continuous, parent 031, child 030, origin xyz=0.0 0.0 -0.5 rpy=0 0 0, axis 1 0 0, limit lower=-3.14159 upper=3.14159 effort=0.0 velocity=0.0
- added joint 101_102: type revolute, parent 101, child 102, origin xyz=0.25 0.25 0.5 rpy=0 0 0, axis 1 0 0, limit lower=-3.14159 upper=3.14159 effort=0.0 velocity=0.0
- added joint 101_200: type continuous, parent 101, child 200, origin xyz=0.5 0.0 0.0 rpy=0 0 0, axis 0 1 0, limit lower=-3.14159 upper=3.14159 effort=0.0 velocity=0.0
- added joint 101_202: type revolute, parent 101, child 202, origin xyz=0.5 0.0 0.5 rpy=0 0 0, axis 0 1 0, limit lower=-3.14159 upper=3.14159 effort=0.0 velocity=0.0
- added joint 112_121: type continuous, parent 112, child 121, origin xyz=0.25 0.25 0.0 rpy=0 0 0, axis 1 0 0, limit lower=-3.14159 upper=3.14159 effort=0.0 velocity=0.0
- added joint 112_122: type continuous, parent 112, child 122, origin xyz=0.25 0.25 0.25 rpy=0 0 0, axis 1 0 0, limit lower=-3.14159 upper=3.14159 effort=0.0 velocity=0.0
- added joint 122_132: type revolute, parent 122, child 132, origin xyz=0.0 0.5 0.25 rpy=0 0 0, axis 1 0 0, limit lower=-3.14159 upper=3.14159 effort=0.0 velocity=0.0

File: files/body4.urdf (robot description, URDF)
Before this commit: robot robot, 21 links, 20 joints
Links:
- removed link 000
- removed link 001
- removed link 021
- removed link 022
- removed link 031
- removed link 100
- removed link 112
- added link 002, mass 1; collision box size=0.5 0.5 0.5; visual box size=0.5 0.5 0.5
- added link 030, mass 1; collision box size=0.5 0.5 0.5; visual box size=0.5 0.5 0.5
- added link 032, mass 1; collision box size=0.5 0.5 0.5; visual box size=0.5 0.5 0.5
- added link 110, mass 1; collision box size=0.5 0.5 0.5; visual box size=0.5 0.5 0.5
- added link 121, mass 1; collision box size=0.5 0.5 0.5; visual box size=0.5 0.5 0.5
- added link 122, mass 1; collision box size=0.5 0.5 0.5; visual box size=0.5 0.5 0.5
- added link 130, mass 1; collision box size=0.5 0.5 0.5; visual box size=0.5 0.5 0.5
- added link 210, mass 1; collision box size=0.5 0.5 0.5; visual box size=0.5 0.5 0.5
- added link 221, mass 1; collision box size=0.5 0.5 0.5; visual box size=0.5 0.5 0.5
- added link 231, mass 1; collision box size=0.5 0.5 0.5; visual box size=0.5 0.5 0.5
Joints:
- removed joint 000_001
- removed joint 000_011
- removed joint 000_100
- removed joint 012_112
- removed joint 020_021
- removed joint 021_022
- removed joint 021_031
- removed joint 021_120
- removed joint 101_102
- removed joint 101_211
- removed joint 102_111
- removed joint 120_220
- removed joint 131_230
- removed joint 131_232
- added joint 002_011: type revolute, parent 002, child 011, origin xyz=0.0 0.25 1.0 rpy=0 0 0, axis 1 0 0, limit lower=-3.14159 upper=3.14159 effort=0.0 velocity=0.0
- added joint 002_102: type revolute, parent 002, child 102, origin xyz=0.25 0.0 1.0 rpy=0 0 0, axis 0 1 0, limit lower=-3.14159 upper=3.14159 effort=0.0 velocity=0.0
- added joint 012_111: type revolute, parent 012, child 111, origin xyz=0.25 -0.25 0.0 rpy=0 0 0, axis 0 1 0, limit lower=-3.14159 upper=3.14159 effort=0.0 velocity=0.0
- added joint 012_122: type continuous, parent 012, child 122, origin xyz=0.25 0.0 0.25 rpy=0 0 0, axis 0 0 1, limit lower=-3.14159 upper=3.14159 effort=0.0 velocity=0.0
- added joint 020_030: type continuous, parent 020, child 030, origin xyz=-0.25 0.5 -0.25 rpy=0 0 0, axis 0 0 1, limit lower=-3.14159 upper=3.14159 effort=0.0 velocity=0.0
- added joint 020_110: type continuous, parent 020, child 110, origin xyz=0.25 0.0 -0.25 rpy=0 0 0, axis 0 0 1, limit lower=-3.14159 upper=3.14159 effort=0.0 velocity=0.0
- added joint 020_130: type revolute, parent 020, child 130, origin xyz=0.25 0.5 -0.25 rpy=0 0 0, axis 0 0 1, limit lower=-3.14159 upper=3.14159 effort=0.0 velocity=0.0
- added joint 110_120: type continuous, parent 110, child 120, origin xyz=0.0 0.0 0.0 rpy=0 0 0, axis 0 0 1, limit lower=-3.14159 upper=3.14159 effort=0.0 velocity=0.0
- added joint 110_210: type revolute, parent 110, child 210, origin xyz=0.5 -0.5 0.0 rpy=0 0 0, axis 0 0 1, limit lower=-3.14159 upper=3.14159 effort=0.0 velocity=0.0
- added joint 110_220: type continuous, parent 110, child 220, origin xyz=0.5 0.0 0.0 rpy=0 0 0, axis 0 0 1, limit lower=-3.14159 upper=3.14159 effort=0.0 velocity=0.0
- added joint 120_121: type continuous, parent 120, child 121, origin xyz=0.0 0.25 0.25 rpy=0 0 0, axis 0 1 0, limit lower=-3.14159 upper=3.14159 effort=0.0 velocity=0.0
- added joint 120_230: type continuous, parent 120, child 230, origin xyz=0.5 0.5 0.0 rpy=0 0 0, axis 0 0 1, limit lower=-3.14159 upper=3.14159 effort=0.0 velocity=0.0
- added joint 122_032: type revolute, parent 122, child 032, origin xyz=0.0 0.5 0.0 rpy=0 0 0, axis 0 0 1, limit lower=-3.14159 upper=3.14159 effort=0.0 velocity=0.0
- added joint 122_232: type revolute, parent 122, child 232, origin xyz=0.5 0.5 0.0 rpy=0 0 0, axis 0 0 1, limit lower=-3.14159 upper=3.14159 effort=0.0 velocity=0.0
- added joint 210_211: type continuous, parent 210, child 211, origin xyz=0.25 0.0 0.25 rpy=0 0 0, axis 1 0 0, limit lower=-3.14159 upper=3.14159 effort=0.0 velocity=0.0
- added joint 220_221: type revolute, parent 220, child 221, origin xyz=0.5 0.25 0.25 rpy=0 0 0, axis 0 1 0, limit lower=-3.14159 upper=3.14159 effort=0.0 velocity=0.0
- added joint 230_231: type continuous, parent 230, child 231, origin xyz=0.25 0.5 0.25 rpy=0 0 0, axis 1 0 0, limit lower=-3.14159 upper=3.14159 effort=0.0 velocity=0.0
- joint 011_012: axis 0 1 0 -> 1 0 0; origin xyz=-0.25 0.25 0.5 rpy=0 0 0 -> xyz=0.0 0.5 0.0 rpy=0 0 0; type continuous -> revolute
- joint 011_020: origin xyz=0.0 0.5 0.0 rpy=0 0 0 -> xyz=0.0 0.5 -0.5 rpy=0 0 0
- joint 011_101: origin xyz=0.25 0.0 0.25 rpy=0 0 0 -> xyz=0.25 0.0 -0.25 rpy=0 0 0; type continuous -> revolute
- joint 101_200: type revolute -> continuous
- joint 120_131: origin xyz=0.25 0.25 0.0 rpy=0 0 0 -> xyz=0.25 0.5 0.25 rpy=0 0 0
- joint 211_212: axis 0 1 0 -> 1 0 0; origin xyz=0.5 0.25 0.25 rpy=0 0 0 -> xyz=0.0 0.25 0.5 rpy=0 0 0
