Commit message: diagrams

File: files/body5.urdf (robot description, URDF)
Before this commit: robot robot, 14 links, 13 joints
Links:
- removed link 022
- removed link 100
- removed link 201
- removed link 231
- added link 002, mass 1; collision box size=0.5 0.5 0.5; visual box size=0.5 0.5 0.5
- added link 010, mass 1; collision box size=0.5 0.5 0.5; visual box size=0.5 0.5 0.5
- added link 021, mass 1; collision box size=0.5 0.5 0.5; visual box size=0.5 0.5 0.5
- added link 030, mass 1; collision box size=0.5 0.5 0.5; visual box size=0.5 0.5 0.5
- added link 031, mass 1; collision box size=0.5 0.5 0.5; visual box size=0.5 0.5 0.5
- added link 101, mass 1; collision box size=0.5 0.5 0.5; visual box size=0.5 0.5 0.5
- added link 111, mass 1; collision box size=0.5 0.5 0.5; visual box size=0.5 0.5 0.5
- added link 120, mass 1; collision box size=0.5 0.5 0.5; visual box size=0.5 0.5 0.5
- added link 121, mass 1; collision box size=0.5 0.5 0.5; visual box size=0.5 0.5 0.5
- added link 130, mass 1; collision box size=0.5 0.5 0.5; visual box size=0.5 0.5 0.5
- added link 131, mass 1; collision box size=0.5 0.5 0.5; visual box size=0.5 0.5 0.5
- added link 221, mass 1; collision box size=0.5 0.5 0.5; visual box size=0.5 0.5 0.5
- added link 222, mass 1; collision box size=0.5 0.5 0.5; visual box size=0.5 0.5 0.5
Joints:
- removed joint 000_100
- removed joint 011_022
- removed joint 022_122
- removed joint 102_201
- removed joint 122_132
- removed joint 132_231
- removed joint 201_210
- removed joint 201_211
- added joint 000_010: type continuous, parent 000, child 010, origin xyz=0.0 0.25 0.25 rpy=0 0 0, axis 1 0 0, limit lower=-3.14159 upper=3.14159 effort=0.0 velocity=0.0
- added joint 010_111: type continuous, parent 010, child 111, origin xyz=0.25 0.25 0.25 rpy=0 0 0, axis 0 1 0, limit lower=-3.14159 upper=3.14159 effort=0.0 velocity=0.0
- added joint 011_101: type revolute, parent 011, child 101, origin xyz=0.25 0.0 0.25 rpy=0 0 0, axis 0 0 1, limit lower=-3.14159 upper=3.14159 effort=0.0 velocity=0.0
- added joint 012_021: type revolute, parent 012, child 021, origin xyz=0.25 0.25 0.0 rpy=0 0 0, axis 1 0 0, limit lower=-3.14159 upper=3.14159 effort=0.0 velocity=0.0
- added joint 012_122: type continuous, parent 012, child 122, origin xyz=0.5 0.25 0.25 rpy=0 0 0, axis 0 0 1, limit lower=-3.14159 upper=3.14159 effort=0.0 velocity=0.0
- added joint 021_030: type revolute, parent 021, child 030, origin xyz=0.0 0.5 -0.5 rpy=0 0 0, axis 1 0 0, limit lower=-3.14159 upper=3.14159 effort=0.0 velocity=0.0
- added joint 021_031: type continuous, parent 021, child 031, origin xyz=0.25 0.5 -0.25 rpy=0 0 0, axis 0 0 1, limit lower=-3.14159 upper=3.14159 effort=0.0 velocity=0.0
- added joint 030_120: type continuous, parent 030, child 120, origin xyz=0.25 0.0 -0.25 rpy=0 0 0, axis 0 0 1, limit lower=-3.14159 upper=3.14159 effort=0.0 velocity=0.0
- added joint 030_130: type continuous, parent 030, child 130, origin xyz=0.25 0.25 0.0 rpy=0 0 0, axis 0 1 0, limit lower=-3.14159 upper=3.14159 effort=0.0 velocity=0.0
- added joint 031_121: type continuous, parent 031, child 121, origin xyz=0.0 0.0 0.0 rpy=0 0 0, axis 0 0 1, limit lower=-3.14159 upper=3.14159 effort=0.0 velocity=0.0
- added joint 102_002: type revolute, parent 102, child 002, origin xyz=0.0 -0.25 0.0 rpy=0 0 0, axis 0 1 0, limit lower=-3.14159 upper=3.14159 effort=0.0 velocity=0.0
- added joint 111_211: type continuous, parent 111, child 211, origin xyz=0.5 0.0 0.25 rpy=0 0 0, axis 0 1 0, limit lower=-3.14159 upper=3.14159 effort=0.0 velocity=0.0
- added joint 120_210: type revolute, parent 120, child 210, origin xyz=0.5 -0.5 0.0 rpy=0 0 0, axis 0 0 1, limit lower=-3.14159 upper=3.14159 effort=0.0 velocity=0.0
- added joint 122_131: type revolute, parent 122, child 131, origin xyz=0.25 0.5 -0.25 rpy=0 0 0, axis 1 0 0, limit lower=-3.14159 upper=3.14159 effort=0.0 velocity=0.0
- added joint 122_221: type revolute, parent 122, child 221, origin xyz=0.5 0.25 -0.25 rpy=0 0 0, axis 0 1 0, limit lower=-3.14159 upper=3.14159 effort=0.0 velocity=0.0
- added joint 131_132: type revolute, parent 131, child 132, origin xyz=0.0 0.5 0.0 rpy=0 0 0, axis 1 0 0, limit lower=-3.14159 upper=3.14159 effort=0.0 velocity=0.0
- added joint 211_222: type revolute, parent 211, child 222, origin xyz=0.25 0.25 0.25 rpy=0 0 0, axis 1 0 0, limit lower=-3.14159 upper=3.14159 effort=0.0 velocity=0.0
- joint 000_011: type revolute -> continuous
- joint 000_110: type continuous -> revolute
- joint 011_012: type continuous -> revolute
- joint 102_212: type continuous -> revolute

File: files/body6.urdf (robot description, URDF)
Before this commit: robot robot, 18 links, 17 joints
Links:
- removed link 000
- removed link 022
- removed link 030
- removed link 112
- removed link 121
- removed link 122
- removed link 131
- removed link 132
- removed link 201
- removed link 231
- removed link 232
- added link 002, mass 1; collision box size=0.5 0.5 0.5; visual box size=0.5 0.5 0.5
- added link 010, mass 1; collision box size=0.5 0.5 0.5; visual box size=0.5 0.5 0.5
- added link 020, mass 1; collision box size=0.5 0.5 0.5; visual box size=0.5 0.5 0.5
- added link 021, mass 1; collision box size=0.5 0.5 0.5; visual box size=0.5 0.5 0.5
- added link 100, mass 1; collision box size=0.5 0.5 0.5; visual box size=0.5 0.5 0.5
- added link 101, mass 1; collision box size=0.5 0.5 0.5; visual box size=0.5 0.5 0.5
- added link 102, mass 1; collision box size=0.5 0.5 0.5; visual box size=0.5 0.5 0.5
- added link 111, mass 1; collision box size=0.5 0.5 0.5; visual box size=0.5 0.5 0.5
- added link 200, mass 1; collision box size=0.5 0.5 0.5; visual box size=0.5 0.5 0.5
- added link 212, mass 1; collision box size=0.5 0.5 0.5; visual box size=0.5 0.5 0.5
- added link 221, mass 1; collision box size=0.5 0.5 0.5; visual box size=0.5 0.5 0.5
- added link 222, mass 1; collision box size=0.5 0.5 0.5; visual box size=0.5 0.5 0.5
Joints:
- removed joint 000_011
- removed joint 011_012
- removed joint 011_022
- removed joint 012_112
- removed joint 022_031
- removed joint 022_032
- removed joint 022_121
- removed joint 022_122
- removed joint 032_131
- removed joint 121_211
- removed joint 131_030
- removed joint 131_132
- removed joint 131_230
- removed joint 131_231
- removed joint 201_210
- removed joint 211_201
- removed joint 231_232
- added joint 002_011: type revolute, parent 002, child 011, origin xyz=0.0 0.25 1.0 rpy=0 0 0, axis 1 0 0, limit lower=-3.14159 upper=3.14159 effort=0.0 velocity=0.0
- added joint 002_012: type continuous, parent 002, child 012, origin xyz=0.25 0.25 1.25 rpy=0 0 0, axis 0 0 1, limit lower=-3.14159 upper=3.14159 effort=0.0 velocity=0.0
- added joint 002_101: type continuous, parent 002, child 101, origin xyz=0.25 0.0 1.0 rpy=0 0 0, axis 0 1 0, limit lower=-3.14159 upper=3.14159 effort=0.0 velocity=0.0
- added joint 002_102: type continuous, parent 002, child 102, origin xyz=0.25 -0.25 1.25 rpy=0 0 0, axis 0 0 1, limit lower=-3.14159 upper=3.14159 effort=0.0 velocity=0.0
- added joint 010_100: type revolute, parent 010, child 100, origin xyz=0.0 -0.25 -0.25 rpy=0 0 0, axis 0 0 1, limit lower=-3.14159 upper=3.14159 effort=0.0 velocity=0.0
- added joint 011_020: type revolute, parent 011, child 020, origin xyz=0.0 0.5 -0.5 rpy=0 0 0, axis 1 0 0, limit lower=-3.14159 upper=3.14159 effort=0.0 velocity=0.0
- added joint 011_021: type continuous, parent 011, child 021, origin xyz=0.0 0.5 0.0 rpy=0 0 0, axis 1 0 0, limit lower=-3.14159 upper=3.14159 effort=0.0 velocity=0.0
- added joint 011_111: type revolute, parent 011, child 111, origin xyz=0.25 0.25 -0.5 rpy=0 0 0, axis 0 1 0, limit lower=-3.14159 upper=3.14159 effort=0.0 velocity=0.0
- added joint 020_031: type continuous, parent 020, child 031, origin xyz=0.0 0.5 0.0 rpy=0 0 0, axis 1 0 0, limit lower=-3.14159 upper=3.14159 effort=0.0 velocity=0.0
- added joint 031_032: type continuous, parent 031, child 032, origin xyz=0.0 0.0 0.5 rpy=0 0 0, axis 1 0 0, limit lower=-3.14159 upper=3.14159 effort=0.0 velocity=0.0
- added joint 101_200: type continuous, parent 101, child 200, origin xyz=0.5 0.0 -0.5 rpy=0 0 0, axis 0 1 0, limit lower=-3.14159 upper=3.14159 effort=0.0 velocity=0.0
- added joint 111_010: type continuous, parent 111, child 010, origin xyz=0.0 0.0 0.0 rpy=0 0 0, axis 0 1 0, limit lower=-3.14159 upper=3.14159 effort=0.0 velocity=0.0
- added joint 111_210: type revolute, parent 111, child 210, origin xyz=0.5 0.0 0.0 rpy=0 0 0, axis 0 1 0, limit lower=-3.14159 upper=3.14159 effort=0.0 velocity=0.0
- added joint 111_212: type continuous, parent 111, child 212, origin xyz=0.5 0.0 0.5 rpy=0 0 0, axis 0 1 0, limit lower=-3.14159 upper=3.14159 effort=0.0 velocity=0.0
- added joint 210_211: type continuous, parent 210, child 211, origin xyz=0.25 -0.25 0.0 rpy=0 0 0, axis 1 0 0, limit lower=-3.14159 upper=3.14159 effort=0.0 velocity=0.0
- added joint 211_221: type revolute, parent 211, child 221, origin xyz=-0.25 0.5 0.25 rpy=0 0 0, axis 0 0 1, limit lower=-3.14159 upper=3.14159 effort=0.0 velocity=0.0
- added joint 211_222: type continuous, parent 211, child 222, origin xyz=0.0 0.5 0.5 rpy=0 0 0, axis 1 0 0, limit lower=-3.14159 upper=3.14159 effort=0.0 velocity=0.0
- added joint 221_230: type revolute, parent 221, child 230, origin xyz=0.25 0.5 -0.25 rpy=0 0 0, axis 1 0 0, limit lower=-3.14159 upper=3.14159 effort=0.0 velocity=0.0

File: files/body7.urdf (robot description, URDF)
Before this commit: robot robot, 18 links, 17 joints
Links:
- removed link 001
- removed link 031
- removed link 101
- removed link 102
- removed link 121
- removed link 210
- removed link 232
- added link 110, mass 1; collision box size=0.5 0.5 0.5; visual box size=0.5 0.5 0.5
- added link 112, mass 1; collision box size=0.5 0.5 0.5; visual box size=0.5 0.5 0.5
- added link 120, mass 1; collision box size=0.5 0.5 0.5; visual box size=0.5 0.5 0.5
- added link 131, mass 1; collision box size=0.5 0.5 0.5; visual box size=0.5 0.5 0.5
- added link 222, mass 1; collision box size=0.5 0.5 0.5; visual box size=0.5 0.5 0.5
- added link 231, mass 1; collision box size=0.5 0.5 0.5; visual box size=0.5 0.5 0.5
Joints:
- removed joint 001_010
- removed joint 001_012
- removed joint 001_100
- removed joint 001_102
- removed joint 011_101
- removed joint 020_031
- removed joint 031_121
- removed joint 101_111
- removed joint 111_210
- removed joint 121_122
- removed joint 121_130
- removed joint 121_211
- removed joint 122_232
- removed joint 130_230
- added joint 010_100: type revolute, parent 010, child 100, origin xyz=0.25 0.25 0.25 rpy=0 0 0, axis 0 0 1, limit lower=-3.14159 upper=3.14159 effort=0.0 velocity=0.0
- added joint 010_110: type continuous, parent 010, child 110, origin xyz=0.25 0.25 0.25 rpy=0 0 0, axis 0 0 1, limit lower=-3.14159 upper=3.14159 effort=0.0 velocity=0.0
- added joint 011_012: type continuous, parent 011, child 012, origin xyz=0.25 0.25 0.5 rpy=0 0 0, axis 0 1 0, limit lower=-3.14159 upper=3.14159 effort=0.0 velocity=0.0
- added joint 012_111: type revolute, parent 012, child 111, origin xyz=0.0 0.0 0.0 rpy=0 0 0, axis 0 1 0, limit lower=-3.14159 upper=3.14159 effort=0.0 velocity=0.0
- added joint 030_120: type revolute, parent 030, child 120, origin xyz=0.25 0.0 0.25 rpy=0 0 0, axis 0 0 1, limit lower=-3.14159 upper=3.14159 effort=0.0 velocity=0.0
- added joint 030_130: type continuous, parent 030, child 130, origin xyz=0.25 0.0 0.25 rpy=0 0 0, axis 0 0 1, limit lower=-3.14159 upper=3.14159 effort=0.0 velocity=0.0
- added joint 111_112: type continuous, parent 111, child 112, origin xyz=0.25 0.0 0.0 rpy=0 0 0, axis 0 1 0, limit lower=-3.14159 upper=3.14159 effort=0.0 velocity=0.0
- added joint 111_122: type revolute, parent 111, child 122, origin xyz=0.25 0.25 0.0 rpy=0 0 0, axis 1 0 0, limit lower=-3.14159 upper=3.14159 effort=0.0 velocity=0.0
- added joint 111_211: type revolute, parent 111, child 211, origin xyz=0.5 0.0 0.0 rpy=0 0 0, axis 0 1 0, limit lower=-3.14159 upper=3.14159 effort=0.0 velocity=0.0
- added joint 112_222: type revolute, parent 112, child 222, origin xyz=0.25 0.25 0.25 rpy=0 0 0, axis 0 0 1, limit lower=-3.14159 upper=3.14159 effort=0.0 velocity=0.0
- added joint 120_131: type continuous, parent 120, child 131, origin xyz=0.25 0.0 0.25 rpy=0 0 0, axis 1 0 0, limit lower=-3.14159 upper=3.14159 effort=0.0 velocity=0.0
- added joint 120_230: type continuous, parent 120, child 230, origin xyz=0.5 0.0 0.0 rpy=0 0 0, axis 0 0 1, limit lower=-3.14159 upper=3.14159 effort=0.0 velocity=0.0
- added joint 131_231: type revolute, parent 131, child 231, origin xyz=0.25 0.0 0.25 rpy=0 0 0, axis 0 0 1, limit lower=-3.14159 upper=3.14159 effort=0.0 velocity=0.0
- joint 010_011: axis 0 1 0 -> 1 0 0; origin xyz=0.25 0.25 0.0 rpy=0 0 0 -> xyz=0.0 0.25 0.5 rpy=0 0 0; type continuous -> revolute
- joint 011_020: origin xyz=-0.25 0.25 0.0 rpy=0 0 0 -> xyz=0.0 0.5 0.0 rpy=0 0 0; type continuous -> revolute
- joint 020_030: axis 0 0 1 -> 1 0 0; origin xyz=0.25 0.5 -0.25 rpy=0 0 0 -> xyz=0.0 0.5 -0.5 rpy=0 0 0; type continuous -> revolute

File: files/body8.urdf (robot description, URDF)
Before this commit: robot robot, 13 links, 12 joints
Links:
- removed link 011
- removed link 131
- added link 120, mass 1; collision box size=0.5 0.5 0.5; visual box size=0.5 0.5 0.5
- added link 221, mass 1; collision box size=0.5 0.5 0.5; visual box size=0.5 0.5 0.5
- added link 231, mass 1; collision box size=0.5 0.5 0.5; visual box size=0.5 0.5 0.5
- added link 232, mass 1; collision box size=0.5 0.5 0.5; visual box size=0.5 0.5 0.5
Joints:
- removed joint 112_011
- removed joint 130_131
- removed joint 130_230
- added joint 121_231: type continuous, parent 121, child 231, origin xyz=0.5 0.25 -0.25 rpy=0 0 0, axis 0 0 1, limit lower=-3.14159 upper=3.14159 effort=0.0 velocity=0.0
- added joint 122_232: type revolute, parent 122, child 232, origin xyz=0.0 0.25 0.25 rpy=0 0 0, axis 0 0 1, limit lower=-3.14159 upper=3.14159 effort=0.0 velocity=0.0
- added joint 211_221: type revolute, parent 211, child 221, origin xyz=0.0 0.25 -0.25 rpy=0 0 0, axis 0 0 1, limit lower=-3.14159 upper=3.14159 effort=0.0 velocity=0.0
- added joint 221_230: type revolute, parent 221, child 230, origin xyz=0.25 0.5 -0.25 rpy=0 0 0, axis 1 0 0, limit lower=-3.14159 upper=3.14159 effort=0.0 velocity=0.0
- added joint 230_120: type continuous, parent 230, child 120, origin xyz=-0.25 0.0 -0.25 rpy=0 0 0, axis 0 0 1, limit lower=-3.14159 upper=3.14159 effort=0.0 velocity=0.0

File: files/body9.urdf (robot description, URDF)
Before this commit: robot robot, 14 links, 13 joints
Links:
- removed link 001
- removed link 002
- removed link 012
- removed link 020
- removed link 021
- removed link 022
- removed link 102
- removed link 121
- removed link 200
- removed link 211
- removed link 221
- added link 010, mass 1; collision box size=0.5 0.5 0.5; visual box size=0.5 0.5 0.5
- added link 030, mass 1; collision box size=0.5 0.5 0.5; visual box size=0.5 0.5 0.5
- added link 031, mass 1; collision box size=0.5 0.5 0.5; visual box size=0.5 0.5 0.5
- added link 032, mass 1; collision box size=0.5 0.5 0.5; visual box size=0.5 0.5 0.5
- added link 100, mass 1; collision box size=0.5 0.5 0.5; visual box size=0.5 0.5 0.5
- added link 111, mass 1; collision box size=0.5 0.5 0.5; visual box size=0.5 0.5 0.5
- added link 122, mass 1; collision box size=0.5 0.5 0.5; visual box size=0.5 0.5 0.5
- added link 131, mass 1; collision box size=0.5 0.5 0.5; visual box size=0.5 0.5 0.5
- added link 210, mass 1; collision box size=0.5 0.5 0.5; visual box size=0.5 0.5 0.5
- added link 230, mass 1; collision box size=0.5 0.5 0.5; visual box size=0.5 0.5 0.5
Joints:
- removed joint 000_001
- removed joint 001_002
- removed joint 001_012
- removed joint 012_021
- removed joint 012_102
- removed joint 021_020
- removed joint 021_121
- removed joint 102_201
- removed joint 121_022
- removed joint 121_221
- removed joint 201_200
- removed joint 201_211
- removed joint 211_220
- added joint 000_010: type continuous, parent 000, child 010, origin xyz=0.25 0.25 0.25 rpy=0 0 0, axis 0 0 1, limit lower=-3.14159 upper=3.14159 effort=0.0 velocity=0.0
- added joint 000_100: type continuous, parent 000, child 100, origin xyz=0.25 0.0 0.5 rpy=0 0 0, axis 0 1 0, limit lower=-3.14159 upper=3.14159 effort=0.0 velocity=0.0
- added joint 010_111: type revolute, parent 010, child 111, origin xyz=0.0 0.25 0.25 rpy=0 0 0, axis 0 1 0, limit lower=-3.14159 upper=3.14159 effort=0.0 velocity=0.0
- added joint 100_201: type revolute, parent 100, child 201, origin xyz=0.5 0.0 0.0 rpy=0 0 0, axis 0 1 0, limit lower=-3.14159 upper=3.14159 effort=0.0 velocity=0.0
- added joint 100_210: type revolute, parent 100, child 210, origin xyz=0.5 0.25 -0.25 rpy=0 0 0, axis 0 0 1, limit lower=-3.14159 upper=3.14159 effort=0.0 velocity=0.0
- added joint 111_122: type continuous, parent 111, child 122, origin xyz=0.25 0.25 0.5 rpy=0 0 0, axis 1 0 0, limit lower=-3.14159 upper=3.14159 effort=0.0 velocity=0.0
- added joint 122_032: type continuous, parent 122, child 032, origin xyz=-0.25 0.5 0.25 rpy=0 0 0, axis 0 0 1, limit lower=-3.14159 upper=3.14159 effort=0.0 velocity=0.0
- added joint 122_131: type revolute, parent 122, child 131, origin xyz=0.0 0.5 0.0 rpy=0 0 0, axis 1 0 0, limit lower=-3.14159 upper=3.14159 effort=0.0 velocity=0.0
- added joint 131_030: type revolute, parent 131, child 030, origin xyz=-0.25 0.25 -0.5 rpy=0 0 0, axis 0 1 0, limit lower=-3.14159 upper=3.14159 effort=0.0 velocity=0.0
- added joint 131_031: type continuous, parent 131, child 031, origin xyz=-0.25 0.0 -0.25 rpy=0 0 0, axis 0 0 1, limit lower=-3.14159 upper=3.14159 effort=0.0 velocity=0.0
- added joint 131_230: type revolute, parent 131, child 230, origin xyz=0.25 0.25 -0.5 rpy=0 0 0, axis 0 1 0, limit lower=-3.14159 upper=3.14159 effort=0.0 velocity=0.0
- added joint 210_220: type revolute, parent 210, child 220, origin xyz=0.25 0.5 0.25 rpy=0 0 0, axis 1 0 0, limit lower=-3.14159 upper=3.14159 effort=0.0 velocity=0.0
